Commit message: fixed image_transform startup bug and fixed camera angle in tf

File: rr_description/speedi/speedi.urdf (robot description, URDF)
Before this commit: robot speedi, 6 links, 5 joints
Links:
- removed link lidar
- added link laser
Joints:
- joint imu: axis 0 0 0 -> (none)
- joint lidar_joint: axis 0 0 0 -> (none); child lidar -> laser

Commit message: image_transform uses a list of topics to transform
also changed ground frame to "map" and deleted the obsolete transform tester

File: rr_description/speedi/speedi.urdf (robot description, URDF)
Before this commit: robot speedi, 6 links, 5 joints
Links:
- removed link ground
- added link map
Joints:
- joint cam_ground_height: parent ground -> map

Commit message: Imports CAD and sets up basic structure of car in URDF for Gazebo.

File: rr_description/speedi/speedi.urdf (robot description, URDF)
Before this commit: robot speedi, 6 links, 5 joints
Links:
- added link back_axle, mass 0.001
- added link steering_front_left, mass 0.001
- added link steering_front_right, mass 0.001
- added link wheel_back_left, mass 1.0; collision mesh filename=package://rr_description/meshes/wheel.dae; visual mesh filename=package://rr_description/meshes/wheel.dae
- added link wheel_back_right, mass 1.0; collision mesh filename=package://rr_description/meshes/wheel.dae; visual mesh filename=package://rr_description/meshes/wheel.dae
- added link wheel_front_left, mass 1.0; collision mesh filename=package://rr_description/meshes/wheel.dae; visual mesh filename=package://rr_description/meshes/wheel.dae
- added link wheel_front_right, mass 1.0; collision mesh filename=package://rr_description/meshes/wheel.dae; visual mesh filename=package://rr_description/meshes/wheel.dae
- link camera: geometry visual box size=0.1 0.1 0.1
- link camera_base: mass None -> 0.001
- link chassis: mass None -> 50.0; geometry collision mesh filename=package://rr_description/meshes/car.dae; visual mesh filename=package://rr_description/meshes/car.dae
- link imu: geometry visual box size=0.1 0.1 0.1
- link laser: geometry visual cylinder length=0.1 radius=0.05
- link map: mass None -> 0.001
Joints:
- added joint axle_to_left_wheel: type fixed, parent back_axle, child wheel_back_left, origin xyz=-0.14439 0 0 rpy=0 0 0
- added joint axle_to_right_wheel: type fixed, parent back_axle, child wheel_back_right, origin xyz=0.14439 0 0 rpy=0 0 0
- added joint chassis_to_back_axle: type continuous, parent chassis, child back_axle, origin xyz=0 0 0 rpy=0 0 0, axis 1 0 0
- added joint chassis_to_left_steering: type continuous, parent chassis, child steering_front_left, origin xyz=-0.14366 0.33246 0 rpy=0 0 0, axis 0 0 1
- added joint chassis_to_right_steering: type continuous, parent chassis, child steering_front_right, origin xyz=0.14366 0.33246 0 rpy=0 0 0, axis 0 0 1
- added joint left_steering_to_wheel: type continuous, parent steering_front_left, child wheel_front_left, origin xyz=0 0 0 rpy=0 0 0, axis 0 0 1
- added joint right_steering_to_wheel: type continuous, parent steering_front_right, child wheel_front_right, origin xyz=0 0 0 rpy=0 0 0, axis 0 0 1

Commit message: Adds velocity control to back axle of simulator. Also fixes a bunch of cmake errors across the projects.

File: rr_description/speedi/speedi.urdf (robot description, URDF)
Before this commit: robot speedi, 13 links, 12 joints
Links:
- link chassis: mass 50.0 -> 5.0
- link wheel_back_left: mass 1.0 -> 0.1
- link wheel_back_right: mass 1.0 -> 0.1
- link wheel_front_left: mass 1.0 -> 0.1
- link wheel_front_right: mass 1.0 -> 0.1
Joints:
- joint left_steering_to_wheel: axis 0 0 1 -> 1 0 0
- joint right_steering_to_wheel: axis 0 0 1 -> 1 0 0

Commit message: Fixes simulator steering. Changes rr_platform/steering messages to radians from degrees.

File: rr_description/speedi/speedi.urdf (robot description, URDF)
Before this commit: robot speedi, 13 links, 12 joints
Links:
- link laser: geometry 
Joints:
- joint axle_to_left_wheel: axis (none) -> 1 0 0; type fixed -> continuous
- joint axle_to_right_wheel: axis (none) -> 1 0 0; type fixed -> continuous
- joint chassis_to_back_axle: axis 1 0 0 -> (none); type continuous -> fixed
- joint chassis_to_left_steering: limit (none) -> lower=-0.366519 upper=0.366519 effort=100000.0 velocity=1000000.0; type continuous -> revolute
- joint chassis_to_right_steering: limit (none) -> lower=-0.366519 upper=0.366519 effort=100000.0 velocity=1000000.0; type continuous -> revolute
- joint lidar_joint: origin xyz=0 0.28575 0 rpy=0 0 0 -> xyz=0 0.255 0.110 rpy=0 0 1.5708

Commit message: Fixes convention breakage in URDF orientations and Gazebo camera setup. NOTE: This breaks the calibration-TF integration.

File: rr_description/speedi/speedi.urdf (robot description, URDF)
Before this commit: robot speedi, 13 links, 12 joints
Links:
- removed link camera
- removed link map
- added link base_footprint, mass 0.001
- added link camera_link, mass 0.001; visual box size=0.1 0.1 0.1
Joints:
- removed joint cam_ground_height
- added joint base_footprint_to_chassis: type fixed, parent base_footprint, child chassis, origin xyz=0 0 0.036 rpy=0 0 0
- joint axle_to_left_wheel: axis 1 0 0 -> 0 1 0; origin xyz=-0.14439 0 0 rpy=0 0 0 -> xyz=0 0.14439 0 rpy=0 0 0
- joint axle_to_right_wheel: axis 1 0 0 -> 0 1 0; origin xyz=0.14439 0 0 rpy=0 0 0 -> xyz=0 -0.14439 0 rpy=0 0 0
- joint cam_chassis_height: axis (none) -> 0 0 1; child chassis -> camera_base; limit (none) -> lower=0.274 upper=0.374 effort=1000.0 velocity=1000.0; origin xyz=0 0 0.3175 rpy=0 0 0 -> xyz=0 0 0 rpy=0 0 0; parent camera_base -> chassis; type fixed -> prismatic
- joint camera_tilt: child camera -> camera_link; limit effort=1000.0 velocity=1000.0 -> lower=0 upper=3.14 effort=1000.0 velocity=1000.0; origin (none) -> xyz=0 0 0 rpy=0 0 0; type continuous -> revolute
- joint chassis_to_left_steering: origin xyz=-0.14366 0.33246 0 rpy=0 0 0 -> xyz=0.33246 0.14366 0 rpy=0 0 0
- joint chassis_to_right_steering: limit lower=-0.366519 upper=0.366519 effort=100000.0 velocity=1000000.0 -> lower=-0.366519 upper=0.366519 effort=1000.0 velocity=1000.0; origin xyz=0.14366 0.33246 0 rpy=0 0 0 -> xyz=0.33246 -0.14366 0 rpy=0 0 0
- joint left_steering_to_wheel: axis 1 0 0 -> 0 1 0
- joint lidar_joint: origin xyz=0 0.255 0.110 rpy=0 0 1.5708 -> xyz=0.255 0 0.110 rpy=0 0 0
- joint right_steering_to_wheel: axis 1 0 0 -> 0 1 0
