Commit message: added imu and named things better

File: rr_description/urdf/speedi.urdf (robot description, URDF)
Before this commit: robot speedi, 4 links, 3 joints
Links:
- removed link base_link
- removed link usb_cam_center
- added link camera
- added link chassis
Joints:
- removed joint lidar
- removed joint usb_cam_center
- added joint camera_joint: type fixed, parent chassis, child camera, origin xyz=0 0 0.3175 rpy=0 0 0, axis 0 0 0
- added joint lidar_joint: type fixed, parent chassis, child lidar, origin xyz=0 0.28575 0 rpy=0 0 0, axis 0 0 0
- joint imu: parent base_link -> chassis

Commit message: sort-of tf publishing success
fixed issues with messages/CMake. robot_state_publisher occasionally fights my nodes by broadcasting over them. todo: make the camera joint prismatic and edit it through the joint state topic

File: rr_description/urdf/speedi.urdf (robot description, URDF)
Before this commit: robot speedi, 4 links, 3 joints
Joints:
- joint camera_joint: type fixed -> floating

Commit message: Last bit of cleanup before merging into master.

File: rr_description/urdf/speedi.urdf (robot description, URDF)
Before this commit: robot speedi, 13 links, 12 joints
Links:
- removed link camera_link
- added link camera, mass 0.001; visual box size=0.1 0.1 0.1
- added link camera_optical
Joints:
- added joint camera_optical_joint: type fixed, parent camera, child camera_optical, origin xyz=0 0 0 rpy=-1.5708 0 -1.5708
- joint camera_tilt: child camera_link -> camera

Commit message: Adds IARRC cone model to Gazebo simulation.

File: rr_description/urdf/speedi.urdf (robot description, URDF)
Before this commit: robot speedi, 14 links, 13 joints
Links:
- link camera: geometry 
- link imu: geometry 

Commit message: Updates speedi model to 2017 car design.

File: rr_description/urdf/speedi.urdf (robot description, URDF)
Before this commit: robot speedi, 14 links, 13 joints
Joints:
- joint cam_chassis_height: limit lower=0.274 upper=0.374 effort=1000.0 velocity=1000.0 -> lower=0.1 upper=0.375 effort=1000.0 velocity=1000.0; origin xyz=0 0 0 rpy=0 0 0 -> xyz=0.21793 0 0 rpy=0 0 0
- joint chassis_to_left_steering: origin xyz=0.33246 0.14366 0 rpy=0 0 0 -> xyz=0.34 0.14366 0 rpy=0 0 0
- joint chassis_to_right_steering: origin xyz=0.33246 -0.14366 0 rpy=0 0 0 -> xyz=0.34 -0.14366 0 rpy=0 0 0

Commit message: color detection fixes

File: rr_description/urdf/speedi.urdf (robot description, URDF)
Before this commit: robot speedi, 14 links, 13 joints
Joints:
- joint cam_chassis_height: limit lower=0.1 upper=0.375 effort=1000.0 velocity=1000.0 -> lower=0.1 upper=1.0 effort=1000.0 velocity=1000.0
