Commit message: bigolifies a few files

File: rr_description/urdf/bigoli.urdf (robot description, URDF)
Before this commit: robot bigoli, 14 links, 13 joints
Joints:
- joint axle_to_left_wheel: origin xyz=0 0.14439 0 rpy=0 0 0 -> xyz=0 0.33 0 rpy=0 0 0
- joint axle_to_right_wheel: origin xyz=0 -0.14439 0 rpy=0 0 0 -> xyz=0 -0.33 0 rpy=0 0 0
- joint base_footprint_to_chassis: origin xyz=0 0 0.036 rpy=0 0 0 -> xyz=0 0 0.125 rpy=0 0 0
- joint cam_chassis_height: origin xyz=0.21793 0 0.22 rpy=0 0 0 -> xyz=1.25 0 0.5825 rpy=0 0 0
- joint chassis_to_left_steering: origin xyz=0.34 0.14366 0 rpy=0 0 0 -> xyz=1.125 0.33 0 rpy=0 0 0
- joint chassis_to_right_steering: origin xyz=0.34 -0.14366 0 rpy=0 0 0 -> xyz=1.125 -0.33 0 rpy=0 0 0
- joint lidar_joint: origin xyz=0.275 0 0.110 rpy=0 0 0 -> xyz=1.142 0 0.110 rpy=0 0 0

Commit message: makes urdf work with realsense

File: rr_description/urdf/bigoli.urdf (robot description, URDF)
Before this commit: robot bigoli, 14 links, 13 joints
Links:
- added link camera_depth_optical_frame
Joints:
- added joint camera_depth_optical_joint: type fixed, parent camera_optical, child camera_depth_optical_frame, origin xyz=0 0 0 rpy=0 0 0

Commit message: gets lidar working and starts to correct planning parameters

File: rr_description/urdf/bigoli.urdf (robot description, URDF)
Before this commit: robot bigoli, 15 links, 14 joints
Joints:
- joint cam_chassis_height: origin xyz=1.25 0 0.5825 rpy=0 0 0 -> xyz=1.25 0 0.455 rpy=0 0 0
- joint camera_tilt: origin xyz=0 0 0 rpy=0 0 0 -> xyz=0 0 0 rpy=0 0.066 0

Commit message: Various changes to make Bigoli work (especially drive+steer relay nodes for latest firmware) (#104)
* untested serial code and tested joystick fixes

* corrects emulation of wireless gamepad in joystick driver test

* sets up ROS end of steering tester

(without breaking the one and only unit test this time)

* interacts with first working firmware

* refactors drive testing files in rr_platform

* added UDEV rules for mbed and arduino

* adds pid constants send over serial

* temporary changes, doesn't compile

* fixes logic errors for sending pid constants over serial

* remembers how c++ works (note: needs new udev rules)

* changes udev rules for multiple arduinos

* bigolifies a few files

* makes urdf work with realsense

* stuff to get front camera working

* gets lidar working and starts to correct planning parameters

* improves launch files, primarily fixes camera nodelet manager name for shitcam

File: rr_description/urdf/bigoli.urdf (robot description, URDF)
Before this commit: robot bigoli, 14 links, 13 joints
Links:
- added link camera_depth_optical_frame
Joints:
- added joint camera_depth_optical_joint: type fixed, parent camera_optical, child camera_depth_optical_frame, origin xyz=0 0 0 rpy=0 0 0
- joint axle_to_left_wheel: origin xyz=0 0.14439 0 rpy=0 0 0 -> xyz=0 0.33 0 rpy=0 0 0
- joint axle_to_right_wheel: origin xyz=0 -0.14439 0 rpy=0 0 0 -> xyz=0 -0.33 0 rpy=0 0 0
- joint base_footprint_to_chassis: origin xyz=0 0 0.036 rpy=0 0 0 -> xyz=0 0 0.125 rpy=0 0 0
- joint cam_chassis_height: origin xyz=0.21793 0 0.22 rpy=0 0 0 -> xyz=1.25 0 0.455 rpy=0 0 0
- joint camera_tilt: origin xyz=0 0 0 rpy=0 0 0 -> xyz=0 0 0 rpy=0 0.066 0
- joint chassis_to_left_steering: origin xyz=0.34 0.14366 0 rpy=0 0 0 -> xyz=1.125 0.33 0 rpy=0 0 0
- joint chassis_to_right_steering: origin xyz=0.34 -0.14366 0 rpy=0 0 0 -> xyz=1.125 -0.33 0 rpy=0 0 0
- joint lidar_joint: origin xyz=0.275 0 0.110 rpy=0 0 0 -> xyz=1.142 0 0.110 rpy=0 0 0
