Commit message: threw out mapper node, reversed lidar on sedani

File: rr_description/urdf/sedani.urdf (robot description, URDF)
Before this commit: robot macaroni, 23 links, 22 joints
Joints:
- joint lidar_joint: origin xyz=0.46 0 0.14 rpy=0 0 0 -> xyz=0.46 0 0.14 rpy=0 0 -3.1415

Commit message: WIP changes at end of 08/31/2018

File: rr_description/urdf/sedani.urdf (robot description, URDF)
Before this commit: robot macaroni, 23 links, 22 joints
Joints:
- joint lidar_joint: origin xyz=0.46 0 0.14 rpy=0 0 -3.1415 -> xyz=0.46 0 0.14 rpy=0 0 3.14159

Commit message: collects all pointcloud changes that have collected in iarrc-integration

File: rr_description/urdf/sedani.urdf (robot description, URDF)
Before this commit: robot macaroni, 22 links, 21 joints
Joints:
- joint camera_joint: origin xyz=0.28 0 0.267 rpy=0 0 0 -> xyz=0.28 0 0.08 rpy=0 -0.04 0

Commit message: good changes from Feb 24 testing day

File: rr_description/urdf/sedani.urdf (robot description, URDF)
Before this commit: robot macaroni, 22 links, 21 joints
Joints:
- joint base_footprint_to_chassis: origin xyz=0 0 0.036 rpy=0 0 0 -> xyz=0 0 0.079 rpy=0 0 0
- joint camera_joint: origin xyz=0.28 0 0.08 rpy=0 -0.04 0 -> xyz=0.28 0 0.1 rpy=0 -0.07 0

Commit message: fixes camera height, pitch direction, and projector point count

File: rr_description/urdf/sedani.urdf (robot description, URDF)
Before this commit: robot macaroni, 22 links, 21 joints
Joints:
- joint camera_joint: origin xyz=0.28 0 0.08 rpy=0 -0.04 0 -> xyz=0.28 0 0.18 rpy=0 -0.04 0

Commit message: adds extra cameras to sedani.urdf

File: rr_description/urdf/sedani.urdf (robot description, URDF)
Before this commit: robot macaroni, 22 links, 21 joints
Links:
- removed link camera
- removed link camera_optical
- removed link ultrasonic_0
- removed link ultrasonic_1
- removed link ultrasonic_2
- removed link ultrasonic_3
- removed link ultrasonic_4
- removed link ultrasonic_5
- removed link ultrasonic_6
- removed link ultrasonic_7
- removed link ultrasonic_array_base
- added link camera_center
- added link camera_center_optical
- added link camera_left
- added link camera_left_optical
- added link camera_right
- added link camera_right_optical
Joints:
- removed joint camera_joint
- removed joint camera_optical_joint
- removed joint ultrasonic_array_base
- removed joint ultrasonic_base_to_0
- removed joint ultrasonic_base_to_1
- removed joint ultrasonic_base_to_2
- removed joint ultrasonic_base_to_3
- removed joint ultrasonic_base_to_4
- removed joint ultrasonic_base_to_5
- removed joint ultrasonic_base_to_6
- removed joint ultrasonic_base_to_7
- added joint camera_center_joint: type fixed, parent base_footprint, child camera_center, origin xyz=0.28 0 0.256 rpy=0 0 0
- added joint camera_center_optical_joint: type fixed, parent camera_center, child camera_center_optical, origin xyz=0 0 0 rpy=-1.5708 0 -1.5708
- added joint camera_left_joint: type fixed, parent base_footprint, child camera_left, origin xyz=0.21 0.115 0.27 rpy=0 0.7854 1.5708
- added joint camera_left_optical_joint: type fixed, parent camera_left, child camera_left_optical, origin xyz=0 0 0 rpy=-1.5708 0 -1.5708
- added joint camera_right_joint: type fixed, parent base_footprint, child camera_right, origin xyz=0.21 -0.115 0.27 rpy=0 0.7854 -1.5708
- added joint camera_right_optical_joint: type fixed, parent camera_right, child camera_right_optical, origin xyz=0 0 0 rpy=-1.5708 0 -1.5708
- joint base_footprint_to_chassis: origin xyz=0 0 0.079 rpy=0 0 0 -> xyz=0 0 0.075 rpy=0 0 0

Commit message: changes from testing day

File: rr_description/urdf/sedani.urdf (robot description, URDF)
Before this commit: robot macaroni, 17 links, 16 joints
Joints:
- joint camera_center_joint: origin xyz=0.28 0 0.256 rpy=0 0 0 -> xyz=0.28 0 0.256 rpy=0 -0.03 0

Commit message: end of day 2, stuff mostly working

File: rr_description/urdf/sedani.urdf (robot description, URDF)
Before this commit: robot macaroni, 17 links, 16 joints
Joints:
- joint camera_center_joint: origin xyz=0.28 0 0.256 rpy=0 -0.03 0 -> xyz=0.28 0 0.256 rpy=0 0.02 0
