Commit message: got rid of actuating camera architecture

File: rr_description/urdf/macaroni.urdf (robot description, URDF)
Before this commit: robot macaroni, 14 links, 13 joints
Joints:
- joint cam_chassis_height: type prismatic -> fixed
- joint camera_tilt: type revolute -> fixed

Commit message: fixes problem where lidar was obstructed in gazebo

File: rr_description/urdf/macaroni.urdf (robot description, URDF)
Before this commit: robot macaroni, 14 links, 13 joints
Joints:
- joint lidar_joint: origin xyz=0.255 0 0.110 rpy=0 0 0 -> xyz=0.265 0 0.110 rpy=0 0 0

Commit message: cleaning more articulating camera stuff

File: rr_description/urdf/macaroni.urdf (robot description, URDF)
Before this commit: robot macaroni, 14 links, 13 joints
Joints:
- joint cam_chassis_height: axis 0 0 1 -> (none); limit lower=0.1 upper=1.0 effort=1000.0 velocity=1000.0 -> (none); origin xyz=0.21793 0 0 rpy=0 0 0 -> xyz=0.21793 0 0.22 rpy=0 0 0

Commit message: positions laser and car models more conveniently

File: rr_description/urdf/macaroni.urdf (robot description, URDF)
Before this commit: robot macaroni, 14 links, 13 joints
Joints:
- joint lidar_joint: origin xyz=0.265 0 0.110 rpy=0 0 0 -> xyz=0.275 0 0.110 rpy=0 0 0

Commit message: Added generic urdf profile for Ultrasonic Sensor Array of 8 sensors. Still needs to be measured in CAD.

File: rr_description/urdf/macaroni.urdf (robot description, URDF)
Before this commit: robot macaroni, 14 links, 13 joints
Links:
- added link ultrasonic_0, mass 0.001
- added link ultrasonic_1, mass 0.001
- added link ultrasonic_2, mass 0.001
- added link ultrasonic_3, mass 0.001
- added link ultrasonic_4, mass 0.001
- added link ultrasonic_5, mass 0.001
- added link ultrasonic_6, mass 0.001
- added link ultrasonic_7, mass 0.001
- added link ultrasonic_array_base, mass 0.001
Joints:
- added joint ultrasonic_array_base: type fixed, parent chassis, child ultrasonic_array_base, origin xyz=0 0 0.1778 rpy=0 0 0
- added joint ultrasonic_base_to_0: type fixed, parent ultrasonic_array_base, child ultrasonic_0, origin xyz=0 0 0.1778 rpy=0 0 0
- added joint ultrasonic_base_to_1: type fixed, parent ultrasonic_array_base, child ultrasonic_1, origin xyz=0 0 0.1778 rpy=0 0 0
- added joint ultrasonic_base_to_2: type fixed, parent ultrasonic_array_base, child ultrasonic_2, origin xyz=0 0 0.1778 rpy=0 0 0
- added joint ultrasonic_base_to_3: type fixed, parent ultrasonic_array_base, child ultrasonic_3, origin xyz=0 0 0.1778 rpy=0 0 0
- added joint ultrasonic_base_to_4: type fixed, parent ultrasonic_array_base, child ultrasonic_4, origin xyz=0 0 0.1778 rpy=0 0 0
- added joint ultrasonic_base_to_5: type fixed, parent ultrasonic_array_base, child ultrasonic_5, origin xyz=0 0 0.1778 rpy=0 0 0
- added joint ultrasonic_base_to_6: type fixed, parent ultrasonic_array_base, child ultrasonic_6, origin xyz=0 0 0.1778 rpy=0 0 0
- added joint ultrasonic_base_to_7: type fixed, parent ultrasonic_array_base, child ultrasonic_7, origin xyz=0 0 0.1778 rpy=0 0 0

Commit message: various changes to move towards a workable state

File: rr_description/urdf/macaroni.urdf (robot description, URDF)
Before this commit: robot macaroni, 23 links, 22 joints
Joints:
- joint ultrasonic_array_base: parent chassis -> base_footprint

Commit message: Update with (temp) ultrasonic values for testing 6 sensors

File: rr_description/urdf/macaroni.urdf (robot description, URDF)
Before this commit: robot macaroni, 23 links, 22 joints
Joints:
- joint ultrasonic_array_base: origin xyz=0 0 0.1778 rpy=0 0 0 -> xyz=0.21793 0 0.22 rpy=0 0 0; parent base_footprint -> chassis
- joint ultrasonic_base_to_0: origin xyz=0 0 0.1778 rpy=0 0 0 -> xyz=-0.045 0.108 0 rpy=0 0 1.57
- joint ultrasonic_base_to_1: origin xyz=0 0 0.1778 rpy=0 0 0 -> xyz=-0.021 0.07 0 rpy=0 0 0.349
- joint ultrasonic_base_to_2: origin xyz=0 0 0.1778 rpy=0 0 0 -> xyz=-0.011 0.027 0 rpy=0 0 0.296
- joint ultrasonic_base_to_3: origin xyz=0 0 0.1778 rpy=0 0 0 -> xyz=-0.011 -0.029 0 rpy=0 0 -0.175
- joint ultrasonic_base_to_4: origin xyz=0 0 0.1778 rpy=0 0 0 -> xyz=-0.024 -0.075 0 rpy=0 0 -0.349
- joint ultrasonic_base_to_5: origin xyz=0 0 0.1778 rpy=0 0 0 -> xyz=-0.045 -0.108 0 rpy=0 0 -1.57
- joint ultrasonic_base_to_6: origin xyz=0 0 0.1778 rpy=0 0 0 -> xyz=0 0 0 rpy=0 0 0
- joint ultrasonic_base_to_7: origin xyz=0 0 0.1778 rpy=0 0 0 -> xyz=0 0 0 rpy=0 0 0

Commit message: updates sedani urdf files and slightly simplifies resulting tf tree

File: rr_description/urdf/macaroni.urdf (robot description, URDF)
Before this commit: robot macaroni, 23 links, 22 joints
Links:
- removed link camera_base
Joints:
- removed joint cam_chassis_height
- removed joint camera_tilt
- added joint camera_joint: type fixed, parent chassis, child camera, origin xyz=0.21793 0 0.22 rpy=0 0 0

File: rr_description/urdf/sedani.urdf (robot description, URDF)
Before this commit: robot macaroni, 23 links, 22 joints
Links:
- removed link camera_base
Joints:
- removed joint cam_chassis_height
- removed joint camera_tilt
- added joint camera_joint: type fixed, parent chassis, child camera, origin xyz=0.28 0 0.267 rpy=0 0 0

Commit message: adds new iarrc cameras to gazebo; fixes keyboard_driver

File: rr_description/urdf/macaroni.urdf (robot description, URDF)
Before this commit: robot macaroni, 22 links, 21 joints
Links:
- removed link camera
- removed link camera_optical
- added link camera_center, mass 0.001
- added link camera_left, mass 0.001
- added link camera_optical_center
- added link camera_optical_left
- added link camera_optical_right
- added link camera_right, mass 0.001
Joints:
- removed joint camera_joint
- removed joint camera_optical_joint
- added joint camera_joint_center: type fixed, parent chassis, child camera_center, origin xyz=0.21793 0 0.22 rpy=0 0 0
- added joint camera_joint_left: type fixed, parent chassis, child camera_left, origin xyz=0.21793 0 0.22 rpy=0 0 0
- added joint camera_joint_right: type fixed, parent chassis, child camera_right, origin xyz=0.21793 0 0.22 rpy=0 0 0
- added joint camera_optical_joint_center: type fixed, parent camera_center, child camera_optical_center, origin xyz=0 0 0 rpy=-1.5708 0 -1.5708
- added joint camera_optical_joint_left: type fixed, parent camera_left, child camera_optical_left, origin xyz=0 0 0 rpy=-1.5708 0 -1.5708
- added joint camera_optical_joint_right: type fixed, parent camera_right, child camera_optical_right, origin xyz=0 0 0 rpy=-1.5708 0 -1.5708

Commit message: sets up EVGP urdf and gazebo control (+ deletes bigoli, + param asserts)

File: rr_description/urdf/macaroni.urdf (robot description, URDF)
Before this commit: robot macaroni, 26 links, 25 joints
Links:
- removed link ultrasonic_0
- removed link ultrasonic_1
- removed link ultrasonic_2
- removed link ultrasonic_3
- removed link ultrasonic_4
- removed link ultrasonic_5
- removed link ultrasonic_6
- removed link ultrasonic_7
- removed link ultrasonic_array_base
- link chassis: geometry collision mesh filename=package://rr_description/meshes/macaroni_car.dae; visual mesh filename=package://rr_description/meshes/macaroni_car.dae
- link wheel_back_left: geometry collision mesh filename=package://rr_description/meshes/macaroni_wheel.dae; visual mesh filename=package://rr_description/meshes/macaroni_wheel.dae
- link wheel_back_right: geometry collision mesh filename=package://rr_description/meshes/macaroni_wheel.dae; visual mesh filename=package://rr_description/meshes/macaroni_wheel.dae
- link wheel_front_left: geometry collision mesh filename=package://rr_description/meshes/macaroni_wheel.dae; visual mesh filename=package://rr_description/meshes/macaroni_wheel.dae
- link wheel_front_right: geometry collision mesh filename=package://rr_description/meshes/macaroni_wheel.dae; visual mesh filename=package://rr_description/meshes/macaroni_wheel.dae
Joints:
- removed joint ultrasonic_array_base
- removed joint ultrasonic_base_to_0
- removed joint ultrasonic_base_to_1
- removed joint ultrasonic_base_to_2
- removed joint ultrasonic_base_to_3
- removed joint ultrasonic_base_to_4
- removed joint ultrasonic_base_to_5
- removed joint ultrasonic_base_to_6
- removed joint ultrasonic_base_to_7

Commit message: fix PR issues

File: rr_description/urdf/macaroni.urdf (robot description, URDF)
Before this commit: robot macaroni, 17 links, 16 joints
Links:
- link wheel_back_left: geometry collision cylinder length=0.0445 radius=0.0524; visual mesh filename=package://rr_description/meshes/macaroni_wheel.dae
- link wheel_back_right: geometry collision cylinder length=0.0445 radius=0.0524; visual mesh filename=package://rr_description/meshes/macaroni_wheel.dae
- link wheel_front_left: geometry collision cylinder length=0.0445 radius=0.0524; visual mesh filename=package://rr_description/meshes/macaroni_wheel.dae
- link wheel_front_right: geometry collision cylinder length=0.0445 radius=0.0524; visual mesh filename=package://rr_description/meshes/macaroni_wheel.dae

Commit message: fix side cameras

File: rr_description/urdf/macaroni.urdf (robot description, URDF)
Before this commit: robot macaroni, 17 links, 16 joints
Joints:
- joint camera_joint_left: origin xyz=0.21793 0 0.22 rpy=0 0 0 -> xyz=0.21 0.115 0.27 rpy=0 0.7854 1.5708; parent chassis -> base_footprint
- joint camera_joint_right: origin xyz=0.21793 0 0.22 rpy=0 0 0 -> xyz=0.21 -0.115 0.27 rpy=0 0.7854 -1.5708; parent chassis -> base_footprint
