Commit message: Add a april tagged car to the rr_gazebo evgp_with_opponent.launch and fix positioning of april tag point tag

File: rr_description/urdf/rigatoni_april6.urdf.xacro (robot description, xacro)
@@ -1,3 +1,3 @@
-<robot name="rigatoni" xmlns:xacro="http://www.ros.org/wiki/xacro">
+<robot name="rigatoni6" xmlns:xacro="http://www.ros.org/wiki/xacro">
     <xacro:property name="use_gpu" value="false"/>
     <xacro:property name="props" value="${load_yaml('../conf/evgp_car_params.yaml')}"/>
@@ -31,7 +31,7 @@
                 <xacro:mesh_geometry/>
             </visual>
-<!--            <collision>-->
-<!--                <xacro:mesh_geometry/>-->
-<!--            </collision>-->
+            <!--            <collision>-->
+            <!--                <xacro:mesh_geometry/>-->
+            <!--            </collision>-->
         </link>
         <xacro:set_link_color link="body_visual_origin" color="${color}"/>
@@ -160,5 +160,5 @@
     </link>
     <gazebo reference="april">
-        <material>Apriltag0</material>
+        <material>Apriltag6</material>
     </gazebo>
     <!-- ************************** Joints *************************** -->
@@ -234,5 +234,5 @@
     <!-- ******************* Sensors *********************** -->
     <!-- Velodyne Puck VLP-16 -->
-    <xacro:VLP-16 parent="base_footprint" name="lidar" topic="/velodyne_points" hz="10" samples="500" gpu="true">
+    <xacro:VLP-16 parent="base_footprint" name="lidar" topic="/velodyne_points_april" hz="10" samples="500" gpu="true">
         <origin xyz="1.25 0 0.3" rpy="0 0 0" />
     </xacro:VLP-16>
@@ -262,7 +262,7 @@
                 <alwaysOn>true</alwaysOn>
                 <cameraName>camera</cameraName>
-                <imageTopicName>image_color_rect</imageTopicName>
-                <cameraInfoTopicName>camera_info</cameraInfoTopicName>
-                <frameName>camera_optical</frameName>
+                <imageTopicName>image_color_rect_april</imageTopicName>
+                <cameraInfoTopicName>camera_info_april</cameraInfoTopicName>
+                <frameName>camera_optical_april</frameName>
                 <distortionK1>0.0</distortionK1>
                 <distortionK2>0.0</distortionK2>
