Commit message: Tranformation in respect to tags on robot

File: rr_description/urdf/rigatoni.urdf (robot description, URDF)
Before this commit: robot rigatoni, 17 links, 16 joints
Links:
- removed link april
- added link 0_april, mass 0.0001; visual box size=0.001 0.3 0.3
- added link 1_april, mass 0.0001; visual box size=0.001 0.3 0.3
- added link 2_april, mass 0.0001; visual box size=0.001 0.3 0.3
- added link 3_april, mass 0.0001; visual box size=0.001 0.3 0.3
- added link 4_april, mass 0.0001; visual box size=0.001 0.3 0.3
- added link 5_april, mass 0.0001; visual box size=0.001 0.3 0.3
- added link 6_april, mass 0.0001; visual box size=0.001 0.3 0.3
- added link 7_april, mass 0.0001; visual box size=0.001 0.3 0.3
- added link white, mass 0.0001; visual box size=0.001 0.3 0.3
- added link white_back_left, mass 0.0001; visual box size=0.001 0.3 0.3
- added link white_back_right, mass 0.0001; visual box size=0.001 0.3 0.3
- added link white_front_left, mass 0.0001; visual box size=0.001 0.3 0.3
- added link white_front_mid, mass 0.0001; visual box size=0.001 0.3 0.3
- added link white_front_right, mass 0.0001; visual box size=0.001 0.3 0.3
- added link white_side_left, mass 0.0001; visual box size=0.001 0.3 0.3
- added link white_side_right, mass 0.0001; visual box size=0.001 0.3 0.3
Joints:
- removed joint base_footprint_to_april
- added joint base_footprint_to_0_april: type fixed, parent base_footprint, child 0_april, origin xyz=1.3256 0 0.51 rpy=0 0 0
- added joint base_footprint_to_1_april: type fixed, parent base_footprint, child 1_april, origin xyz=1.2414 -.3937 0.51 rpy=0 0 -0.7853981633974483
- added joint base_footprint_to_2_april: type fixed, parent base_footprint, child 2_april, origin xyz=.512 -.3937 0.51 rpy=0 0 -1.5707963267948966
- added joint base_footprint_to_3_april: type fixed, parent base_footprint, child 3_april, origin xyz=-.21581 -.3937 0.51 rpy=0 0 0.7853981633974483
- added joint base_footprint_to_4_april: type fixed, parent base_footprint, child 4_april, origin xyz=-.3 0 0.51 rpy=0 0 0
- added joint base_footprint_to_5_april: type fixed, parent base_footprint, child 5_april, origin xyz=-.21581 .3937 0.51 rpy=0 0 -0.7853981633974483
- added joint base_footprint_to_6_april: type fixed, parent base_footprint, child 6_april, origin xyz=.512 .45 0.51 rpy=0 0 -1.5707963267948966
- added joint base_footprint_to_7_april: type fixed, parent base_footprint, child 7_april, origin xyz=1.2414 .3937 0.51 rpy=0 0 0.7853981633974483
- added joint base_footprint_to_back_left_april_white: type fixed, parent base_footprint, child white_back_left, origin xyz=-.20581 .3837 0.51 rpy=0 0 -0.7853981633974483
- added joint base_footprint_to_back_mid_april_white: type fixed, parent base_footprint, child white, origin xyz=-.29 0 0.51 rpy=0 0 0
- added joint base_footprint_to_back_right_april_white: type fixed, parent base_footprint, child white_back_right, origin xyz=-.20581 -.3837 0.51 rpy=0 0 0.7853981633974483
- added joint base_footprint_to_front_left_april_white: type fixed, parent base_footprint, child white_front_left, origin xyz=1.2314 .3837 0.51 rpy=0 0 0.7853981633974483
- added joint base_footprint_to_front_mid_april_white: type fixed, parent base_footprint, child white_front_mid, origin xyz=1.3156 0 0.51 rpy=0 0 0
- added joint base_footprint_to_front_right_april_white: type fixed, parent base_footprint, child white_front_right, origin xyz=1.2314 -.3837 0.51 rpy=0 0 -0.7853981633974483
- added joint base_footprint_to_side_left_april_white: type fixed, parent base_footprint, child white_side_left, origin xyz=.512 .44 0.51 rpy=0 0 -1.5707963267948966
- added joint base_footprint_to_side_right_april_white: type fixed, parent base_footprint, child white_side_right, origin xyz=.512 -.3837 0.51 rpy=0 0 -1.5707963267948966

File: rr_description/urdf/rigatoni.urdf.xacro (robot description, xacro)
@@ -151,14 +151,170 @@
     </link>
     <xacro:set_link_color link="imu_bottom_link" color="Gold"/>
-    <link name='april'>
-        <xacro:null_inertia/>
-        <visual>
-            <geometry>
-                <box size="0.001 0.3 0.3 "/>
-            </geometry>
-        </visual>
-    </link>
-    <gazebo reference="april">
+    <link name="white">
+        <xacro:null_inertia/>
+        <visual>
+            <geometry>
+                <box size="0.001 0.3 0.3 "/>
+            </geometry>
+        </visual>
+    </link>
+    <gazebo reference="white">
+        <material>none</material>
+    </gazebo>
+    <link name="white_back_left">
+        <xacro:null_inertia/>
+        <visual>
+            <geometry>
+                <box size="0.001 0.3 0.3 "/>
+            </geometry>
+        </visual>
+    </link>
+    <gazebo reference="white_back_left">
+        <material>none</material>
+    </gazebo>
+    <link name="white_side_left">
+        <xacro:null_inertia/>
+        <visual>
+            <geometry>
+                <box size="0.001 0.3 0.3 "/>
+            </geometry>
+        </visual>
+    </link>
+    <gazebo reference="white_side_left">
+        <material>none</material>
+    </gazebo>
+    <link name="white_front_left">
+        <xacro:null_inertia/>
+        <visual>
+            <geometry>
+                <box size="0.001 0.3 0.3 "/>
+            </geometry>
+        </visual>
+    </link>
+    <gazebo reference="white_front_left">
+        <material>none</material>
+    </gazebo>
+    <link name="white_front_mid">
+        <xacro:null_inertia/>
+        <visual>
+            <geometry>
+                <box size="0.001 0.3 0.3 "/>
+            </geometry>
+        </visual>
+    </link>
+    <gazebo reference="white_front_mid">
+        <material>none</material>
+    </gazebo>
+    <link name="white_front_right">
+        <xacro:null_inertia/>
+        <visual>
+            <geometry>
+                <box size="0.001 0.3 0.3 "/>
+            </geometry>
+        </visual>
+    </link>
+    <link name="white_side_right">
+        <xacro:null_inertia/>
+        <visual>
+            <geometry>
+                <box size="0.001 0.3 0.3 "/>
+            </geometry>
+        </visual>
+    </link>
+    <link name="white_back_right">
+        <xacro:null_inertia/>
+        <visual>
+            <geometry>
+                <box size="0.001 0.3 0.3 "/>
+            </geometry>
+        </visual>
+    </link>
+    <link name="4_april">
+        <xacro:null_inertia/>
+        <visual>
+            <geometry>
+                <box size="0.001 0.3 0.3 "/>
+            </geometry>
+        </visual>
+    </link>
+    <gazebo reference="4_april">
+        <material>Apriltag4</material>
+    </gazebo>
+    <link name="5_april">
+        <xacro:null_inertia/>
+        <visual>
+            <geometry>
+                <box size="0.001 0.3 0.3 "/>
+            </geometry>
+        </visual>
+    </link>
+    <gazebo reference="5_april">
+        <material>Apriltag5</material>
+    </gazebo>
+    <link name="6_april">
+        <xacro:null_inertia/>
+        <visual>
+            <geometry>
+                <box size="0.001 0.3 0.3 "/>
+            </geometry>
+        </visual>
+    </link>
+    <gazebo reference="6_april">
+        <material>Apriltag6</material>
+    </gazebo>
+    <link name="7_april">
+        <xacro:null_inertia/>
+        <visual>
+            <geometry>
+                <box size="0.001 0.3 0.3 "/>
+            </geometry>
+        </visual>
+    </link>
+    <gazebo reference="7_april">
+        <material>Apriltag7</material>
+    </gazebo>
+    <link name="0_april">
+        <xacro:null_inertia/>
+        <visual>
+            <geometry>
+                <box size="0.001 0.3 0.3 "/>
+            </geometry>
+        </visual>
+    </link>
+    <gazebo reference="0_april">
         <material>Apriltag0</material>
+    </gazebo>
+    <link name="1_april">
+        <xacro:null_inertia/>
+        <visual>
+            <geometry>
+                <box size="0.001 0.3 0.3 "/>
+            </geometry>
+        </visual>
+    </link>
+    <gazebo reference="1_april">
+        <material>Apriltag1</material>
+    </gazebo>
+    <link name="2_april">
+        <xacro:null_inertia/>
+        <visual>
+            <geometry>
+                <box size="0.001 0.3 0.3 "/>
+            </geometry>
+        </visual>
+    </link>
+    <gazebo reference="2_april">
+        <material>Apriltag2</material>
+    </gazebo>
+    <link name="3_april">
+        <xacro:null_inertia/>
+        <visual>
+            <geometry>
+                <box size="0.001 0.3 0.3 "/>
+            </geometry>
+        </visual>
+    </link>
+    <gazebo reference="3_april">
+        <material>Apriltag3</material>
     </gazebo>
     <!-- ************************** Joints *************************** -->
@@ -227,8 +383,83 @@
         <origin xyz="0 0 0.21" rpy="0 0 0"/>
     </joint>
-    <joint name="base_footprint_to_april" type="fixed">
-        <parent link="base_footprint"/>
-        <child link="april"/>
+    <joint name="base_footprint_to_4_april" type="fixed">
+        <parent link="base_footprint"/>
+        <child link="4_april"/>
         <origin xyz="-.3 0 0.51" rpy="0 0 0"/>
+    </joint>
+    <joint name="base_footprint_to_back_mid_april_white" type="fixed">
+        <parent link="base_footprint"/>
+        <child link="white"/>
+        <origin xyz="-.29 0 0.51" rpy="0 0 0"/>
+    </joint>
+    <joint name="base_footprint_to_5_april" type="fixed">
+        <parent link="base_footprint"/>
+        <child link="5_april"/>
+        <origin xyz="-.21581 .3937 0.51" rpy="0 0 -${pi/4}"/>
+    </joint>
+    <joint name="base_footprint_to_back_left_april_white" type="fixed">
+        <parent link="base_footprint"/>
+        <child link="white_back_left"/>
+        <origin xyz="-.20581 .3837 0.51" rpy="0 0 -${pi/4}"/>
+    </joint>
+    <joint name="base_footprint_to_6_april" type="fixed">
+        <parent link="base_footprint"/>
+        <child link="6_april"/>
+        <origin xyz=".512 .45 0.51" rpy="0 0 -${pi/2}"/>
+    </joint>
+    <joint name="base_footprint_to_side_left_april_white" type="fixed">
+        <parent link="base_footprint"/>
+        <child link="white_side_left"/>
+        <origin xyz=".512 .44 0.51" rpy="0 0 -${pi/2}"/>
+    </joint>
+    <joint name="base_footprint_to_7_april" type="fixed">
+        <parent link="base_footprint"/>
+        <child link="7_april"/>
+        <origin xyz="1.2414 .3937 0.51" rpy="0 0 ${pi/4}"/>
+    </joint>
+    <joint name="base_footprint_to_front_left_april_white" type="fixed">
+        <parent link="base_footprint"/>
+        <child link="white_front_left"/>
+        <origin xyz="1.2314 .3837 0.51" rpy="0 0 ${pi/4}"/>
+    </joint>
+    <joint name="base_footprint_to_0_april" type="fixed">
+        <parent link="base_footprint"/>
+        <child link="0_april"/>
+        <origin xyz="1.3256 0 0.51" rpy="0 0 0"/>
+    </joint>
+    <joint name="base_footprint_to_front_mid_april_white" type="fixed">
+        <parent link="base_footprint"/>
+        <child link="white_front_mid"/>
+        <origin xyz="1.3156 0 0.51" rpy="0 0 0"/>
+    </joint>
+    <joint name="base_footprint_to_1_april" type="fixed">
+        <parent link="base_footprint"/>
+        <child link="1_april"/>
+        <origin xyz="1.2414 -.3937 0.51" rpy="0 0 -${pi/4}"/>
+    </joint>
+    <joint name="base_footprint_to_front_right_april_white" type="fixed">
+        <parent link="base_footprint"/>
+        <child link="white_front_right"/>
+        <origin xyz="1.2314 -.3837 0.51" rpy="0 0 -${pi/4}"/>
+    </joint>
+    <joint name="base_footprint_to_2_april" type="fixed">
+        <parent link="base_footprint"/>
+        <child link="2_april"/>
+        <origin xyz=".512 -.3937 0.51" rpy="0 0 -${pi/2}"/>
+    </joint>
+    <joint name="base_footprint_to_side_right_april_white" type="fixed">
+        <parent link="base_footprint"/>
+        <child link="white_side_right"/>
+        <origin xyz=".512 -.3837 0.51" rpy="0 0 -${pi/2}"/>
+    </joint>
+    <joint name="base_footprint_to_3_april" type="fixed">
+        <parent link="base_footprint"/>
+        <child link="3_april"/>
+        <origin xyz="-.21581 -.3937 0.51" rpy="0 0 ${pi/4}"/>
+    </joint>
+    <joint name="base_footprint_to_back_right_april_white" type="fixed">
+        <parent link="base_footprint"/>
+        <child link="white_back_right"/>
+        <origin xyz="-.20581 -.3837 0.51" rpy="0 0 ${pi/4}"/>
     </joint>
     <!-- ******************* Sensors *********************** -->

File: rr_description/urdf/rigatoni_opponent.urdf (robot description, URDF)
Before this commit: robot rigatoni_opponent, 32 links, 31 joints
Links:
- removed link back_left_april
- removed link back_mid_april
- removed link back_right_april
- removed link base_footprint
- removed link front_left_april
- removed link front_mid_april
- removed link front_right_april
- removed link side_left_april
- removed link side_right_april
- added link 0_april, mass 0.0001; visual box size=0.001 0.3 0.3
- added link 1_april, mass 0.0001; visual box size=0.001 0.3 0.3
- added link 2_april, mass 0.0001; visual box size=0.001 0.3 0.3
- added link 3_april, mass 0.0001; visual box size=0.001 0.3 0.3
- added link 4_april, mass 0.0001; visual box size=0.001 0.3 0.3
- added link 5_april, mass 0.0001; visual box size=0.001 0.3 0.3
- added link 6_april, mass 0.0001; visual box size=0.001 0.3 0.3
- added link 7_april, mass 0.0001; visual box size=0.001 0.3 0.3
- added link opponent_base_footprint, mass 0.0001
Joints:
- removed joint base_footprint_to_back_left_april
- removed joint base_footprint_to_back_left_april_white
- removed joint base_footprint_to_back_mid_april
- removed joint base_footprint_to_back_mid_april_white
- removed joint base_footprint_to_back_right_april
- removed joint base_footprint_to_back_right_april_white
- removed joint base_footprint_to_body_inertial_center
- removed joint base_footprint_to_camera
- removed joint base_footprint_to_front_left_april
- removed joint base_footprint_to_front_left_april_white
- removed joint base_footprint_to_front_mid_april
- removed joint base_footprint_to_front_mid_april_white
- removed joint base_footprint_to_front_right_april
- removed joint base_footprint_to_front_right_april_white
- removed joint base_footprint_to_gps
- removed joint base_footprint_to_imu
- removed joint base_footprint_to_imu2
- removed joint base_footprint_to_mesh_origin
- removed joint base_footprint_to_side_left_april
- removed joint base_footprint_to_side_left_april_white
- removed joint base_footprint_to_side_right_april
- removed joint base_footprint_to_side_right_april_white
- removed joint base_footprint_to_steering_link_left
- removed joint base_footprint_to_steering_link_right
- removed joint base_footprint_to_wheel_BL
- removed joint base_footprint_to_wheel_BR
- added joint opponent_base_footprint_to_0_april: type fixed, parent opponent_base_footprint, child 0_april, origin xyz=1.3256 0 0.51 rpy=0 0 0
- added joint opponent_base_footprint_to_1_april: type fixed, parent opponent_base_footprint, child 1_april, origin xyz=1.2414 -.3937 0.51 rpy=0 0 -0.7853981633974483
- added joint opponent_base_footprint_to_2_april: type fixed, parent opponent_base_footprint, child 2_april, origin xyz=.512 -.3937 0.51 rpy=0 0 -1.5707963267948966
- added joint opponent_base_footprint_to_3_april: type fixed, parent opponent_base_footprint, child 3_april, origin xyz=-.21581 -.3937 0.51 rpy=0 0 0.7853981633974483
- added joint opponent_base_footprint_to_4_april: type fixed, parent opponent_base_footprint, child 4_april, origin xyz=-.3 0 0.51 rpy=0 0 0
- added joint opponent_base_footprint_to_5_april: type fixed, parent opponent_base_footprint, child 5_april, origin xyz=-.21581 .3937 0.51 rpy=0 0 -0.7853981633974483
- added joint opponent_base_footprint_to_6_april: type fixed, parent opponent_base_footprint, child 6_april, origin xyz=.512 .45 0.51 rpy=0 0 -1.5707963267948966
- added joint opponent_base_footprint_to_7_april: type fixed, parent opponent_base_footprint, child 7_april, origin xyz=1.2414 .3937 0.51 rpy=0 0 0.7853981633974483
- added joint opponent_base_footprint_to_back_left_april_white: type fixed, parent opponent_base_footprint, child white_back_left, origin xyz=-.20581 .3837 0.51 rpy=0 0 -0.7853981633974483
- added joint opponent_base_footprint_to_back_mid_april_white: type fixed, parent opponent_base_footprint, child white, origin xyz=-.29 0 0.51 rpy=0 0 0
- added joint opponent_base_footprint_to_back_right_april_white: type fixed, parent opponent_base_footprint, child white_back_right, origin xyz=-.20581 -.3837 0.51 rpy=0 0 0.7853981633974483
- added joint opponent_base_footprint_to_body_inertial_center: type fixed, parent opponent_base_footprint, child body_inertial_center, origin xyz=0.4 0 0.1
- added joint opponent_base_footprint_to_camera: type fixed, parent opponent_base_footprint, child camera, origin xyz=0.68 0.4 0.8 rpy=0 0.2 0
- added joint opponent_base_footprint_to_front_left_april_white: type fixed, parent opponent_base_footprint, child white_front_left, origin xyz=1.2314 .3837 0.51 rpy=0 0 0.7853981633974483
- added joint opponent_base_footprint_to_front_mid_april_white: type fixed, parent opponent_base_footprint, child white_front_mid, origin xyz=1.3156 0 0.51 rpy=0 0 0
- added joint opponent_base_footprint_to_front_right_april_white: type fixed, parent opponent_base_footprint, child white_front_right, origin xyz=1.2314 -.3837 0.51 rpy=0 0 -0.7853981633974483
- added joint opponent_base_footprint_to_gps: type fixed, parent opponent_base_footprint, child gps_link, origin xyz=0.63 0.4 1.27 rpy=0 0 0
- added joint opponent_base_footprint_to_imu: type fixed, parent opponent_base_footprint, child imu_top_link, origin xyz=0.67 0.4 0.67 rpy=0 0 0
- added joint opponent_base_footprint_to_imu2: type fixed, parent opponent_base_footprint, child imu_bottom_link, origin xyz=0 0 0.21 rpy=0 0 0
- added joint opponent_base_footprint_to_mesh_origin: type fixed, parent opponent_base_footprint, child body_visual_origin, origin xyz=0.53 0 0 rpy=1.5707963267948966 0 1.5707963267948966
- added joint opponent_base_footprint_to_side_left_april_white: type fixed, parent opponent_base_footprint, child white_side_left, origin xyz=.512 .44 0.51 rpy=0 0 -1.5707963267948966
- added joint opponent_base_footprint_to_side_right_april_white: type fixed, parent opponent_base_footprint, child white_side_right, origin xyz=.512 -.3837 0.51 rpy=0 0 -1.5707963267948966
- added joint opponent_base_footprint_to_steering_link_left: type revolute, parent opponent_base_footprint, child steering_link_left, origin xyz=0.97 0.52 0.0625 rpy=0 0 0, axis 0 0 1, limit lower=-0.3 upper=0.3 effort=10000.0 velocity=2.0
- added joint opponent_base_footprint_to_steering_link_right: type revolute, parent opponent_base_footprint, child steering_link_right, origin xyz=0.97 -0.52 0.0625 rpy=0 0 0, axis 0 0 1, limit lower=-0.3 upper=0.3 effort=10000.0 velocity=2.0
- added joint opponent_base_footprint_to_wheel_BL: type continuous, parent opponent_base_footprint, child wheel_BL, origin xyz=0 0.52 0.0325 rpy=-1.5707963267948966 0 0, axis 0 0 1
- added joint opponent_base_footprint_to_wheel_BR: type continuous, parent opponent_base_footprint, child wheel_BR, origin xyz=0 -0.52 0.0325 rpy=-1.5707963267948966 0 0, axis 0 0 1
- joint lidar_base_mount_joint: parent base_footprint -> opponent_base_footprint
