Commit message: Tranformation in respect to tags on robot

File: rr_description/urdf/rigatoni_opponent.urdf.xacro (robot description, xacro)
@@ -23,5 +23,5 @@
     <xacro:macro name="evgp_body" params="collision_bitmask color">
         <!-- ************************** Links *************************** -->
-        <link name="base_footprint">
+        <link name="opponent_base_footprint">
             <xacro:null_inertia/>
         </link>
@@ -54,11 +54,11 @@
         <gazebo reference="body_inertial_center"/>
         <!-- ************************** Joints *************************** -->
-        <joint name="base_footprint_to_mesh_origin" type="fixed">
-            <parent link="base_footprint"/>
+        <joint name="opponent_base_footprint_to_mesh_origin" type="fixed">
+            <parent link="opponent_base_footprint"/>
             <child link="body_visual_origin"/>
             <origin xyz="0.53 0 0" rpy="${pi/2} 0 ${pi/2}"/>
         </joint>
-        <joint name="base_footprint_to_body_inertial_center" type="fixed">
-            <parent link="base_footprint"/>
+        <joint name="opponent_base_footprint_to_body_inertial_center" type="fixed">
+            <parent link="opponent_base_footprint"/>
             <child link="body_inertial_center"/>
             <origin xyz="${' '.join(str(x) for x in props['body_com'])}"/>
@@ -230,90 +230,90 @@
         </visual>
     </link>
-    <link name="back_mid_april">
-        <xacro:null_inertia/>
-        <visual>
-            <geometry>
-                <box size="0.001 0.3 0.3 "/>
-            </geometry>
-        </visual>
-    </link>
-    <gazebo reference="back_mid_april">
+    <link name="4_april">
+        <xacro:null_inertia/>
+        <visual>
+            <geometry>
+                <box size="0.001 0.3 0.3 "/>
+            </geometry>
+        </visual>
+    </link>
+    <gazebo reference="4_april">
         <material>Apriltag4</material>
     </gazebo>
-    <link name="back_left_april">
-        <xacro:null_inertia/>
-        <visual>
-            <geometry>
-                <box size="0.001 0.3 0.3 "/>
-            </geometry>
-        </visual>
-    </link>
-    <gazebo reference="back_left_april">
+    <link name="5_april">
+        <xacro:null_inertia/>
+        <visual>
+            <geometry>
+                <box size="0.001 0.3 0.3 "/>
+            </geometry>
+        </visual>
+    </link>
+    <gazebo reference="5_april">
         <material>Apriltag5</material>
     </gazebo>
-    <link name="side_left_april">
-        <xacro:null_inertia/>
-        <visual>
-            <geometry>
-                <box size="0.001 0.3 0.3 "/>
-            </geometry>
-        </visual>
-    </link>
-    <gazebo reference="side_left_april">
+    <link name="6_april">
+        <xacro:null_inertia/>
+        <visual>
+            <geometry>
+                <box size="0.001 0.3 0.3 "/>
+            </geometry>
+        </visual>
+    </link>
+    <gazebo reference="6_april">
         <material>Apriltag6</material>
     </gazebo>
-    <link name="front_left_april">
-        <xacro:null_inertia/>
-        <visual>
-            <geometry>
-                <box size="0.001 0.3 0.3 "/>
-            </geometry>
-        </visual>
-    </link>
-    <gazebo reference="front_left_april">
+    <link name="7_april">
+        <xacro:null_inertia/>
+        <visual>
+            <geometry>
+                <box size="0.001 0.3 0.3 "/>
+            </geometry>
+        </visual>
+    </link>
+    <gazebo reference="7_april">
         <material>Apriltag7</material>
     </gazebo>
-    <link name="front_mid_april">
-        <xacro:null_inertia/>
-        <visual>
-            <geometry>
-                <box size="0.001 0.3 0.3 "/>
-            </geometry>
-        </visual>
-    </link>
-    <gazebo reference="front_mid_april">
+    <link name="0_april">
+        <xacro:null_inertia/>
+        <visual>
+            <geometry>
+                <box size="0.001 0.3 0.3 "/>
+            </geometry>
+        </visual>
+    </link>
+    <gazebo reference="0_april">
         <material>Apriltag0</material>
     </gazebo>
-    <link name="front_right_april">
-        <xacro:null_inertia/>
-        <visual>
-            <geometry>
-                <box size="0.001 0.3 0.3 "/>
-            </geometry>
-        </visual>
-    </link>
-    <gazebo reference="front_right_april">
+    <link name="1_april">
+        <xacro:null_inertia/>
+        <visual>
+            <geometry>
+                <box size="0.001 0.3 0.3 "/>
+            </geometry>
+        </visual>
+    </link>
+    <gazebo reference="1_april">
         <material>Apriltag1</material>
     </gazebo>
-    <link name="side_right_april">
-        <xacro:null_inertia/>
-        <visual>
-            <geometry>
-                <box size="0.001 0.3 0.3 "/>
-            </geometry>
-        </visual>
-    </link>
-    <gazebo reference="side_right_april">
+    <link name="2_april">
+        <xacro:null_inertia/>
+        <visual>
+            <geometry>
+                <box size="0.001 0.3 0.3 "/>
+            </geometry>
+        </visual>
+    </link>
+    <gazebo reference="2_april">
         <material>Apriltag2</material>
     </gazebo>
-    <link name="back_right_april">
-        <xacro:null_inertia/>
-        <visual>
-            <geometry>
-                <box size="0.001 0.3 0.3 "/>
-            </geometry>
-        </visual>
-    </link>
-    <gazebo reference="back_right_april">
+    <link name="3_april">
+        <xacro:null_inertia/>
+        <visual>
+            <geometry>
+                <box size="0.001 0.3 0.3 "/>
+            </geometry>
+        </visual>
+    </link>
+    <gazebo reference="3_april">
         <material>Apriltag3</material>
     </gazebo>
@@ -321,11 +321,11 @@
     <xacro:property name="joint_flop_both" value="0.03"/>
     <xacro:macro name="back_wheel_joint" params="dest_link y">
-        <joint name="base_footprint_to_${dest_link}" type="continuous">
-            <parent link="base_footprint"/>
+        <joint name="opponent_base_footprint_to_${dest_link}" type="continuous">
+            <parent link="opponent_base_footprint"/>
             <child link="${dest_link}"/>
             <origin xyz="0 ${y} ${(props['wheel_radius_back'] / 2) - joint_flop_both}" rpy="${-pi/2} 0 0"/>
             <axis xyz="0 0 1"/>
         </joint>
-        <gazebo reference="base_footprint_to_${dest_link}"/>
+        <gazebo reference="opponent_base_footprint_to_${dest_link}"/>
     </xacro:macro>
     <xacro:back_wheel_joint dest_link="wheel_BL" y="${props['track'] / 2}"/>
@@ -333,6 +333,6 @@
     <xacro:property name="joint_flop_front" value="0.007"/>
     <xacro:macro name="steering_joints" params="steering_link wheel_link y">
-        <joint name="base_footprint_to_${steering_link}" type="revolute">
-            <parent link="base_footprint"/>
+        <joint name="opponent_base_footprint_to_${steering_link}" type="revolute">
+            <parent link="opponent_base_footprint"/>
             <child link="${steering_link}"/>
             <origin xyz="${props['wheelbase']} ${y} ${props['wheel_radius_front'] / 2}" rpy="0 0 0"/>
@@ -341,5 +341,5 @@
                    velocity="${props['steering_speed']}"/>
         </joint>
-        <gazebo reference="base_footprint_to_${steering_link}"/>
+        <gazebo reference="opponent_base_footprint_to_${steering_link}"/>
         <joint name="${steering_link}_to_${wheel_link}" type="continuous">
             <origin xyz="0 0 ${-joint_flop_both - joint_flop_front}" rpy="${pi/2} 0 0"/>
@@ -352,11 +352,11 @@
     <xacro:steering_joints steering_link="steering_link_left" wheel_link="wheel_FL" y="${props['track'] / 2}"/>
     <xacro:steering_joints steering_link="steering_link_right" wheel_link="wheel_FR" y="${-props['track'] / 2}"/>
-    <joint name="base_footprint_to_gps" type="fixed">
-        <parent link="base_footprint"/>
+    <joint name="opponent_base_footprint_to_gps" type="fixed">
+        <parent link="opponent_base_footprint"/>
         <child link="gps_link"/>
         <origin xyz="0.63 0.4 1.27" rpy="0 0 0"/>
     </joint>
-    <joint name="base_footprint_to_camera" type="fixed">
-        <parent link="base_footprint"/>
+    <joint name="opponent_base_footprint_to_camera" type="fixed">
+        <parent link="opponent_base_footprint"/>
         <child link="camera"/>
         <origin xyz="0.68 0.4 0.8" rpy="0 0.2 0"/>
@@ -373,91 +373,91 @@
     </xacro:macro>
     <xacro:camera_optical_frame camera_link="camera"/>
-    <joint name="base_footprint_to_imu" type="fixed">
-        <parent link="base_footprint"/>
+    <joint name="opponent_base_footprint_to_imu" type="fixed">
+        <parent link="opponent_base_footprint"/>
         <child link="imu_top_link"/>
         <origin xyz="0.67 0.4 0.67" rpy="0 0 0"/>
     </joint>
-    <joint name="base_footprint_to_imu2" type="fixed">
-        <parent link="base_footprint"/>
+    <joint name="opponent_base_footprint_to_imu2" type="fixed">
+        <parent link="opponent_base_footprint"/>
         <child link="imu_bottom_link"/>
         <origin xyz="0 0 0.21" rpy="0 0 0"/>
     </joint>
-    <joint name="base_footprint_to_back_mid_april" type="fixed">
-        <parent link="base_footprint"/>
-        <child link="back_mid_april"/>
+    <joint name="opponent_base_footprint_to_4_april" type="fixed">
+        <parent link="opponent_base_footprint"/>
+        <child link="4_april"/>
         <origin xyz="-.3 0 0.51" rpy="0 0 0"/>
     </joint>
-    <joint name="base_footprint_to_back_mid_april_white" type="fixed">
-        <parent link="base_footprint"/>
+    <joint name="opponent_base_footprint_to_back_mid_april_white" type="fixed">
+        <parent link="opponent_base_footprint"/>
         <child link="white"/>
         <origin xyz="-.29 0 0.51" rpy="0 0 0"/>
     </joint>
-    <joint name="base_footprint_to_back_left_april" type="fixed">
-        <parent link="base_footprint"/>
-        <child link="back_left_april"/>
+    <joint name="opponent_base_footprint_to_5_april" type="fixed">
+        <parent link="opponent_base_footprint"/>
+        <child link="5_april"/>
         <origin xyz="-.21581 .3937 0.51" rpy="0 0 -${pi/4}"/>
     </joint>
-    <joint name="base_footprint_to_back_left_april_white" type="fixed">
-        <parent link="base_footprint"/>
+    <joint name="opponent_base_footprint_to_back_left_april_white" type="fixed">
+        <parent link="opponent_base_footprint"/>
         <child link="white_back_left"/>
         <origin xyz="-.20581 .3837 0.51" rpy="0 0 -${pi/4}"/>
     </joint>
-    <joint name="base_footprint_to_side_left_april" type="fixed">
-        <parent link="base_footprint"/>
-        <child link="side_left_april"/>
+    <joint name="opponent_base_footprint_to_6_april" type="fixed">
+        <parent link="opponent_base_footprint"/>
+        <child link="6_april"/>
         <origin xyz=".512 .45 0.51" rpy="0 0 -${pi/2}"/>
     </joint>
-    <joint name="base_footprint_to_side_left_april_white" type="fixed">
-        <parent link="base_footprint"/>
+    <joint name="opponent_base_footprint_to_side_left_april_white" type="fixed">
+        <parent link="opponent_base_footprint"/>
         <child link="white_side_left"/>
         <origin xyz=".512 .44 0.51" rpy="0 0 -${pi/2}"/>
     </joint>
-    <joint name="base_footprint_to_front_left_april" type="fixed">
-        <parent link="base_footprint"/>
-        <child link="front_left_april"/>
+    <joint name="opponent_base_footprint_to_7_april" type="fixed">
+        <parent link="opponent_base_footprint"/>
+        <child link="7_april"/>
         <origin xyz="1.2414 .3937 0.51" rpy="0 0 ${pi/4}"/>
     </joint>
-    <joint name="base_footprint_to_front_left_april_white" type="fixed">
-        <parent link="base_footprint"/>
+    <joint name="opponent_base_footprint_to_front_left_april_white" type="fixed">
+        <parent link="opponent_base_footprint"/>
         <child link="white_front_left"/>
         <origin xyz="1.2314 .3837 0.51" rpy="0 0 ${pi/4}"/>
     </joint>
-    <joint name="base_footprint_to_front_mid_april" type="fixed">
-        <parent link="base_footprint"/>
-        <child link="front_mid_april"/>
+    <joint name="opponent_base_footprint_to_0_april" type="fixed">
+        <parent link="opponent_base_footprint"/>
+        <child link="0_april"/>
         <origin xyz="1.3256 0 0.51" rpy="0 0 0"/>
     </joint>
-    <joint name="base_footprint_to_front_mid_april_white" type="fixed">
-        <parent link="base_footprint"/>
+    <joint name="opponent_base_footprint_to_front_mid_april_white" type="fixed">
+        <parent link="opponent_base_footprint"/>
         <child link="white_front_mid"/>
         <origin xyz="1.3156 0 0.51" rpy="0 0 0"/>
     </joint>
-    <joint name="base_footprint_to_front_right_april" type="fixed">
-        <parent link="base_footprint"/>
-        <child link="front_right_april"/>
+    <joint name="opponent_base_footprint_to_1_april" type="fixed">
+        <parent link="opponent_base_footprint"/>
+        <child link="1_april"/>
         <origin xyz="1.2414 -.3937 0.51" rpy="0 0 -${pi/4}"/>
     </joint>
-    <joint name="base_footprint_to_front_right_april_white" type="fixed">
-        <parent link="base_footprint"/>
+    <joint name="opponent_base_footprint_to_front_right_april_white" type="fixed">
+        <parent link="opponent_base_footprint"/>
         <child link="white_front_right"/>
         <origin xyz="1.2314 -.3837 0.51" rpy="0 0 -${pi/4}"/>
     </joint>
-    <joint name="base_footprint_to_side_right_april" type="fixed">
-        <parent link="base_footprint"/>
-        <child link="side_right_april"/>
+    <joint name="opponent_base_footprint_to_2_april" type="fixed">
+        <parent link="opponent_base_footprint"/>
+        <child link="2_april"/>
         <origin xyz=".512 -.3937 0.51" rpy="0 0 -${pi/2}"/>
     </joint>
-    <joint name="base_footprint_to_side_right_april_white" type="fixed">
-        <parent link="base_footprint"/>
+    <joint name="opponent_base_footprint_to_side_right_april_white" type="fixed">
+        <parent link="opponent_base_footprint"/>
         <child link="white_side_right"/>
         <origin xyz=".512 -.3837 0.51" rpy="0 0 -${pi/2}"/>
     </joint>
-    <joint name="base_footprint_to_back_right_april" type="fixed">
-        <parent link="base_footprint"/>
-        <child link="back_right_april"/>
+    <joint name="opponent_base_footprint_to_3_april" type="fixed">
+        <parent link="opponent_base_footprint"/>
+        <child link="3_april"/>
         <origin xyz="-.21581 -.3937 0.51" rpy="0 0 ${pi/4}"/>
     </joint>
-    <joint name="base_footprint_to_back_right_april_white" type="fixed">
-        <parent link="base_footprint"/>
+    <joint name="opponent_base_footprint_to_back_right_april_white" type="fixed">
+        <parent link="opponent_base_footprint"/>
         <child link="white_back_right"/>
         <origin xyz="-.20581 -.3837 0.51" rpy="0 0 ${pi/4}"/>
@@ -465,5 +465,5 @@
     <!-- ******************* Sensors *********************** -->
     <!-- Velodyne Puck VLP-16 -->
-    <xacro:VLP-16 parent="base_footprint" name="lidar" topic="/velodyne_points_april" hz="10" samples="500" gpu="true">
+    <xacro:VLP-16 parent="opponent_base_footprint" name="lidar" topic="/velodyne_points_april" hz="10" samples="500" gpu="true">
         <origin xyz="1.25 0 0.3" rpy="0 0 0" />
     </xacro:VLP-16>
@@ -570,5 +570,5 @@
             <alwaysOn>true</alwaysOn>
             <updateRate>10.0</updateRate>
-            <bodyName>base_footprint</bodyName>
+            <bodyName>opponent_base_footprint</bodyName>
             <topicName>/odometry/ground_truth</topicName>
             <gaussianNoise>0.0</gaussianNoise>
@@ -596,5 +596,5 @@
     <transmission name="trans_back_right">
         <type>transmission_interface/SimpleTransmission</type>
-        <joint name="base_footprint_to_wheel_BR">
+        <joint name="opponent_base_footprint_to_wheel_BR">
             <hardwareInterface>hardware_interface/EffortJointInterface</hardwareInterface>
         </joint>
@@ -606,5 +606,5 @@
     <transmission name="left_steering_trans">
         <type>transmission_interface/SimpleTransmission</type>
-        <joint name="base_footprint_to_steering_link_left">
+        <joint name="opponent_base_footprint_to_steering_link_left">
             <hardwareInterface>hardware_interface/EffortJointInterface</hardwareInterface>
         </joint>
@@ -616,5 +616,5 @@
     <transmission name="right_steering_trans">
         <type>transmission_interface/SimpleTransmission</type>
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