Commit message: Change evgp opponent to a rigatoni opponent. Begin using tag bundles to detect opponent cars.

File: rr_description/urdf/rigatoni_opponent.urdf (robot description, URDF)
Before this commit: robot rigatoni, 17 links, 16 joints
Links:
- added link corner_april, mass 0.0001; visual box size=0.001 0.3 0.3
Joints:
- added joint base_footprint_to_corner_april: type fixed, parent base_footprint, child corner_april, origin xyz=-.3 .3 0.51 rpy=0 0 -0.7853981633974483

File: rr_description/urdf/rigatoni_opponent.urdf.xacro (robot description, xacro)
@@ -1,3 +1,3 @@
-<robot name="rigatoni6" xmlns:xacro="http://www.ros.org/wiki/xacro">
+<robot name="rigatoni_opponent" xmlns:xacro="http://www.ros.org/wiki/xacro">
     <xacro:property name="use_gpu" value="false"/>
     <xacro:property name="props" value="${load_yaml('../conf/evgp_car_params.yaml')}"/>
@@ -151,5 +151,5 @@
     </link>
     <xacro:set_link_color link="imu_bottom_link" color="Gold"/>
-    <link name='april'>
+    <link name="april">
         <xacro:null_inertia/>
         <visual>
@@ -161,4 +161,15 @@
     <gazebo reference="april">
         <material>Apriltag6</material>
+    </gazebo>
+    <link name="corner_april">
+        <xacro:null_inertia/>
+        <visual>
+            <geometry>
+                <box size="0.001 0.3 0.3 "/>
+            </geometry>
+        </visual>
+    </link>
+    <gazebo reference="corner_april">
+        <material>Apriltag0</material>
     </gazebo>
     <!-- ************************** Joints *************************** -->
@@ -231,4 +242,9 @@
         <child link="april"/>
         <origin xyz="-.3 0 0.51" rpy="0 0 0"/>
+    </joint>
+    <joint name="base_footprint_to_corner_april" type="fixed">
+        <parent link="base_footprint"/>
+        <child link="corner_april"/>
+        <origin xyz="-.3 .3 0.51" rpy="0 0 -${pi/4}"/>
     </joint>
     <!-- ******************* Sensors *********************** -->

Commit message: Add total of 8 preliminary tags to rigatoni opponent

File: rr_description/urdf/rigatoni_opponent.urdf (robot description, URDF)
Before this commit: robot rigatoni_opponent, 18 links, 17 joints
Links:
- removed link april
- removed link corner_april
- added link back_left_april, mass 0.0001; visual box size=0.001 0.3 0.3
- added link back_mid_april, mass 0.0001; visual box size=0.001 0.3 0.3
- added link back_right_april, mass 0.0001; visual box size=0.001 0.3 0.3
- added link front_left_april, mass 0.0001; visual box size=0.001 0.3 0.3
- added link front_mid_april, mass 0.0001; visual box size=0.001 0.3 0.3
- added link front_right_april, mass 0.0001; visual box size=0.001 0.3 0.3
- added link side_left_april, mass 0.0001; visual box size=0.001 0.3 0.3
- added link side_right_april, mass 0.0001; visual box size=0.001 0.3 0.3
Joints:
- removed joint base_footprint_to_april
- removed joint base_footprint_to_corner_april
- added joint base_footprint_to_back_left_april: type fixed, parent base_footprint, child back_left_april, origin xyz=-.3 .3 0.51 rpy=0 0 -0.7853981633974483
- added joint base_footprint_to_back_mid_april: type fixed, parent base_footprint, child back_mid_april, origin xyz=-.3 0 0.51 rpy=0 0 0
- added joint base_footprint_to_back_right_april: type fixed, parent base_footprint, child back_right_april, origin xyz=-.3 -.3 0.51 rpy=0 0 0.7853981633974483
- added joint base_footprint_to_front_left_april: type fixed, parent base_footprint, child front_left_april, origin xyz=1.5 .3 0.51 rpy=0 0 0.7853981633974483
- added joint base_footprint_to_front_mid_april: type fixed, parent base_footprint, child front_mid_april, origin xyz=1.5 0 0.51 rpy=0 0 0
- added joint base_footprint_to_front_right_april: type fixed, parent base_footprint, child front_right_april, origin xyz=1.5 0 0.51 rpy=0 0 -0.7853981633974483
- added joint base_footprint_to_side_left_april: type fixed, parent base_footprint, child side_left_april, origin xyz=.8 .3 0.51 rpy=0 0 -1.5707963267948966
- added joint base_footprint_to_side_right_april: type fixed, parent base_footprint, child side_right_april, origin xyz=.8 -.3 0.51 rpy=0 0 -1.5707963267948966

File: rr_description/urdf/rigatoni_opponent.urdf.xacro (robot description, xacro)
@@ -151,25 +151,91 @@
     </link>
     <xacro:set_link_color link="imu_bottom_link" color="Gold"/>
-    <link name="april">
-        <xacro:null_inertia/>
-        <visual>
-            <geometry>
-                <box size="0.001 0.3 0.3 "/>
-            </geometry>
-        </visual>
-    </link>
-    <gazebo reference="april">
+    <link name="back_mid_april">
+        <xacro:null_inertia/>
+        <visual>
+            <geometry>
+                <box size="0.001 0.3 0.3 "/>
+            </geometry>
+        </visual>
+    </link>
+    <gazebo reference="back_mid_april">
+        <material>Apriltag0</material>
+    </gazebo>
+    <link name="back_left_april">
+        <xacro:null_inertia/>
+        <visual>
+            <geometry>
+                <box size="0.001 0.3 0.3 "/>
+            </geometry>
+        </visual>
+    </link>
+    <gazebo reference="back_left_april">
+        <material>Apriltag1</material>
+    </gazebo>
+    <link name="side_left_april">
+        <xacro:null_inertia/>
+        <visual>
+            <geometry>
+                <box size="0.001 0.3 0.3 "/>
+            </geometry>
+        </visual>
+    </link>
+    <gazebo reference="side_left_april">
+        <material>Apriltag2</material>
+    </gazebo>
+    <link name="front_left_april">
+        <xacro:null_inertia/>
+        <visual>
+            <geometry>
+                <box size="0.001 0.3 0.3 "/>
+            </geometry>
+        </visual>
+    </link>
+    <gazebo reference="front_left_april">
+        <material>Apriltag3</material>
+    </gazebo>
+    <link name="front_mid_april">
+        <xacro:null_inertia/>
+        <visual>
+            <geometry>
+                <box size="0.001 0.3 0.3 "/>
+            </geometry>
+        </visual>
+    </link>
+    <gazebo reference="front_mid_april">
+        <material>Apriltag4</material>
+    </gazebo>
+    <link name="front_right_april">
+        <xacro:null_inertia/>
+        <visual>
+            <geometry>
+                <box size="0.001 0.3 0.3 "/>
+            </geometry>
+        </visual>
+    </link>
+    <gazebo reference="front_right_april">
+        <material>Apriltag5</material>
+    </gazebo>
+    <link name="side_right_april">
+        <xacro:null_inertia/>
+        <visual>
+            <geometry>
+                <box size="0.001 0.3 0.3 "/>
+            </geometry>
+        </visual>
+    </link>
+    <gazebo reference="side_right_april">
         <material>Apriltag6</material>
     </gazebo>
-    <link name="corner_april">
-        <xacro:null_inertia/>
-        <visual>
-            <geometry>
-                <box size="0.001 0.3 0.3 "/>
-            </geometry>
-        </visual>
-    </link>
-    <gazebo reference="corner_april">
-        <material>Apriltag0</material>
+    <link name="back_right_april">
+        <xacro:null_inertia/>
+        <visual>
+            <geometry>
+                <box size="0.001 0.3 0.3 "/>
+            </geometry>
+        </visual>
+    </link>
+    <gazebo reference="back_right_april">
+        <material>Apriltag7</material>
     </gazebo>
     <!-- ************************** Joints *************************** -->
@@ -238,13 +304,43 @@
         <origin xyz="0 0 0.21" rpy="0 0 0"/>
     </joint>
-    <joint name="base_footprint_to_april" type="fixed">
-        <parent link="base_footprint"/>
-        <child link="april"/>
+    <joint name="base_footprint_to_back_mid_april" type="fixed">
+        <parent link="base_footprint"/>
+        <child link="back_mid_april"/>
         <origin xyz="-.3 0 0.51" rpy="0 0 0"/>
     </joint>
-    <joint name="base_footprint_to_corner_april" type="fixed">
-        <parent link="base_footprint"/>
-        <child link="corner_april"/>
+    <joint name="base_footprint_to_back_left_april" type="fixed">
+        <parent link="base_footprint"/>
+        <child link="back_left_april"/>
         <origin xyz="-.3 .3 0.51" rpy="0 0 -${pi/4}"/>
+    </joint>
+    <joint name="base_footprint_to_side_left_april" type="fixed">
+        <parent link="base_footprint"/>
+        <child link="side_left_april"/>
+        <origin xyz=".8 .3 0.51" rpy="0 0 -${pi/2}"/>
+    </joint>
+    <joint name="base_footprint_to_front_left_april" type="fixed">
+        <parent link="base_footprint"/>
+        <child link="front_left_april"/>
+        <origin xyz="1.5 .3 0.51" rpy="0 0 ${pi/4}"/>
+    </joint>
+    <joint name="base_footprint_to_front_mid_april" type="fixed">
+        <parent link="base_footprint"/>
+        <child link="front_mid_april"/>
+        <origin xyz="1.5 0 0.51" rpy="0 0 0"/>
+    </joint>
+    <joint name="base_footprint_to_front_right_april" type="fixed">
+        <parent link="base_footprint"/>
+        <child link="front_right_april"/>
+        <origin xyz="1.5 -.3 0.51" rpy="0 0 -${pi/4}"/>
+    </joint>
+    <joint name="base_footprint_to_side_right_april" type="fixed">
+        <parent link="base_footprint"/>
+        <child link="side_right_april"/>
+        <origin xyz=".8 -.3 0.51" rpy="0 0 -${pi/2}"/>
+    </joint>
+    <joint name="base_footprint_to_back_right_april" type="fixed">
+        <parent link="base_footprint"/>
+        <child link="back_right_april"/>
+        <origin xyz="-.3 -.3 0.51" rpy="0 0 ${pi/4}"/>
     </joint>
     <!-- ******************* Sensors *********************** -->

Commit message: Placed april tags in correct locations and ids. Began adding them to the bundle

File: rr_description/urdf/rigatoni_opponent.urdf (robot description, URDF)
Before this commit: robot rigatoni_opponent, 24 links, 23 joints
Joints:
- joint base_footprint_to_back_left_april: origin xyz=-.3 .3 0.51 rpy=0 0 -0.7853981633974483 -> xyz=-.21581 .3937 0.51 rpy=0 0 -0.7853981633974483
- joint base_footprint_to_back_right_april: origin xyz=-.3 -.3 0.51 rpy=0 0 0.7853981633974483 -> xyz=-.21581 -.3937 0.51 rpy=0 0 0.7853981633974483
- joint base_footprint_to_front_left_april: origin xyz=1.5 .3 0.51 rpy=0 0 0.7853981633974483 -> xyz=1.2414 .3937 0.51 rpy=0 0 0.7853981633974483
- joint base_footprint_to_front_mid_april: origin xyz=1.5 0 0.51 rpy=0 0 0 -> xyz=1.3256 0 0.51 rpy=0 0 0
- joint base_footprint_to_front_right_april: origin xyz=1.5 0 0.51 rpy=0 0 -0.7853981633974483 -> xyz=1.2414 -.3937 0.51 rpy=0 0 -0.7853981633974483
- joint base_footprint_to_side_left_april: origin xyz=.8 .3 0.51 rpy=0 0 -1.5707963267948966 -> xyz=.512 .3937 0.51 rpy=0 0 -1.5707963267948966
- joint base_footprint_to_side_right_april: origin xyz=.8 -.3 0.51 rpy=0 0 -1.5707963267948966 -> xyz=.512 -.3937 0.51 rpy=0 0 -1.5707963267948966

File: rr_description/urdf/rigatoni_opponent.urdf.xacro (robot description, xacro)
@@ -160,82 +160,82 @@
     </link>
     <gazebo reference="back_mid_april">
+        <material>Apriltag4</material>
+    </gazebo>
+    <link name="back_left_april">
+        <xacro:null_inertia/>
+        <visual>
+            <geometry>
+                <box size="0.001 0.3 0.3 "/>
+            </geometry>
+        </visual>
+    </link>
+    <gazebo reference="back_left_april">
+        <material>Apriltag5</material>
+    </gazebo>
+    <link name="side_left_april">
+        <xacro:null_inertia/>
+        <visual>
+            <geometry>
+                <box size="0.001 0.3 0.3 "/>
+            </geometry>
+        </visual>
+    </link>
+    <gazebo reference="side_left_april">
+        <material>Apriltag6</material>
+    </gazebo>
+    <link name="front_left_april">
+        <xacro:null_inertia/>
+        <visual>
+            <geometry>
+                <box size="0.001 0.3 0.3 "/>
+            </geometry>
+        </visual>
+    </link>
+    <gazebo reference="front_left_april">
+        <material>Apriltag7</material>
+    </gazebo>
+    <link name="front_mid_april">
+        <xacro:null_inertia/>
+        <visual>
+            <geometry>
+                <box size="0.001 0.3 0.3 "/>
+            </geometry>
+        </visual>
+    </link>
+    <gazebo reference="front_mid_april">
         <material>Apriltag0</material>
     </gazebo>
-    <link name="back_left_april">
-        <xacro:null_inertia/>
-        <visual>
-            <geometry>
-                <box size="0.001 0.3 0.3 "/>
-            </geometry>
-        </visual>
-    </link>
-    <gazebo reference="back_left_april">
+    <link name="front_right_april">
+        <xacro:null_inertia/>
+        <visual>
+            <geometry>
+                <box size="0.001 0.3 0.3 "/>
+            </geometry>
+        </visual>
+    </link>
+    <gazebo reference="front_right_april">
         <material>Apriltag1</material>
     </gazebo>
-    <link name="side_left_april">
-        <xacro:null_inertia/>
-        <visual>
-            <geometry>
-                <box size="0.001 0.3 0.3 "/>
-            </geometry>
-        </visual>
-    </link>
-    <gazebo reference="side_left_april">
+    <link name="side_right_april">
+        <xacro:null_inertia/>
+        <visual>
+            <geometry>
+                <box size="0.001 0.3 0.3 "/>
+            </geometry>
+        </visual>
+    </link>
+    <gazebo reference="side_right_april">
         <material>Apriltag2</material>
     </gazebo>
-    <link name="front_left_april">
-        <xacro:null_inertia/>
-        <visual>
-            <geometry>
-                <box size="0.001 0.3 0.3 "/>
-            </geometry>
-        </visual>
-    </link>
-    <gazebo reference="front_left_april">
+    <link name="back_right_april">
+        <xacro:null_inertia/>
+        <visual>
+            <geometry>
+                <box size="0.001 0.3 0.3 "/>
+            </geometry>
+        </visual>
+    </link>
+    <gazebo reference="back_right_april">
         <material>Apriltag3</material>
-    </gazebo>
-    <link name="front_mid_april">
-        <xacro:null_inertia/>
-        <visual>
-            <geometry>
-                <box size="0.001 0.3 0.3 "/>
-            </geometry>
-        </visual>
-    </link>
-    <gazebo reference="front_mid_april">
-        <material>Apriltag4</material>
-    </gazebo>
-    <link name="front_right_april">
-        <xacro:null_inertia/>
-        <visual>
-            <geometry>
-                <box size="0.001 0.3 0.3 "/>
-            </geometry>
-        </visual>
-    </link>
-    <gazebo reference="front_right_april">
-        <material>Apriltag5</material>
-    </gazebo>
-    <link name="side_right_april">
-        <xacro:null_inertia/>
-        <visual>
-            <geometry>
-                <box size="0.001 0.3 0.3 "/>
-            </geometry>
-        </visual>
-    </link>
-    <gazebo reference="side_right_april">
-        <material>Apriltag6</material>
-    </gazebo>
-    <link name="back_right_april">
-        <xacro:null_inertia/>
-        <visual>
-            <geometry>
-                <box size="0.001 0.3 0.3 "/>
-            </geometry>
-        </visual>
-    </link>
-    <gazebo reference="back_right_april">
-        <material>Apriltag7</material>
     </gazebo>
     <!-- ************************** Joints *************************** -->
@@ -312,35 +312,35 @@
         <parent link="base_footprint"/>
         <child link="back_left_april"/>
-        <origin xyz="-.3 .3 0.51" rpy="0 0 -${pi/4}"/>
+        <origin xyz="-.21581 .3937 0.51" rpy="0 0 -${pi/4}"/>
     </joint>
     <joint name="base_footprint_to_side_left_april" type="fixed">
         <parent link="base_footprint"/>
         <child link="side_left_april"/>
-        <origin xyz=".8 .3 0.51" rpy="0 0 -${pi/2}"/>
+        <origin xyz=".512 .3937 0.51" rpy="0 0 -${pi/2}"/>
     </joint>
     <joint name="base_footprint_to_front_left_april" type="fixed">
         <parent link="base_footprint"/>
         <child link="front_left_april"/>
-        <origin xyz="1.5 .3 0.51" rpy="0 0 ${pi/4}"/>
+        <origin xyz="1.2414 .3937 0.51" rpy="0 0 ${pi/4}"/>
     </joint>
     <joint name="base_footprint_to_front_mid_april" type="fixed">
         <parent link="base_footprint"/>
         <child link="front_mid_april"/>
-        <origin xyz="1.5 0 0.51" rpy="0 0 0"/>
+        <origin xyz="1.3256 0 0.51" rpy="0 0 0"/>
     </joint>
     <joint name="base_footprint_to_front_right_april" type="fixed">
         <parent link="base_footprint"/>
         <child link="front_right_april"/>
-        <origin xyz="1.5 -.3 0.51" rpy="0 0 -${pi/4}"/>
+        <origin xyz="1.2414 -.3937 0.51" rpy="0 0 -${pi/4}"/>
     </joint>
     <joint name="base_footprint_to_side_right_april" type="fixed">
         <parent link="base_footprint"/>
         <child link="side_right_april"/>
-        <origin xyz=".8 -.3 0.51" rpy="0 0 -${pi/2}"/>
+        <origin xyz=".512 -.3937 0.51" rpy="0 0 -${pi/2}"/>
     </joint>
     <joint name="base_footprint_to_back_right_april" type="fixed">
         <parent link="base_footprint"/>
         <child link="back_right_april"/>
-        <origin xyz="-.3 -.3 0.51" rpy="0 0 ${pi/4}"/>
+        <origin xyz="-.21581 -.3937 0.51" rpy="0 0 ${pi/4}"/>
     </joint>
     <!-- ******************* Sensors *********************** -->

Commit message: Added back tags to the bundle.

File: rr_description/urdf/rigatoni_opponent.urdf (robot description, URDF)
Before this commit: robot rigatoni_opponent, 24 links, 23 joints
Joints:
- joint base_footprint_to_side_left_april: origin xyz=.512 .3937 0.51 rpy=0 0 -1.5707963267948966 -> xyz=.512 .45 0.51 rpy=0 0 -1.5707963267948966

File: rr_description/urdf/rigatoni_opponent.urdf.xacro (robot description, xacro)
@@ -317,5 +317,5 @@
         <parent link="base_footprint"/>
         <child link="side_left_april"/>
-        <origin xyz=".512 .3937 0.51" rpy="0 0 -${pi/2}"/>
+        <origin xyz=".512 .45 0.51" rpy="0 0 -${pi/2}"/>
     </joint>
     <joint name="base_footprint_to_front_left_april" type="fixed">
