Commit message: Before removing tags

File: rr_description/urdf/rigatoni_opponent.urdf (robot description, URDF)
Before this commit: robot rigatoni_opponent, 24 links, 23 joints
Links:
- added link white, mass 0.0001; visual box size=0.001 0.3 0.3
- added link white_back_left, mass 0.0001; visual box size=0.001 0.3 0.3
- added link white_back_right, mass 0.0001; visual box size=0.001 0.3 0.3
- added link white_front_left, mass 0.0001; visual box size=0.001 0.3 0.3
- added link white_front_mid, mass 0.0001; visual box size=0.001 0.3 0.3
- added link white_front_right, mass 0.0001; visual box size=0.001 0.3 0.3
- added link white_side_left, mass 0.0001; visual box size=0.001 0.3 0.3
- added link white_side_right, mass 0.0001; visual box size=0.001 0.3 0.3
Joints:
- added joint base_footprint_to_back_left_april_white: type fixed, parent base_footprint, child white_back_left, origin xyz=-.20581 .3837 0.51 rpy=0 0 -0.7853981633974483
- added joint base_footprint_to_back_mid_april_white: type fixed, parent base_footprint, child white, origin xyz=-.29 0 0.51 rpy=0 0 0
- added joint base_footprint_to_back_right_april_white: type fixed, parent base_footprint, child white_back_right, origin xyz=-.20581 -.3837 0.51 rpy=0 0 0.7853981633974483
- added joint base_footprint_to_front_left_april_white: type fixed, parent base_footprint, child white_front_left, origin xyz=1.2314 .3837 0.51 rpy=0 0 0.7853981633974483
- added joint base_footprint_to_front_mid_april_white: type fixed, parent base_footprint, child white_front_mid, origin xyz=1.3156 0 0.51 rpy=0 0 0
- added joint base_footprint_to_front_right_april_white: type fixed, parent base_footprint, child white_front_right, origin xyz=1.2314 -.3837 0.51 rpy=0 0 -0.7853981633974483
- added joint base_footprint_to_side_left_april_white: type fixed, parent base_footprint, child white_side_left, origin xyz=.512 .44 0.51 rpy=0 0 -1.5707963267948966
- added joint base_footprint_to_side_right_april_white: type fixed, parent base_footprint, child white_side_right, origin xyz=.512 -.3837 0.51 rpy=0 0 -1.5707963267948966

File: rr_description/urdf/rigatoni_opponent.urdf.xacro (robot description, xacro)
@@ -151,4 +151,83 @@
     </link>
     <xacro:set_link_color link="imu_bottom_link" color="Gold"/>
+    <link name="white">
+        <xacro:null_inertia/>
+        <visual>
+            <geometry>
+                <box size="0.001 0.3 0.3 "/>
+            </geometry>
+        </visual>
+    </link>
+    <gazebo reference="white">
+        <material>none</material>
+    </gazebo>
+    <link name="white_back_left">
+        <xacro:null_inertia/>
+        <visual>
+            <geometry>
+                <box size="0.001 0.3 0.3 "/>
+            </geometry>
+        </visual>
+    </link>
+    <gazebo reference="white_back_left">
+        <material>none</material>
+    </gazebo>
+    <link name="white_side_left">
+        <xacro:null_inertia/>
+        <visual>
+            <geometry>
+                <box size="0.001 0.3 0.3 "/>
+            </geometry>
+        </visual>
+    </link>
+    <gazebo reference="white_side_left">
+        <material>none</material>
+    </gazebo>
+    <link name="white_front_left">
+        <xacro:null_inertia/>
+        <visual>
+            <geometry>
+                <box size="0.001 0.3 0.3 "/>
+            </geometry>
+        </visual>
+    </link>
+    <gazebo reference="white_front_left">
+        <material>none</material>
+    </gazebo>
+    <link name="white_front_mid">
+        <xacro:null_inertia/>
+        <visual>
+            <geometry>
+                <box size="0.001 0.3 0.3 "/>
+            </geometry>
+        </visual>
+    </link>
+    <gazebo reference="white_front_mid">
+        <material>none</material>
+    </gazebo>
+    <link name="white_front_right">
+        <xacro:null_inertia/>
+        <visual>
+            <geometry>
+                <box size="0.001 0.3 0.3 "/>
+            </geometry>
+        </visual>
+    </link>
+    <link name="white_side_right">
+        <xacro:null_inertia/>
+        <visual>
+            <geometry>
+                <box size="0.001 0.3 0.3 "/>
+            </geometry>
+        </visual>
+    </link>
+    <link name="white_back_right">
+        <xacro:null_inertia/>
+        <visual>
+            <geometry>
+                <box size="0.001 0.3 0.3 "/>
+            </geometry>
+        </visual>
+    </link>
     <link name="back_mid_april">
         <xacro:null_inertia/>
@@ -309,4 +388,9 @@
         <origin xyz="-.3 0 0.51" rpy="0 0 0"/>
     </joint>
+    <joint name="base_footprint_to_back_mid_april_white" type="fixed">
+        <parent link="base_footprint"/>
+        <child link="white"/>
+        <origin xyz="-.29 0 0.51" rpy="0 0 0"/>
+    </joint>
     <joint name="base_footprint_to_back_left_april" type="fixed">
         <parent link="base_footprint"/>
@@ -314,4 +398,9 @@
         <origin xyz="-.21581 .3937 0.51" rpy="0 0 -${pi/4}"/>
     </joint>
+    <joint name="base_footprint_to_back_left_april_white" type="fixed">
+        <parent link="base_footprint"/>
+        <child link="white_back_left"/>
+        <origin xyz="-.20581 .3837 0.51" rpy="0 0 -${pi/4}"/>
+    </joint>
     <joint name="base_footprint_to_side_left_april" type="fixed">
         <parent link="base_footprint"/>
@@ -319,4 +408,9 @@
         <origin xyz=".512 .45 0.51" rpy="0 0 -${pi/2}"/>
     </joint>
+    <joint name="base_footprint_to_side_left_april_white" type="fixed">
+        <parent link="base_footprint"/>
+        <child link="white_side_left"/>
+        <origin xyz=".512 .44 0.51" rpy="0 0 -${pi/2}"/>
+    </joint>
     <joint name="base_footprint_to_front_left_april" type="fixed">
         <parent link="base_footprint"/>
@@ -324,4 +418,9 @@
         <origin xyz="1.2414 .3937 0.51" rpy="0 0 ${pi/4}"/>
     </joint>
+    <joint name="base_footprint_to_front_left_april_white" type="fixed">
+        <parent link="base_footprint"/>
+        <child link="white_front_left"/>
+        <origin xyz="1.2314 .3837 0.51" rpy="0 0 ${pi/4}"/>
+    </joint>
     <joint name="base_footprint_to_front_mid_april" type="fixed">
         <parent link="base_footprint"/>
@@ -329,4 +428,9 @@
         <origin xyz="1.3256 0 0.51" rpy="0 0 0"/>
     </joint>
+    <joint name="base_footprint_to_front_mid_april_white" type="fixed">
+        <parent link="base_footprint"/>
+        <child link="white_front_mid"/>
+        <origin xyz="1.3156 0 0.51" rpy="0 0 0"/>
+    </joint>
     <joint name="base_footprint_to_front_right_april" type="fixed">
         <parent link="base_footprint"/>
@@ -334,4 +438,9 @@
         <origin xyz="1.2414 -.3937 0.51" rpy="0 0 -${pi/4}"/>
     </joint>
+    <joint name="base_footprint_to_front_right_april_white" type="fixed">
+        <parent link="base_footprint"/>
+        <child link="white_front_right"/>
+        <origin xyz="1.2314 -.3837 0.51" rpy="0 0 -${pi/4}"/>
+    </joint>
     <joint name="base_footprint_to_side_right_april" type="fixed">
         <parent link="base_footprint"/>
@@ -339,8 +448,18 @@
         <origin xyz=".512 -.3937 0.51" rpy="0 0 -${pi/2}"/>
     </joint>
+    <joint name="base_footprint_to_side_right_april_white" type="fixed">
+        <parent link="base_footprint"/>
+        <child link="white_side_right"/>
+        <origin xyz=".512 -.3837 0.51" rpy="0 0 -${pi/2}"/>
+    </joint>
     <joint name="base_footprint_to_back_right_april" type="fixed">
         <parent link="base_footprint"/>
         <child link="back_right_april"/>
         <origin xyz="-.21581 -.3937 0.51" rpy="0 0 ${pi/4}"/>
+    </joint>
+    <joint name="base_footprint_to_back_right_april_white" type="fixed">
+        <parent link="base_footprint"/>
+        <child link="white_back_right"/>
+        <origin xyz="-.20581 -.3837 0.51" rpy="0 0 ${pi/4}"/>
     </joint>
     <!-- ******************* Sensors *********************** -->

Commit message: fix base_footprint guess

File: rr_description/urdf/rigatoni_opponent.urdf (robot description, URDF)
Before this commit: robot rigatoni_opponent, 32 links, 31 joints
Links:
- removed link lidar
- removed link lidar_base_link
Joints:
- removed joint lidar_base_mount_joint
- removed joint lidar_base_scan_joint

File: rr_description/urdf/rigatoni_opponent.urdf.xacro (robot description, xacro)
@@ -3,5 +3,4 @@
     <xacro:property name="props" value="${load_yaml('../conf/evgp_car_params.yaml')}"/>
     <xacro:property name="body_inertia" value="${props['body_inertia']}"/>
-    <xacro:include filename="$(find velodyne_description)/urdf/VLP-16.urdf.xacro"/>
     <!-- ************************** Links *************************** -->
     <xacro:macro name="null_inertia">
@@ -464,163 +463,3 @@
     </joint>
     <!-- ******************* Sensors *********************** -->
-    <!-- Velodyne Puck VLP-16 -->
-    <xacro:VLP-16 parent="opponent_base_footprint" name="lidar" topic="/velodyne_points_april" hz="10" samples="500" gpu="true">
-        <origin xyz="1.25 0 0.3" rpy="0 0 0" />
-    </xacro:VLP-16>
-    <!-- FLIR Blackfly + wide-angle lens -->
-    <gazebo reference="camera">
-        <sensor name="camera_sensor" type="camera">
-            <camera>
-                <horizontal_fov>1.6955</horizontal_fov>
-                <image>
-                    <width>1280</width>
-                    <height>964</height>
-                    <format>R8G8B8</format>
-                </image>
-                <clip>
-                    <near>0.05</near>
-                    <far>100</far>
-                </clip>
-                <noise>
-                    <type>gaussian</type>
-                    <mean>0.0</mean>
-                    <stddev>0.007</stddev>
-                </noise>
-            </camera>
-            <always_on>true</always_on>
-            <update_rate>15</update_rate>
-            <plugin name="camera_controller" filename="libgazebo_ros_camera.so">
-                <alwaysOn>true</alwaysOn>
-                <cameraName>camera</cameraName>
-                <imageTopicName>image_color_rect_april</imageTopicName>
-                <cameraInfoTopicName>camera_info_april</cameraInfoTopicName>
-                <frameName>camera_optical_april</frameName>
-                <distortionK1>0.0</distortionK1>
-                <distortionK2>0.0</distortionK2>
-                <distortionK3>0.0</distortionK3>
-                <distortionT1>0.0</distortionT1>
-                <distortionT2>0.0</distortionT2>
-            </plugin>
-        </sensor>
-    </gazebo>
-    <!-- IMU -->
-    <gazebo reference="imu_top_link">
-        <gravity>true</gravity>
-        <sensor name="imu_sensor" type="imu">
-            <always_on>true</always_on>
-            <update_rate>100</update_rate>
-            <visualize>true</visualize>
-            <topic>__default_topic__</topic>
-            <plugin filename="libgazebo_ros_imu_sensor.so" name="imu_plugin">
-                <topicName>imu</topicName>
-                <bodyName>imu_top_link</bodyName>
-                <updateRateHZ>20.0</updateRateHZ>
-                <gaussianNoise>0.005</gaussianNoise>
-                <xyzOffset>0 0 0</xyzOffset>
-                <rpyOffset>0 0 0</rpyOffset>
-                <frameName>imu_top_link</frameName>
-            </plugin>
-            <pose>0 0 0 0 0 0</pose>
-        </sensor>
-    </gazebo>
-    <!-- IMU -->
-    <gazebo reference="imu_bottom_link">
-        <gravity>true</gravity>
-        <sensor name="imu_sensor_bottom" type="imu">
-            <always_on>true</always_on>
-            <update_rate>100</update_rate>
-            <visualize>true</visualize>
-            <topic>__default_topic__</topic>
-            <plugin filename="libgazebo_ros_imu_sensor.so" name="imu_plugin">
-                <topicName>imu</topicName>
-                <bodyName>imu_bottom_link</bodyName>
-                <updateRateHZ>20.0</updateRateHZ>
-                <gaussianNoise>0.005</gaussianNoise>
-                <xyzOffset>0 0 0</xyzOffset>
-                <rpyOffset>0 0 0</rpyOffset>
-                <frameName>imu_bottom_link</frameName>
-            </plugin>
-            <pose>0 0 0 0 0 0</pose>
-        </sensor>
-    </gazebo>
-    <!-- GPS -->
-    <gazebo>
-        <plugin name="gps_controller" filename="libhector_gazebo_ros_gps.so">
-            <robotNamespace>/</robotNamespace>
-            <updateRate>10</updateRate>
-            <bodyName>gps_link</bodyName>
-            <frameId>gps_link</frameId>
-            <topicName>gps/fix</topicName>
-            <velocityTopicName>gps/vel</velocityTopicName>
-            <referenceLatitude>33.8</referenceLatitude>
-            <referenceLongitude>-84.4</referenceLongitude>
-            <referenceHeading>0</referenceHeading>
-            <referenceAltitude>0</referenceAltitude>
-            <drift>0.2 0.2 0.2</drift>
-            <driftFrequency>0.01 0.01 0.01</driftFrequency>
-            <gaussianNoise>0.05 0.05 0.05</gaussianNoise>
-            <velocityDrift>0.05 0.05 0.05</velocityDrift>
-            <velocityDriftFrequency>0.1 0.1 0.1</velocityDriftFrequency>
-            <velocityGaussianNoise>0.05 0.05 0.05</velocityGaussianNoise>
-        </plugin>
-    </gazebo>
-    <!-- ground-truth localization plugin -->
-    <gazebo>
-        <plugin name="ground_truth_tracker" filename="libgazebo_ros_p3d.so">
-            <alwaysOn>true</alwaysOn>
-            <updateRate>10.0</updateRate>
-            <bodyName>opponent_base_footprint</bodyName>
-            <topicName>/odometry/ground_truth</topicName>
-            <gaussianNoise>0.0</gaussianNoise>
-            <frameName>world</frameName>
-            <xyzOffsets>0 0 0</xyzOffsets>
-            <rpyOffsets>0 0 0</rpyOffsets>
-        </plugin>
-    </gazebo>
-    <!-- ****************** Actuators ********************** -->
-    <gazebo>
-        <plugin name="gazebo_ros_control" filename="libgazebo_ros_control.so">
-            <robotNamespace>/</robotNamespace>
-        </plugin>
-    </gazebo>
-    <transmission name="trans_back_left">
-        <type>transmission_interface/SimpleTransmission</type>
-        <joint name="base_footprint_to_wheel_BL">
-            <hardwareInterface>hardware_interface/EffortJointInterface</hardwareInterface>
-        </joint>
-        <actuator name="motor_left">
-            <hardwareInterface>hardware_interface/EffortJointInterface</hardwareInterface>
-            <mechanicalReduction>1</mechanicalReduction>
-        </actuator>
-    </transmission>
-    <transmission name="trans_back_right">
-        <type>transmission_interface/SimpleTransmission</type>
-        <joint name="opponent_base_footprint_to_wheel_BR">
-            <hardwareInterface>hardware_interface/EffortJointInterface</hardwareInterface>
-        </joint>
-        <actuator name="motor_right">
-            <hardwareInterface>hardware_interface/EffortJointInterface</hardwareInterface>
-            <mechanicalReduction>1</mechanicalReduction>
-        </actuator>
-    </transmission>
-    <transmission name="left_steering_trans">
-        <type>transmission_interface/SimpleTransmission</type>
-        <joint name="opponent_base_footprint_to_steering_link_left">
-            <hardwareInterface>hardware_interface/EffortJointInterface</hardwareInterface>
-        </joint>
-        <actuator name="left_steer_motor">
-            <hardwareInterface>hardware_interface/EffortJointInterface</hardwareInterface>
-            <mechanicalReduction>1</mechanicalReduction>
-        </actuator>
-    </transmission>
-    <transmission name="right_steering_trans">
-        <type>transmission_interface/SimpleTransmission</type>
-        <joint name="opponent_base_footprint_to_steering_link_right">
-            <hardwareInterface>hardware_interface/EffortJointInterface</hardwareInterface>
-        </joint>
-        <actuator name="right_steer_motor">
-            <hardwareInterface>hardware_interface/EffortJointInterface</hardwareInterface>
-            <mechanicalReduction>1</mechanicalReduction>
-        </actuator>
-    </transmission>
 </robot>
