Commit message: remove extra april tag scripts

File: rr_description/urdf/rigatoni_opponent.urdf.xacro (robot description, xacro)
@@ -238,5 +238,5 @@
     </link>
     <gazebo reference="4_april">
-        <material>Apriltag4</material>
+        <material>tag36_11_00004</material>
     </gazebo>
     <link name="5_april">
@@ -249,5 +249,5 @@
     </link>
     <gazebo reference="5_april">
-        <material>Apriltag5</material>
+        <material>tag36_11_00005</material>
     </gazebo>
     <link name="6_april">
@@ -260,5 +260,5 @@
     </link>
     <gazebo reference="6_april">
-        <material>Apriltag6</material>
+        <material>tag36_11_00006</material>
     </gazebo>
     <link name="7_april">
@@ -271,5 +271,5 @@
     </link>
     <gazebo reference="7_april">
-        <material>Apriltag7</material>
+        <material>tag36_11_00007</material>
     </gazebo>
     <link name="0_april">
@@ -282,5 +282,5 @@
     </link>
     <gazebo reference="0_april">
-        <material>Apriltag0</material>
+        <material>tag36_11_00000</material>
     </gazebo>
     <link name="1_april">
@@ -293,5 +293,5 @@
     </link>
     <gazebo reference="1_april">
-        <material>Apriltag1</material>
+        <material>tag36_11_00001</material>
     </gazebo>
     <link name="2_april">
@@ -304,5 +304,5 @@
     </link>
     <gazebo reference="2_april">
-        <material>Apriltag2</material>
+        <material>tag36_11_00002</material>
     </gazebo>
     <link name="3_april">
@@ -315,5 +315,5 @@
     </link>
     <gazebo reference="3_april">
-        <material>Apriltag3</material>
+        <material>tag36_11_00003</material>
     </gazebo>
     <!-- ************************** Joints *************************** -->
