Commit message: evgp tf and sensors

File: rr_description/urdf/evgp.urdf.xacro (robot description, xacro)
@@ -4,6 +4,6 @@
     <xacro:macro name="null_inertia">
         <inertial>
-            <mass value="0.001"/>
-            <inertia ixx="0.001" ixy="0" ixz="0" iyy="0.001" iyz="0" izz="0.001"/>
+            <mass value="0.0001"/>
+            <inertia ixx="0.0001" ixy="0" ixz="0" iyy="0.0001" iyz="0" izz="0.0001"/>
         </inertial>
     </xacro:macro>
@@ -69,9 +69,31 @@
         <xacro:null_inertia/>
     </link>
+    <link name="lidar">
+        <xacro:null_inertia/>
+        <visual>
+            <geometry>
+                <cylinder radius="0.1" length="0.1"/>
+            </geometry>
+        </visual>
+    </link>
+    <link name="camera_center">
+        <xacro:null_inertia/>
+        <visual>
+            <geometry>
+                <box size="0.05 0.05 0.05"/>
+            </geometry>
+        </visual>
+        <visual>
+            <origin rpy="0 ${pi/2} 0" xyz="0.05 0 0"/>
+            <geometry>
+                <cylinder radius="0.03" length="0.05"/>
+            </geometry>
+        </visual>
+    </link>
     <!-- ************************** Joints *************************** -->
     <joint name="base_footprint_to_mesh_origin" type="fixed">
         <parent link="base_footprint"/>
         <child link="body_visual_origin"/>
-        <origin xyz="1.45 0.508 -0.051"  rpy="${pi/2} 0 ${-pi/2}"/>
+        <origin xyz="1.45 0.515 -0.051"  rpy="${pi/2} 0 ${-pi/2}"/>
     </joint>
     <joint name="base_footprint_to_body_inertial_center" type="fixed">
@@ -112,4 +134,94 @@
     <xacro:steering_joints steering_link="steering_link_left" wheel_link="wheel_FL" y="${props['track'] / 2}"/>
     <xacro:steering_joints steering_link="steering_link_right" wheel_link="wheel_FR" y="${-props['track'] / 2}"/>
+    <joint name="base_footprint_to_lidar" type="fixed">
+        <parent link="base_footprint"/>
+        <child link="lidar"/>
+        <origin xyz="1.2 0 0.18" rpy="0 0 0"/>
+    </joint>
+    <joint name="base_footprint_to_camera_center" type="fixed">
+        <parent link="base_footprint"/>
+        <child link="camera_center"/>
+        <origin xyz="0.1 0 0.7" rpy="0 0.2 0"/>
+    </joint>
+    <xacro:macro name="camera_optical_frame" params="camera_link">
+        <link name="${camera_link}_optical">
+            <xacro:null_inertia/>
+        </link>
+        <joint name="${camera_link}_to_optical" type="fixed">
+            <parent link="${camera_link}"/>
+            <child link="${camera_link}_optical"/>
+            <origin xyz="0 0 0" rpy="${-pi/2} 0 ${-pi/2}"/>
+        </joint>
+    </xacro:macro>
+    <xacro:camera_optical_frame camera_link="camera_center"/>
+    <!-- ******************* Sensors *********************** -->
+    <!-- SICK TiM551 -->
+    <gazebo reference="lidar">
+        <sensor type="gpu_ray" name="lidar_sensor">
+            <pose>0 0 0 0 0 0</pose>
+            <visualize>true</visualize>
+            <update_rate>15</update_rate>
+            <ray>
+                <scan>
+                    <horizontal>
+                        <samples>270</samples>
+                        <resolution>1</resolution>  <!-- controls interpolation, leave at 1 -->
+                        <min_angle>${-pi*0.75}</min_angle>
+                        <max_angle>${pi*0.75}</max_angle>
+                    </horizontal>
+                </scan>
+                <range>
+                    <min>0.10</min>
+                    <max>8.0</max>
+                    <resolution>0.01</resolution>
+                </range>
+                <noise>
+                    <type>gaussian</type>
+                    <mean>0.0</mean>
+                    <stddev>0.02</stddev>
+                </noise>
+            </ray>
+            <plugin name="gazebo_ros_head_hokuyo_controller" filename="libgazebo_ros_gpu_laser.so">
+                <topicName>/scan</topicName>
+                <frameName>lidar</frameName>
+            </plugin>
+        </sensor>
+    </gazebo>
+    <!-- FLIR Blackfly + wide-angle lens -->
+    <gazebo reference="camera_center">
+        <sensor name="camera_sensor" type="camera">
+            <camera>
+                <horizontal_fov>1.6955</horizontal_fov>
+                <image>
+                    <width>1280</width>
+                    <height>964</height>
+                    <format>R8G8B8</format>
+                </image>
+                <clip>
+                    <near>0.05</near>
+                    <far>100</far>
+                </clip>
+                <noise>
+                    <type>gaussian</type>
+                    <mean>0.0</mean>
+                    <stddev>0.007</stddev>
+                </noise>
+            </camera>
+            <always_on>true</always_on>
+            <update_rate>15</update_rate>
+            <plugin name="camera_controller" filename="libgazebo_ros_camera.so">
+                <alwaysOn>true</alwaysOn>
+                <cameraName>camera_center</cameraName>
+                <imageTopicName>image_color_rect</imageTopicName>
+                <cameraInfoTopicName>camera_info</cameraInfoTopicName>
+                <frameName>camera_center_optical</frameName>
+                <distortionK1>0.0</distortionK1>
+                <distortionK2>0.0</distortionK2>
+                <distortionK3>0.0</distortionK3>
+                <distortionT1>0.0</distortionT1>
+                <distortionT2>0.0</distortionT2>
+            </plugin>
+        </sensor>
+    </gazebo>
     <!-- ****************** Actuators ********************** -->
     <gazebo>

Commit message: adds gps to simulator, tunes behavior in planner and physics conf

File: rr_description/urdf/evgp.urdf.xacro (robot description, xacro)
@@ -53,6 +53,6 @@
         </link>
         <gazebo reference="${name}">
-            <mu1>5.0</mu1>
-            <mu2>5.0</mu2>
+            <mu1>0.7</mu1>
+            <mu2>0.7</mu2>
             <kp>1000000</kp>
             <kd>1000000</kd>
@@ -77,4 +77,12 @@
         </visual>
     </link>
+    <link name="gps_link">
+        <xacro:null_inertia/>
+        <visual>
+            <geometry>
+                <box size="0.05 0.05 0.05"/>
+            </geometry>
+        </visual>
+    </link>
     <link name="camera_center">
         <xacro:null_inertia/>
@@ -95,5 +103,5 @@
         <parent link="base_footprint"/>
         <child link="body_visual_origin"/>
-        <origin xyz="1.45 0.515 -0.051"  rpy="${pi/2} 0 ${-pi/2}"/>
+        <origin xyz="1.45 0.515 -0.051" rpy="${pi/2} 0 ${-pi/2}"/>
     </joint>
     <joint name="base_footprint_to_body_inertial_center" type="fixed">
@@ -102,9 +110,10 @@
         <origin xyz="${' '.join(str(x) for x in props['body_com'])}"/>
     </joint>
+    <xacro:property name="joint_flop_distance" value="0.02"/>
     <xacro:macro name="back_wheel_joint" params="dest_link y">
         <joint name="base_footprint_to_${dest_link}" type="continuous">
             <parent link="base_footprint"/>
             <child link="${dest_link}"/>
-            <origin xyz="0 ${y} ${props['wheel_radius_back'] / 2}" rpy="${-pi/2} 0 0"/>
+            <origin xyz="0 ${y} ${(props['wheel_radius_back'] / 2) - joint_flop_distance}" rpy="${-pi/2} 0 0"/>
             <axis xyz="0 0 1"/>
             <dynamics damping="0.01"/>
@@ -125,5 +134,5 @@
         <gazebo reference="base_footprint_to_${steering_link}"/>
         <joint name="${steering_link}_to_${wheel_link}" type="continuous">
-            <origin xyz="0 0 0" rpy="${pi/2} 0 0"/>
+            <origin xyz="0 0 ${-joint_flop_distance}" rpy="${pi/2} 0 0"/>
             <parent link="${steering_link}"/>
             <child link="${wheel_link}"/>
@@ -138,4 +147,9 @@
         <child link="lidar"/>
         <origin xyz="1.2 0 0.18" rpy="0 0 0"/>
+    </joint>
+    <joint name="base_footprint_to_gps" type="fixed">
+        <parent link="base_footprint"/>
+        <child link="gps_link"/>
+        <origin xyz="0.5 0.5 0.1" rpy="0 0 0"/>
     </joint>
     <joint name="base_footprint_to_camera_center" type="fixed">
@@ -224,4 +238,25 @@
         </sensor>
     </gazebo>
+    <!-- GPS -->
+    <gazebo>
+        <plugin name="gps_controller" filename="libhector_gazebo_ros_gps.so">
+            <robotNamespace>/</robotNamespace>
+            <updateRate>10</updateRate>
+            <bodyName>gps_link</bodyName>
+            <frameId>gps_link</frameId>
+            <topicName>gps/fix</topicName>
+            <velocityTopicName>gps/vel</velocityTopicName>
+            <referenceLatitude>33.8</referenceLatitude>
+            <referenceLongitude>-84.4</referenceLongitude>
+            <referenceHeading>0</referenceHeading>
+            <referenceAltitude>0</referenceAltitude>
+            <drift>0.2 0.2 0.2</drift>
+            <driftFrequency>0.01 0.01 0.01</driftFrequency>
+            <gaussianNoise>0.05 0.05 0.05</gaussianNoise>
+            <velocityDrift>0.05 0.05 0.05</velocityDrift>
+            <velocityDriftFrequency>0.1 0.1 0.1</velocityDriftFrequency>
+            <velocityGaussianNoise>0.05 0.05 0.05</velocityGaussianNoise>
+        </plugin>
+    </gazebo>
     <!-- ****************** Actuators ********************** -->
     <gazebo>

Commit message: fixes car and track colors

File: rr_description/urdf/evgp.urdf.xacro (robot description, xacro)
@@ -13,4 +13,9 @@
         </geometry>
     </xacro:macro>
+    <xacro:macro name="set_link_color" params="link color">
+        <gazebo reference="${link}">
+            <material>Gazebo/${color}</material>
+        </gazebo>
+    </xacro:macro>
     <link name="base_footprint">
         <xacro:null_inertia/>
@@ -25,4 +30,5 @@
         </collision>
     </link>
+    <xacro:set_link_color link="body_visual_origin" color="Grey"/>
     <xacro:property name="body_inertia" value="${props['body_inertia']}"/>
     <link name="body_inertial_center">
@@ -58,4 +64,5 @@
             <kd>1000000</kd>
         </gazebo>
+        <xacro:set_link_color link="${name}" color="Black"/>
     </xacro:macro>
     <xacro:wheel_link name="wheel_BL" radius="${props['wheel_radius_back']}" width="${props['wheel_width_back']}"/>
@@ -77,4 +84,5 @@
         </visual>
     </link>
+    <xacro:set_link_color link="lidar" color="Gold"/>
     <link name="gps_link">
         <xacro:null_inertia/>
@@ -85,5 +93,6 @@
         </visual>
     </link>
-    <link name="camera_center">
+    <xacro:set_link_color link="gps_link" color="Gold"/>
+    <link name="camera">
         <xacro:null_inertia/>
         <visual>
@@ -99,4 +108,5 @@
         </visual>
     </link>
+    <xacro:set_link_color link="camera" color="Gold"/>
     <!-- ************************** Joints *************************** -->
     <joint name="base_footprint_to_mesh_origin" type="fixed">
@@ -153,7 +163,7 @@
         <origin xyz="0.5 0.5 0.1" rpy="0 0 0"/>
     </joint>
-    <joint name="base_footprint_to_camera_center" type="fixed">
-        <parent link="base_footprint"/>
-        <child link="camera_center"/>
+    <joint name="base_footprint_to_camera" type="fixed">
+        <parent link="base_footprint"/>
+        <child link="camera"/>
         <origin xyz="0.1 0 0.7" rpy="0 0.2 0"/>
     </joint>
@@ -168,5 +178,5 @@
         </joint>
     </xacro:macro>
-    <xacro:camera_optical_frame camera_link="camera_center"/>
+    <xacro:camera_optical_frame camera_link="camera"/>
     <!-- ******************* Sensors *********************** -->
     <!-- SICK TiM551 -->
@@ -203,5 +213,5 @@
     </gazebo>
     <!-- FLIR Blackfly + wide-angle lens -->
-    <gazebo reference="camera_center">
+    <gazebo reference="camera">
         <sensor name="camera_sensor" type="camera">
             <camera>
@@ -226,8 +236,8 @@
             <plugin name="camera_controller" filename="libgazebo_ros_camera.so">
                 <alwaysOn>true</alwaysOn>
-                <cameraName>camera_center</cameraName>
+                <cameraName>camera</cameraName>
                 <imageTopicName>image_color_rect</imageTopicName>
                 <cameraInfoTopicName>camera_info</cameraInfoTopicName>
-                <frameName>camera_center_optical</frameName>
+                <frameName>camera_optical</frameName>
                 <distortionK1>0.0</distortionK1>
                 <distortionK2>0.0</distortionK2>

Commit message: replaces sdf actor system with custom model controller

File: rr_description/urdf/evgp.urdf.xacro (robot description, xacro)
@@ -1,4 +1,5 @@
 <robot name="evgp" xmlns:xacro="http://www.ros.org/wiki/xacro">
     <xacro:property name="props" value="${load_yaml('../conf/evgp_car_params.yaml')}"/>
+    <xacro:include filename="evgp_body.sdf.xacro"/>
     <!-- ************************** Links *************************** -->
     <xacro:macro name="null_inertia">
@@ -18,26 +19,4 @@
         </gazebo>
     </xacro:macro>
-    <link name="base_footprint">
-        <xacro:null_inertia/>
-    </link>
-    <link name="body_visual_origin">
-        <xacro:null_inertia/>
-        <visual>
-            <xacro:mesh_geometry/>
-        </visual>
-        <collision>
-            <xacro:mesh_geometry/>
-        </collision>
-    </link>
-    <xacro:set_link_color link="body_visual_origin" color="Grey"/>
-    <xacro:property name="body_inertia" value="${props['body_inertia']}"/>
-    <link name="body_inertial_center">
-        <inertial>
-            <mass value="${props['body_mass']}"/>
-            <inertia ixx="${body_inertia[0]}" ixy="${body_inertia[1]}" ixz="${body_inertia[2]}"
-                     iyy="${body_inertia[3]}" iyz="${body_inertia[4]}" izz="${body_inertia[5]}"/>
-        </inertial>
-    </link>
-    <gazebo reference="body_inertial_center"/>
     <xacro:macro name="wheel_link" params="name radius width">
         <link name="${name}">
@@ -110,14 +89,4 @@
     <xacro:set_link_color link="camera" color="Gold"/>
     <!-- ************************** Joints *************************** -->
-    <joint name="base_footprint_to_mesh_origin" type="fixed">
-        <parent link="base_footprint"/>
-        <child link="body_visual_origin"/>
-        <origin xyz="1.45 0.515 -0.051" rpy="${pi/2} 0 ${-pi/2}"/>
-    </joint>
-    <joint name="base_footprint_to_body_inertial_center" type="fixed">
-        <parent link="base_footprint"/>
-        <child link="body_inertial_center"/>
-        <origin xyz="${' '.join(str(x) for x in props['body_com'])}"/>
-    </joint>
     <xacro:property name="joint_flop_distance" value="0.02"/>
     <xacro:macro name="back_wheel_joint" params="dest_link y">

Commit message: Added IMU and set up some files for localization

File: rr_description/urdf/evgp.urdf.xacro (robot description, xacro)
@@ -109,4 +109,13 @@
     </link>
     <xacro:set_link_color link="camera" color="Gold"/>
+    <link name="imu_link">
+        <xacro:null_inertia/>
+        <visual>
+            <geometry>
+                <box size="0.05 0.05 0.05"/>
+            </geometry>
+        </visual>
+    </link>
+    <xacro:set_link_color link="imu_link" color="Gold"/>
     <!-- ************************** Joints *************************** -->
     <joint name="base_footprint_to_mesh_origin" type="fixed">
@@ -179,8 +188,13 @@
     </xacro:macro>
     <xacro:camera_optical_frame camera_link="camera"/>
+    <joint name="base_footprint_to_imu" type="fixed">
+        <parent link="base_footprint"/>
+        <child link="imu_link"/>
+        <origin xyz="0.75 0.5 0.1" rpy="0 0 0"/>
+    </joint>
     <!-- ******************* Sensors *********************** -->
     <!-- SICK TiM551 -->
     <gazebo reference="lidar">
-        <sensor type="gpu_ray" name="lidar_sensor">
+        <sensor type="ray" name="lidar_sensor">
             <pose>0 0 0 0 0 0</pose>
             <visualize>false</visualize>
@@ -206,5 +220,5 @@
                 </noise>
             </ray>
-            <plugin name="gazebo_ros_head_hokuyo_controller" filename="libgazebo_ros_gpu_laser.so">
+            <plugin name="gazebo_ros_head_hokuyo_controller" filename="libgazebo_ros_laser.so">
                 <topicName>/scan</topicName>
                 <frameName>lidar</frameName>
@@ -248,4 +262,24 @@
         </sensor>
     </gazebo>
+    <!-- IMU -->
+    <gazebo reference="imu_link">
+        <gravity>true</gravity>
+        <sensor name="imu_sensor" type="imu">
+            <always_on>true</always_on>
+            <update_rate>100</update_rate>
+            <visualize>true</visualize>
+            <topic>__default_topic__</topic>
+            <plugin filename="libgazebo_ros_imu_sensor.so" name="imu_plugin">
+            <topicName>imu</topicName>
+            <bodyName>imu_link</bodyName>
+            <updateRateHZ>10.0</updateRateHZ>
+            <gaussianNoise>0.0</gaussianNoise>
+            <xyzOffset>0 0 0</xyzOffset>
+            <rpyOffset>0 0 0</rpyOffset>
+            <frameName>imu_link</frameName>
+            </plugin>
+            <pose>0 0 0 0 0 0</pose>
+        </sensor>
+    </gazebo>
     <!-- GPS -->
     <gazebo>

Commit message: addresses PR issues: collisions and start location

File: rr_description/urdf/evgp.urdf.xacro (robot description, xacro)
@@ -2,4 +2,5 @@
     <xacro:property name="props" value="${load_yaml('../conf/evgp_car_params.yaml')}"/>
     <xacro:include filename="evgp_body.urdf.xacro"/>
+    <xacro:evgp_body collide="true" color="Grey"/>
     <!-- ************************** Links *************************** -->
     <xacro:macro name="null_inertia">

File: rr_description/urdf/evgp_body.urdf.xacro (robot description, xacro)
@@ -1,5 +1,5 @@
 <robot name="evgp" xmlns:xacro="http://www.ros.org/wiki/xacro">
     <xacro:property name="props" value="${load_yaml('../conf/evgp_car_params.yaml')}"/>
-    <!-- ************************** Links *************************** -->
+    <xacro:property name="body_inertia" value="${props['body_inertia']}"/>
     <xacro:macro name="null_inertia">
         <inertial>
@@ -18,36 +18,41 @@
         </gazebo>
     </xacro:macro>
-    <link name="base_footprint">
-        <xacro:null_inertia/>
-    </link>
-    <link name="body_visual_origin">
-        <xacro:null_inertia/>
-        <visual>
-            <xacro:mesh_geometry/>
-        </visual>
-        <collision>
-            <xacro:mesh_geometry/>
-        </collision>
-    </link>
-    <xacro:set_link_color link="body_visual_origin" color="Grey"/>
-    <xacro:property name="body_inertia" value="${props['body_inertia']}"/>
-    <link name="body_inertial_center">
-        <inertial>
-            <mass value="${props['body_mass']}"/>
-            <inertia ixx="${body_inertia[0]}" ixy="${body_inertia[1]}" ixz="${body_inertia[2]}"
-                     iyy="${body_inertia[3]}" iyz="${body_inertia[4]}" izz="${body_inertia[5]}"/>
-        </inertial>
-    </link>
-    <gazebo reference="body_inertial_center"/>
-    <!-- ************************** Joints *************************** -->
-    <joint name="base_footprint_to_mesh_origin" type="fixed">
-        <parent link="base_footprint"/>
-        <child link="body_visual_origin"/>
-        <origin xyz="1.45 0.515 -0.051" rpy="${pi/2} 0 ${-pi/2}"/>
-    </joint>
-    <joint name="base_footprint_to_body_inertial_center" type="fixed">
-        <parent link="base_footprint"/>
-        <child link="body_inertial_center"/>
-        <origin xyz="${' '.join(str(x) for x in props['body_com'])}"/>
-    </joint>
+    <!-- leave 'name' empty for ego robot -->
+    <xacro:macro name="evgp_body" params="collide color">
+        <!-- ************************** Links *************************** -->
+        <link name="base_footprint">
+            <xacro:null_inertia/>
+        </link>
+        <link name="body_visual_origin">
+            <xacro:null_inertia/>
+            <visual>
+                <xacro:mesh_geometry/>
+            </visual>
+            <xacro:if value="${collide}">
+                <collision>
+                    <xacro:mesh_geometry/>
+                </collision>
+            </xacro:if>
+        </link>
+        <xacro:set_link_color link="body_visual_origin" color="${color}"/>
+        <link name="body_inertial_center">
+            <inertial>
+                <mass value="${props['body_mass']}"/>
+                <inertia ixx="${body_inertia[0]}" ixy="${body_inertia[1]}" ixz="${body_inertia[2]}"
+                         iyy="${body_inertia[3]}" iyz="${body_inertia[4]}" izz="${body_inertia[5]}"/>
+            </inertial>
+        </link>
+        <gazebo reference="body_inertial_center"/>
+        <!-- ************************** Joints *************************** -->
+        <joint name="base_footprint_to_mesh_origin" type="fixed">
+            <parent link="base_footprint"/>
+            <child link="body_visual_origin"/>
+            <origin xyz="1.45 0.515 -0.051" rpy="${pi/2} 0 ${-pi/2}"/>
+        </joint>
+        <joint name="base_footprint_to_body_inertial_center" type="fixed">
+            <parent link="base_footprint"/>
+            <child link="body_inertial_center"/>
+            <origin xyz="${' '.join(str(x) for x in props['body_com'])}"/>
+        </joint>
+    </xacro:macro>
 </robot>

File: rr_description/urdf/evgp_opponent.urdf.xacro (robot description, xacro)
@@ -1,4 +1,5 @@
 <robot name="evgp_opponent" xmlns:xacro="http://www.ros.org/wiki/xacro">
     <xacro:include filename="evgp_body.urdf.xacro"/>
+    <xacro:evgp_body collide="false" color="Blue"/>
     <gazebo reference="base_footprint">
         <kinematic>true</kinematic>
