Commit message: Evgp localization from sensors (#279)
* Sets up simulation IMU

* Sets up EKF with encoder, IMU, GPS odometry

* Sets up robot_localization estimate

File: rr_description/urdf/evgp.urdf.xacro (robot description, xacro)
@@ -109,4 +109,13 @@
     </link>
     <xacro:set_link_color link="camera" color="Gold"/>
+    <link name="imu_link">
+        <xacro:null_inertia/>
+        <visual>
+            <geometry>
+                <box size="0.05 0.05 0.05"/>
+            </geometry>
+        </visual>
+    </link>
+    <xacro:set_link_color link="imu_link" color="Gold"/>
     <!-- ************************** Joints *************************** -->
     <joint name="base_footprint_to_mesh_origin" type="fixed">
@@ -179,8 +188,13 @@
     </xacro:macro>
     <xacro:camera_optical_frame camera_link="camera"/>
+    <joint name="base_footprint_to_imu" type="fixed">
+        <parent link="base_footprint"/>
+        <child link="imu_link"/>
+        <origin xyz="0.75 0.5 0.1" rpy="0 0 0"/>
+    </joint>
     <!-- ******************* Sensors *********************** -->
     <!-- SICK TiM551 -->
     <gazebo reference="lidar">
-        <sensor type="gpu_ray" name="lidar_sensor">
+        <sensor type="ray" name="lidar_sensor">
             <pose>0 0 0 0 0 0</pose>
             <visualize>false</visualize>
@@ -206,5 +220,5 @@
                 </noise>
             </ray>
-            <plugin name="gazebo_ros_head_hokuyo_controller" filename="libgazebo_ros_gpu_laser.so">
+            <plugin name="gazebo_ros_head_hokuyo_controller" filename="libgazebo_ros_laser.so">
                 <topicName>/scan</topicName>
                 <frameName>lidar</frameName>
@@ -248,4 +262,24 @@
         </sensor>
     </gazebo>
+    <!-- IMU -->
+    <gazebo reference="imu_link">
+        <gravity>true</gravity>
+        <sensor name="imu_sensor" type="imu">
+            <always_on>true</always_on>
+            <update_rate>100</update_rate>
+            <visualize>true</visualize>
+            <topic>__default_topic__</topic>
+            <plugin filename="libgazebo_ros_imu_sensor.so" name="imu_plugin">
+                <topicName>imu</topicName>
+                <bodyName>imu_link</bodyName>
+                <updateRateHZ>20.0</updateRateHZ>
+                <gaussianNoise>0.005</gaussianNoise>
+                <xyzOffset>0 0 0</xyzOffset>
+                <rpyOffset>0 0 0</rpyOffset>
+                <frameName>imu_link</frameName>
+            </plugin>
+            <pose>0 0 0 0 0 0</pose>
+        </sensor>
+    </gazebo>
     <!-- GPS -->
     <gazebo>

Commit message: add switch for using gpu lidar plugin

File: rr_description/urdf/evgp.urdf.xacro (robot description, xacro)
@@ -1,3 +1,4 @@
 <robot name="evgp" xmlns:xacro="http://www.ros.org/wiki/xacro">
+    <xacro:property name="use_gpu" value="false"/>
     <xacro:property name="props" value="${load_yaml('../conf/evgp_car_params.yaml')}"/>
     <xacro:include filename="evgp_body.urdf.xacro"/>
@@ -165,6 +166,7 @@
     <!-- ******************* Sensors *********************** -->
     <!-- SICK TiM551 -->
+    <xacro:property name="gpu_string" value="${'gpu_' if use_gpu else ''}"/>
     <gazebo reference="lidar">
-        <sensor type="ray" name="lidar_sensor">
+        <sensor type="${gpu_string}ray" name="lidar_sensor">
             <pose>0 0 0 0 0 0</pose>
             <visualize>false</visualize>
@@ -190,5 +192,5 @@
                 </noise>
             </ray>
-            <plugin name="gazebo_ros_head_hokuyo_controller" filename="libgazebo_ros_laser.so">
+            <plugin name="laser_controller" filename="libgazebo_ros_${gpu_string}laser.so">
                 <topicName>/scan</topicName>
                 <frameName>lidar</frameName>

Commit message: cherry-pick 'add switch for using gpu lidar plugin'

File: rr_description/urdf/evgp.urdf.xacro (robot description, xacro)
@@ -1,3 +1,4 @@
 <robot name="evgp" xmlns:xacro="http://www.ros.org/wiki/xacro">
+    <xacro:property name="use_gpu" value="false"/>
     <xacro:property name="props" value="${load_yaml('../conf/evgp_car_params.yaml')}"/>
     <xacro:include filename="evgp_body.urdf.xacro"/>
@@ -151,6 +152,7 @@
     <!-- ******************* Sensors *********************** -->
     <!-- SICK TiM551 -->
+    <xacro:property name="gpu_string" value="${'gpu_' if use_gpu else ''}"/>
     <gazebo reference="lidar">
-        <sensor type="gpu_ray" name="lidar_sensor">
+        <sensor type="${gpu_string}ray" name="lidar_sensor">
             <pose>0 0 0 0 0 0</pose>
             <visualize>false</visualize>
@@ -176,5 +178,5 @@
                 </noise>
             </ray>
-            <plugin name="gazebo_ros_head_hokuyo_controller" filename="libgazebo_ros_gpu_laser.so">
+            <plugin name="laser_controller" filename="libgazebo_ros_${gpu_string}laser.so">
                 <topicName>/scan</topicName>
                 <frameName>lidar</frameName>

Commit message: fixes bug where non-gpu laser plugin could not see opponent car

File: rr_description/urdf/evgp.urdf.xacro (robot description, xacro)
@@ -2,5 +2,5 @@
     <xacro:property name="props" value="${load_yaml('../conf/evgp_car_params.yaml')}"/>
     <xacro:include filename="evgp_body.urdf.xacro"/>
-    <xacro:evgp_body collide="true" color="Grey"/>
+    <xacro:evgp_body collision_bitmask="0x1" color="Grey"/>
     <!-- ************************** Links *************************** -->
     <xacro:macro name="null_inertia">
@@ -43,4 +43,11 @@
             <kp>1000000</kp>
             <kd>1000000</kd>
+            <collision>
+                <surface>
+                    <contact>
+                        <collide_bitmask>0x1</collide_bitmask>
+                    </contact>
+                </surface>
+            </collision>
         </gazebo>
         <xacro:set_link_color link="${name}" color="Black"/>
@@ -165,6 +172,7 @@
     <!-- ******************* Sensors *********************** -->
     <!-- SICK TiM551 -->
+    <!-- note, gpu_ray and libgazebo_ros_gpu_laser.so must be used if opponent body has collisions disabled -->
     <gazebo reference="lidar">
-        <sensor type="ray" name="lidar_sensor">
+        <sensor type="gpu_ray" name="lidar_sensor">
             <pose>0 0 0 0 0 0</pose>
             <visualize>false</visualize>
@@ -190,5 +198,5 @@
                 </noise>
             </ray>
-            <plugin name="gazebo_ros_head_hokuyo_controller" filename="libgazebo_ros_laser.so">
+            <plugin name="gazebo_ros_head_hokuyo_controller" filename="libgazebo_ros_gpu_laser.so">
                 <topicName>/scan</topicName>
                 <frameName>lidar</frameName>
@@ -197,39 +205,39 @@
     </gazebo>
     <!-- FLIR Blackfly + wide-angle lens -->
-    <gazebo reference="camera">
-        <sensor name="camera_sensor" type="camera">
-            <camera>
-                <horizontal_fov>1.6955</horizontal_fov>
-                <image>
-                    <width>1280</width>
-                    <height>964</height>
-                    <format>R8G8B8</format>
-                </image>
-                <clip>
-                    <near>0.05</near>
-                    <far>100</far>
-                </clip>
-                <noise>
-                    <type>gaussian</type>
-                    <mean>0.0</mean>
-                    <stddev>0.007</stddev>
-                </noise>
-            </camera>
-            <always_on>true</always_on>
-            <update_rate>15</update_rate>
-            <plugin name="camera_controller" filename="libgazebo_ros_camera.so">
-                <alwaysOn>true</alwaysOn>
-                <cameraName>camera</cameraName>
-                <imageTopicName>image_color_rect</imageTopicName>
-                <cameraInfoTopicName>camera_info</cameraInfoTopicName>
-                <frameName>camera_optical</frameName>
-                <distortionK1>0.0</distortionK1>
-                <distortionK2>0.0</distortionK2>
-                <distortionK3>0.0</distortionK3>
-                <distortionT1>0.0</distortionT1>
-                <distortionT2>0.0</distortionT2>
-            </plugin>
-        </sensor>
-    </gazebo>
+<!--    <gazebo reference="camera">-->
+<!--        <sensor name="camera_sensor" type="camera">-->
+<!--            <camera>-->
+<!--                <horizontal_fov>1.6955</horizontal_fov>-->
+<!--                <image>-->
+<!--                    <width>1280</width>-->
+<!--                    <height>964</height>-->
+<!--                    <format>R8G8B8</format>-->
+<!--                </image>-->
+<!--                <clip>-->
+<!--                    <near>0.05</near>-->
+<!--                    <far>100</far>-->
+<!--                </clip>-->
+<!--                <noise>-->
+<!--                    <type>gaussian</type>-->
+<!--                    <mean>0.0</mean>-->
+<!--                    <stddev>0.007</stddev>-->
+<!--                </noise>-->
+<!--            </camera>-->
+<!--            <always_on>true</always_on>-->
+<!--            <update_rate>15</update_rate>-->
+<!--            <plugin name="camera_controller" filename="libgazebo_ros_camera.so">-->
+<!--                <alwaysOn>true</alwaysOn>-->
+<!--                <cameraName>camera</cameraName>-->
+<!--                <imageTopicName>image_color_rect</imageTopicName>-->
+<!--                <cameraInfoTopicName>camera_info</cameraInfoTopicName>-->
+<!--                <frameName>camera_optical</frameName>-->
+<!--                <distortionK1>0.0</distortionK1>-->
+<!--                <distortionK2>0.0</distortionK2>-->
+<!--                <distortionK3>0.0</distortionK3>-->
+<!--                <distortionT1>0.0</distortionT1>-->
+<!--                <distortionT2>0.0</distortionT2>-->
+<!--            </plugin>-->
+<!--        </sensor>-->
+<!--    </gazebo>-->
     <!-- IMU -->
     <gazebo reference="imu_link">
@@ -274,16 +282,16 @@
     </gazebo>
     <!-- ground-truth localization plugin -->
-    <gazebo>
-        <plugin name="ground_truth_tracker" filename="libgazebo_ros_p3d.so">
-            <alwaysOn>true</alwaysOn>
-            <updateRate>50.0</updateRate>
-            <bodyName>base_footprint</bodyName>
-            <topicName>/odometry/ground_truth</topicName>
-            <gaussianNoise>0.0</gaussianNoise>
-            <frameName>world</frameName>
-            <xyzOffsets>0 0 0</xyzOffsets>
-            <rpyOffsets>0 0 0</rpyOffsets>
-        </plugin>
-    </gazebo>
+<!--    <gazebo>-->
+<!--        <plugin name="ground_truth_tracker" filename="libgazebo_ros_p3d.so">-->
+<!--            <alwaysOn>true</alwaysOn>-->
+<!--            <updateRate>10.0</updateRate>-->
+<!--            <bodyName>base_footprint</bodyName>-->
+<!--            <topicName>/odometry/ground_truth</topicName>-->
+<!--            <gaussianNoise>0.0</gaussianNoise>-->
+<!--            <frameName>world</frameName>-->
+<!--            <xyzOffsets>0 0 0</xyzOffsets>-->
+<!--            <rpyOffsets>0 0 0</rpyOffsets>-->
+<!--        </plugin>-->
+<!--    </gazebo>-->
     <!-- ****************** Actuators ********************** -->
     <gazebo>

File: rr_description/urdf/evgp_body.urdf.xacro (robot description, xacro)
@@ -18,6 +18,5 @@
         </gazebo>
     </xacro:macro>
-    <!-- leave 'name' empty for ego robot -->
-    <xacro:macro name="evgp_body" params="collide color">
+    <xacro:macro name="evgp_body" params="collision_bitmask color">
         <!-- ************************** Links *************************** -->
         <link name="base_footprint">
@@ -29,11 +28,18 @@
                 <xacro:mesh_geometry/>
             </visual>
-            <xacro:if value="${collide}">
-                <collision>
-                    <xacro:mesh_geometry/>
-                </collision>
-            </xacro:if>
+            <collision>
+                <xacro:mesh_geometry/>
+            </collision>
         </link>
         <xacro:set_link_color link="body_visual_origin" color="${color}"/>
+        <gazebo reference="body_visual_origin">
+            <collision>
+                <surface>
+                    <contact>
+                        <collide_bitmask>${collision_bitmask}</collide_bitmask>
+                    </contact>
+                </surface>
+            </collision>
+        </gazebo>
         <link name="body_inertial_center">
             <inertial>

File: rr_description/urdf/evgp_opponent.urdf.xacro (robot description, xacro)
@@ -1,5 +1,5 @@
 <robot name="evgp_opponent" xmlns:xacro="http://www.ros.org/wiki/xacro">
     <xacro:include filename="evgp_body.urdf.xacro"/>
-    <xacro:evgp_body collide="false" color="Blue"/>
+    <xacro:evgp_body collision_bitmask="0x2" color="Blue"/>
     <gazebo reference="base_footprint">
         <kinematic>true</kinematic>

Commit message: cherry-pick 'fixes bug where non-gpu laser plugin could not see opponent car'

File: rr_description/urdf/evgp.urdf.xacro (robot description, xacro)
@@ -3,5 +3,5 @@
     <xacro:property name="props" value="${load_yaml('../conf/evgp_car_params.yaml')}"/>
     <xacro:include filename="evgp_body.urdf.xacro"/>
-    <xacro:evgp_body collide="true" color="Grey"/>
+    <xacro:evgp_body collision_bitmask="0x1" color="Grey"/>
     <!-- ************************** Links *************************** -->
     <xacro:macro name="null_inertia">
@@ -44,4 +44,11 @@
             <kp>1000000</kp>
             <kd>1000000</kd>
+            <collision>
+                <surface>
+                    <contact>
+                        <collide_bitmask>0x1</collide_bitmask>
+                    </contact>
+                </surface>
+            </collision>
         </gazebo>
         <xacro:set_link_color link="${name}" color="Black"/>
@@ -199,39 +206,39 @@
     </gazebo>
     <!-- FLIR Blackfly + wide-angle lens -->
-    <gazebo reference="camera">
-        <sensor name="camera_sensor" type="camera">
-            <camera>
-                <horizontal_fov>1.6955</horizontal_fov>
-                <image>
-                    <width>1280</width>
-                    <height>964</height>
-                    <format>R8G8B8</format>
-                </image>
-                <clip>
-                    <near>0.05</near>
-                    <far>100</far>
-                </clip>
-                <noise>
-                    <type>gaussian</type>
-                    <mean>0.0</mean>
-                    <stddev>0.007</stddev>
-                </noise>
-            </camera>
-            <always_on>true</always_on>
-            <update_rate>15</update_rate>
-            <plugin name="camera_controller" filename="libgazebo_ros_camera.so">
-                <alwaysOn>true</alwaysOn>
-                <cameraName>camera</cameraName>
-                <imageTopicName>image_color_rect</imageTopicName>
-                <cameraInfoTopicName>camera_info</cameraInfoTopicName>
-                <frameName>camera_optical</frameName>
-                <distortionK1>0.0</distortionK1>
-                <distortionK2>0.0</distortionK2>
-                <distortionK3>0.0</distortionK3>
-                <distortionT1>0.0</distortionT1>
-                <distortionT2>0.0</distortionT2>
-            </plugin>
-        </sensor>
-    </gazebo>
+<!--    <gazebo reference="camera">-->
+<!--        <sensor name="camera_sensor" type="camera">-->
+<!--            <camera>-->
+<!--                <horizontal_fov>1.6955</horizontal_fov>-->
+<!--                <image>-->
+<!--                    <width>1280</width>-->
+<!--                    <height>964</height>-->
+<!--                    <format>R8G8B8</format>-->
+<!--                </image>-->
+<!--                <clip>-->
+<!--                    <near>0.05</near>-->
+<!--                    <far>100</far>-->
+<!--                </clip>-->
+<!--                <noise>-->
+<!--                    <type>gaussian</type>-->
+<!--                    <mean>0.0</mean>-->
+<!--                    <stddev>0.007</stddev>-->
+<!--                </noise>-->
+<!--            </camera>-->
+<!--            <always_on>true</always_on>-->
+<!--            <update_rate>15</update_rate>-->
+<!--            <plugin name="camera_controller" filename="libgazebo_ros_camera.so">-->
+<!--                <alwaysOn>true</alwaysOn>-->
+<!--                <cameraName>camera</cameraName>-->
+<!--                <imageTopicName>image_color_rect</imageTopicName>-->
+<!--                <cameraInfoTopicName>camera_info</cameraInfoTopicName>-->
+<!--                <frameName>camera_optical</frameName>-->
+<!--                <distortionK1>0.0</distortionK1>-->
+<!--                <distortionK2>0.0</distortionK2>-->
+<!--                <distortionK3>0.0</distortionK3>-->
+<!--                <distortionT1>0.0</distortionT1>-->
+<!--                <distortionT2>0.0</distortionT2>-->
+<!--            </plugin>-->
+<!--        </sensor>-->
+<!--    </gazebo>-->
     <!-- IMU -->
     <gazebo reference="imu_link">
@@ -276,16 +283,16 @@
     </gazebo>
     <!-- ground-truth localization plugin -->
-    <gazebo>
-        <plugin name="ground_truth_tracker" filename="libgazebo_ros_p3d.so">
-            <alwaysOn>true</alwaysOn>
-            <updateRate>50.0</updateRate>
-            <bodyName>base_footprint</bodyName>
-            <topicName>/odometry/ground_truth</topicName>
-            <gaussianNoise>0.0</gaussianNoise>
-            <frameName>world</frameName>
-            <xyzOffsets>0 0 0</xyzOffsets>
-            <rpyOffsets>0 0 0</rpyOffsets>
-        </plugin>
-    </gazebo>
+<!--    <gazebo>-->
+<!--        <plugin name="ground_truth_tracker" filename="libgazebo_ros_p3d.so">-->
+<!--            <alwaysOn>true</alwaysOn>-->
+<!--            <updateRate>10.0</updateRate>-->
+<!--            <bodyName>base_footprint</bodyName>-->
+<!--            <topicName>/odometry/ground_truth</topicName>-->
+<!--            <gaussianNoise>0.0</gaussianNoise>-->
+<!--            <frameName>world</frameName>-->
+<!--            <xyzOffsets>0 0 0</xyzOffsets>-->
+<!--            <rpyOffsets>0 0 0</rpyOffsets>-->
+<!--        </plugin>-->
+<!--    </gazebo>-->
     <!-- ****************** Actuators ********************** -->
     <gazebo>
