Commit message: Simulating dynamic obstacles (#269)
* binary filter test layer

* slower updates

* adds script to generate opponent actors

* replaces sdf actor system with custom model controller

* makes urdf names slightly more consistent

* fix xacro build issue

* fix xacro build issue

* replaces test layer with full-custom obstacle layer

* better drawing

* fixes bug when rolling_window is true

* fix opponent controller escalating to sigkill issue

* addresses PR issues: collisions and start location

* add non-filtered mapping config back

* set non-filtering mapper as the default

* revert "Merge pull request #274"

* cherry-pick 'add switch for using gpu lidar plugin'

* cherry-pick 'fixes bug where non-gpu laser plugin could not see opponent car'

* adds back ground truth plugin to evgp gazebo which was mistakenly removed

* undo changes to imu refresh

* Keep max speed 5

File: rr_description/urdf/evgp.urdf.xacro (robot description, xacro)
@@ -1,4 +1,7 @@
 <robot name="evgp" xmlns:xacro="http://www.ros.org/wiki/xacro">
+    <xacro:property name="use_gpu" value="false"/>
     <xacro:property name="props" value="${load_yaml('../conf/evgp_car_params.yaml')}"/>
+    <xacro:include filename="evgp_body.urdf.xacro"/>
+    <xacro:evgp_body collision_bitmask="0x1" color="Grey"/>
     <!-- ************************** Links *************************** -->
     <xacro:macro name="null_inertia">
@@ -18,26 +21,4 @@
         </gazebo>
     </xacro:macro>
-    <link name="base_footprint">
-        <xacro:null_inertia/>
-    </link>
-    <link name="body_visual_origin">
-        <xacro:null_inertia/>
-        <visual>
-            <xacro:mesh_geometry/>
-        </visual>
-        <collision>
-            <xacro:mesh_geometry/>
-        </collision>
-    </link>
-    <xacro:set_link_color link="body_visual_origin" color="Grey"/>
-    <xacro:property name="body_inertia" value="${props['body_inertia']}"/>
-    <link name="body_inertial_center">
-        <inertial>
-            <mass value="${props['body_mass']}"/>
-            <inertia ixx="${body_inertia[0]}" ixy="${body_inertia[1]}" ixz="${body_inertia[2]}"
-                     iyy="${body_inertia[3]}" iyz="${body_inertia[4]}" izz="${body_inertia[5]}"/>
-        </inertial>
-    </link>
-    <gazebo reference="body_inertial_center"/>
     <xacro:macro name="wheel_link" params="name radius width">
         <link name="${name}">
@@ -63,4 +44,11 @@
             <kp>1000000</kp>
             <kd>1000000</kd>
+            <collision>
+                <surface>
+                    <contact>
+                        <collide_bitmask>0x1</collide_bitmask>
+                    </contact>
+                </surface>
+            </collision>
         </gazebo>
         <xacro:set_link_color link="${name}" color="Black"/>
@@ -119,14 +107,4 @@
     <xacro:set_link_color link="imu_link" color="Gold"/>
     <!-- ************************** Joints *************************** -->
-    <joint name="base_footprint_to_mesh_origin" type="fixed">
-        <parent link="base_footprint"/>
-        <child link="body_visual_origin"/>
-        <origin xyz="1.45 0.515 -0.051" rpy="${pi/2} 0 ${-pi/2}"/>
-    </joint>
-    <joint name="base_footprint_to_body_inertial_center" type="fixed">
-        <parent link="base_footprint"/>
-        <child link="body_inertial_center"/>
-        <origin xyz="${' '.join(str(x) for x in props['body_com'])}"/>
-    </joint>
     <xacro:property name="joint_flop_distance" value="0.02"/>
     <xacro:macro name="back_wheel_joint" params="dest_link y">
@@ -195,6 +173,7 @@
     <!-- ******************* Sensors *********************** -->
     <!-- SICK TiM551 -->
+    <xacro:property name="gpu_string" value="${'gpu_' if use_gpu else ''}"/>
     <gazebo reference="lidar">
-        <sensor type="ray" name="lidar_sensor">
+        <sensor type="${gpu_string}ray" name="lidar_sensor">
             <pose>0 0 0 0 0 0</pose>
             <visualize>false</visualize>
@@ -220,5 +199,5 @@
                 </noise>
             </ray>
-            <plugin name="gazebo_ros_head_hokuyo_controller" filename="libgazebo_ros_laser.so">
+            <plugin name="laser_controller" filename="libgazebo_ros_${gpu_string}laser.so">
                 <topicName>/scan</topicName>
                 <frameName>lidar</frameName>
@@ -227,39 +206,39 @@
     </gazebo>
     <!-- FLIR Blackfly + wide-angle lens -->
-    <gazebo reference="camera">
-        <sensor name="camera_sensor" type="camera">
-            <camera>
-                <horizontal_fov>1.6955</horizontal_fov>
-                <image>
-                    <width>1280</width>
-                    <height>964</height>
-                    <format>R8G8B8</format>
-                </image>
-                <clip>
-                    <near>0.05</near>
-                    <far>100</far>
-                </clip>
-                <noise>
-                    <type>gaussian</type>
-                    <mean>0.0</mean>
-                    <stddev>0.007</stddev>
-                </noise>
-            </camera>
-            <always_on>true</always_on>
-            <update_rate>15</update_rate>
-            <plugin name="camera_controller" filename="libgazebo_ros_camera.so">
-                <alwaysOn>true</alwaysOn>
-                <cameraName>camera</cameraName>
-                <imageTopicName>image_color_rect</imageTopicName>
-                <cameraInfoTopicName>camera_info</cameraInfoTopicName>
-                <frameName>camera_optical</frameName>
-                <distortionK1>0.0</distortionK1>
-                <distortionK2>0.0</distortionK2>
-                <distortionK3>0.0</distortionK3>
-                <distortionT1>0.0</distortionT1>
-                <distortionT2>0.0</distortionT2>
-            </plugin>
-        </sensor>
-    </gazebo>
+<!--    <gazebo reference="camera">-->
+<!--        <sensor name="camera_sensor" type="camera">-->
+<!--            <camera>-->
+<!--                <horizontal_fov>1.6955</horizontal_fov>-->
+<!--                <image>-->
+<!--                    <width>1280</width>-->
+<!--                    <height>964</height>-->
+<!--                    <format>R8G8B8</format>-->
+<!--                </image>-->
+<!--                <clip>-->
+<!--                    <near>0.05</near>-->
+<!--                    <far>100</far>-->
+<!--                </clip>-->
+<!--                <noise>-->
+<!--                    <type>gaussian</type>-->
+<!--                    <mean>0.0</mean>-->
+<!--                    <stddev>0.007</stddev>-->
+<!--                </noise>-->
+<!--            </camera>-->
+<!--            <always_on>true</always_on>-->
+<!--            <update_rate>15</update_rate>-->
+<!--            <plugin name="camera_controller" filename="libgazebo_ros_camera.so">-->
+<!--                <alwaysOn>true</alwaysOn>-->
+<!--                <cameraName>camera</cameraName>-->
+<!--                <imageTopicName>image_color_rect</imageTopicName>-->
+<!--                <cameraInfoTopicName>camera_info</cameraInfoTopicName>-->
+<!--                <frameName>camera_optical</frameName>-->
+<!--                <distortionK1>0.0</distortionK1>-->
+<!--                <distortionK2>0.0</distortionK2>-->
+<!--                <distortionK3>0.0</distortionK3>-->
+<!--                <distortionT1>0.0</distortionT1>-->
+<!--                <distortionT2>0.0</distortionT2>-->
+<!--            </plugin>-->
+<!--        </sensor>-->
+<!--    </gazebo>-->
     <!-- IMU -->
     <gazebo reference="imu_link">

Commit message: planning with longer range lidar and no straight path bias 🎉

File: rr_description/urdf/evgp.urdf.xacro (robot description, xacro)
@@ -1,4 +1,4 @@
 <robot name="evgp" xmlns:xacro="http://www.ros.org/wiki/xacro">
-    <xacro:property name="use_gpu" value="false"/>
+    <xacro:property name="use_gpu" value="true"/>
     <xacro:property name="props" value="${load_yaml('../conf/evgp_car_params.yaml')}"/>
     <xacro:include filename="evgp_body.urdf.xacro"/>
@@ -172,5 +172,5 @@
     </joint>
     <!-- ******************* Sensors *********************** -->
-    <!-- SICK TiM551 -->
+    <!-- Velodyne Puck VLP-16 -->
     <xacro:property name="gpu_string" value="${'gpu_' if use_gpu else ''}"/>
     <gazebo reference="lidar">
@@ -178,17 +178,17 @@
             <pose>0 0 0 0 0 0</pose>
             <visualize>false</visualize>
-            <update_rate>15</update_rate>
+            <update_rate>10</update_rate>
             <ray>
                 <scan>
                     <horizontal>
-                        <samples>270</samples>
+                        <samples>360</samples>
                         <resolution>1</resolution>  <!-- controls interpolation, leave at 1 -->
-                        <min_angle>${-pi*0.75}</min_angle>
-                        <max_angle>${pi*0.75}</max_angle>
+                        <min_angle>${-pi}</min_angle>
+                        <max_angle>${pi}</max_angle>
                     </horizontal>
                 </scan>
                 <range>
-                    <min>0.10</min>
-                    <max>8.0</max>
+                    <min>1.0</min>
+                    <max>100.0</max>
                     <resolution>0.01</resolution>
                 </range>
@@ -196,5 +196,5 @@
                     <type>gaussian</type>
                     <mean>0.0</mean>
-                    <stddev>0.02</stddev>
+                    <stddev>0.005</stddev>
                 </noise>
             </ray>

Commit message: fixes sim lidar angle

File: rr_description/urdf/evgp.urdf.xacro (robot description, xacro)
@@ -107,12 +107,11 @@
     <xacro:set_link_color link="imu_link" color="Gold"/>
     <!-- ************************** Joints *************************** -->
-    <xacro:property name="joint_flop_distance" value="0.02"/>
+    <xacro:property name="joint_flop_both" value="0.03"/>
     <xacro:macro name="back_wheel_joint" params="dest_link y">
         <joint name="base_footprint_to_${dest_link}" type="continuous">
             <parent link="base_footprint"/>
             <child link="${dest_link}"/>
-            <origin xyz="0 ${y} ${(props['wheel_radius_back'] / 2) - joint_flop_distance}" rpy="${-pi/2} 0 0"/>
+            <origin xyz="0 ${y} ${(props['wheel_radius_back'] / 2) - joint_flop_both}" rpy="${-pi/2} 0 0"/>
             <axis xyz="0 0 1"/>
-            <dynamics damping="0.01"/>
         </joint>
         <gazebo reference="base_footprint_to_${dest_link}"/>
@@ -120,4 +119,5 @@
     <xacro:back_wheel_joint dest_link="wheel_BL" y="${props['track'] / 2}"/>
     <xacro:back_wheel_joint dest_link="wheel_BR" y="${-props['track'] / 2}"/>
+    <xacro:property name="joint_flop_front" value="0.007"/>
     <xacro:macro name="steering_joints" params="steering_link wheel_link y">
         <joint name="base_footprint_to_${steering_link}" type="revolute">
@@ -131,5 +131,5 @@
         <gazebo reference="base_footprint_to_${steering_link}"/>
         <joint name="${steering_link}_to_${wheel_link}" type="continuous">
-            <origin xyz="0 0 ${-joint_flop_distance}" rpy="${pi/2} 0 0"/>
+            <origin xyz="0 0 ${-joint_flop_both - joint_flop_front}" rpy="${pi/2} 0 0"/>
             <parent link="${steering_link}"/>
             <child link="${wheel_link}"/>

Commit message: bugfixes from pull request review

File: rr_description/urdf/evgp.urdf.xacro (robot description, xacro)
@@ -1,4 +1,4 @@
 <robot name="evgp" xmlns:xacro="http://www.ros.org/wiki/xacro">
-    <xacro:property name="use_gpu" value="true"/>
+    <xacro:property name="use_gpu" value="false"/>
     <xacro:property name="props" value="${load_yaml('../conf/evgp_car_params.yaml')}"/>
     <xacro:include filename="evgp_body.urdf.xacro"/>

Commit message: Correct lidar and imu

File: rr_description/urdf/evgp.urdf.xacro (robot description, xacro)
@@ -143,5 +143,5 @@
         <parent link="base_footprint"/>
         <child link="lidar"/>
-        <origin xyz="1.2 0 0.18" rpy="0 0 0"/>
+        <origin xyz=".825 -.19 0.27875" rpy="0 0 0"/>
     </joint>
     <joint name="base_footprint_to_gps" type="fixed">
@@ -169,5 +169,5 @@
         <parent link="base_footprint"/>
         <child link="imu_link"/>
-        <origin xyz="0.75 0.5 0.1" rpy="0 0 0"/>
+        <origin xyz="0.065 0.22 0.97" rpy="0 0 0"/>
     </joint>
     <!-- ******************* Sensors *********************** -->

Commit message: reset changes to evgp

File: rr_description/urdf/evgp.urdf.xacro (robot description, xacro)
@@ -143,5 +143,5 @@
         <parent link="base_footprint"/>
         <child link="lidar"/>
-        <origin xyz=".825 -.19 0.27875" rpy="0 0 0"/>
+        <origin xyz="1.2 0 0.18" rpy="0 0 0"/>
     </joint>
     <joint name="base_footprint_to_gps" type="fixed">
@@ -169,5 +169,5 @@
         <parent link="base_footprint"/>
         <child link="imu_link"/>
-        <origin xyz="0.065 0.22 0.97" rpy="0 0 0"/>
+        <origin xyz="0.75 0.5 0.1" rpy="0 0 0"/>
     </joint>
     <!-- ******************* Sensors *********************** -->
