Commit message: Add location for IMUs and LIDAR

File: rr_description/urdf/rigatoni.urdf.xacro (robot description, xacro)
@@ -223,6 +223,6 @@
     <xacro:set_base_footprint_to_link link_name="gps_link" xyz="0.55 0.39 1.22" rpy="0 0 0"/>
     <xacro:set_base_footprint_to_link link_name="camera" xyz="0.61 0.39 1.03" rpy="0 0 0"/>
-    <xacro:set_base_footprint_to_link link_name="imu_bottom_link" xyz="0 0 0.21" rpy="0 0 0"/>
-    <xacro:set_base_footprint_to_link link_name="imu_top_link" xyz="0.60 0.39 0.95" rpy="0 0 0"/>
+    <xacro:set_base_footprint_to_link link_name="imu_bottom_link" xyz=".22 .065 0.97" rpy="0 0 0"/>
+    <xacro:set_base_footprint_to_link link_name="imu_top_link" xyz="-0.53 -0.2 0.2375" rpy="0 0 0"/>
     <xacro:set_base_footprint_to_link link_name="april_2" xyz=".48  -0.55 0.26" rpy="0 0 ${pi/2}"/>
     <xacro:set_base_footprint_to_link link_name="april_3" xyz="-.19 -0.43 0.26" rpy="0 0 ${pi/4}"/>
@@ -233,5 +233,5 @@
     <!-- Velodyne Puck VLP-16 -->
     <xacro:VLP-16 parent="base_footprint" name="lidar" topic="/velodyne_points" hz="10" samples="500" gpu="true">
-        <origin xyz="1.175 0 0.175" rpy="0 0 0" />
+        <origin xyz=".825 -0.19 0.27875" rpy="0 0 0" />
     </xacro:VLP-16>
     <!-- FLIR Blackfly + wide-angle lens -->

Commit message: Add location to rigatoni

File: rr_description/urdf/rigatoni.urdf.xacro (robot description, xacro)
@@ -222,7 +222,7 @@
     </xacro:macro>
     <xacro:set_base_footprint_to_link link_name="gps_link" xyz="0.55 0.39 1.22" rpy="0 0 0"/>
-    <xacro:set_base_footprint_to_link link_name="camera" xyz="0.61 0.39 1.03" rpy="0 0.4 0"/>
-    <xacro:set_base_footprint_to_link link_name="imu_bottom_link" xyz="0 0 0.21" rpy="0 0 0"/>
-    <xacro:set_base_footprint_to_link link_name="imu_top_link" xyz="0.60 0.39 0.95" rpy="0 0 0"/>
+    <xacro:set_base_footprint_to_link link_name="camera" xyz="0.61 0.39 1.03" rpy="0 0 0"/>
+    <xacro:set_base_footprint_to_link link_name="imu_bottom_link" xyz=".22 .065 0.97" rpy="0 0 0"/>
+    <xacro:set_base_footprint_to_link link_name="imu_top_link" xyz="-0.53 -0.2 0.2375" rpy="0 0 0"/>
     <xacro:set_base_footprint_to_link link_name="april_2" xyz=".48  -0.55 0.26" rpy="0 0 ${pi/2}"/>
     <xacro:set_base_footprint_to_link link_name="april_3" xyz="-.19 -0.43 0.26" rpy="0 0 ${pi/4}"/>
@@ -233,5 +233,5 @@
     <!-- Velodyne Puck VLP-16 -->
     <xacro:VLP-16 parent="base_footprint" name="lidar" topic="/velodyne_points" hz="10" samples="500" gpu="true">
-        <origin xyz="1.175 0 0.175" rpy="0 0 0" />
+        <origin xyz=".825 -0.19 0.27875" rpy="0 0 0" />
     </xacro:VLP-16>
     <!-- FLIR Blackfly + wide-angle lens -->

Commit message: hotfix

File: rr_description/urdf/rigatoni.urdf.xacro (robot description, xacro)
@@ -109,4 +109,7 @@
         <xacro:null_inertia/>
     </link>
+    <link name="velodyne">
+        <xacro:null_inertia/>
+    </link>
     <link name="gps_link">
         <xacro:null_inertia/>
@@ -235,4 +238,5 @@
         <origin xyz="1.175 0 0.175" rpy="0 0 0" />
     </xacro:VLP-16>
+    <xacro:set_base_footprint_to_link link_name="velodyne" xyz="0 0 0" rpy="0 0 0"/>
     <!-- FLIR Blackfly + wide-angle lens -->
     <gazebo reference="camera">

Commit message: cone connection

File: rr_description/urdf/rigatoni.urdf.xacro (robot description, xacro)
@@ -230,4 +230,12 @@
     <xacro:set_base_footprint_to_link link_name="april_5" xyz="-.19  0.43 0.26" rpy="0 0 -${pi/4}"/>
     <xacro:set_base_footprint_to_link link_name="april_6" xyz=".48   0.55 0.26" rpy="0 0 ${pi/2}"/>
+    <link name="velodyne">
+        <xacro:null_inertia/>
+    </link>
+    <joint name="AHHHH" type="fixed">
+        <parent link="lidar"/>
+        <child link="velodyne"/>
+        <origin xyz="0 0 0" rpy="0 0 0"/>
+    </joint>
     <!-- ******************* Sensors *********************** -->
     <!-- Velodyne Puck VLP-16 -->

Commit message: cone

File: rr_description/urdf/rigatoni.urdf.xacro (robot description, xacro)
@@ -230,4 +230,9 @@
     <xacro:set_base_footprint_to_link link_name="april_5" xyz="-.19  0.43 0.26" rpy="0 0 -${pi/4}"/>
     <xacro:set_base_footprint_to_link link_name="april_6" xyz=".48   0.55 0.26" rpy="0 0 ${pi/2}"/>
+    <!-- ******************* Sensors *********************** -->
+    <!-- Velodyne Puck VLP-16 -->
+    <xacro:VLP-16 parent="base_footprint" name="lidar" topic="/velodyne_points" hz="10" samples="500" gpu="true">
+        <origin xyz=".825 -0.19 0.27875" rpy="0 0 0" />
+    </xacro:VLP-16>
     <link name="velodyne">
         <xacro:null_inertia/>
@@ -238,9 +243,4 @@
         <origin xyz="0 0 0" rpy="0 0 0"/>
     </joint>
-    <!-- ******************* Sensors *********************** -->
-    <!-- Velodyne Puck VLP-16 -->
-    <xacro:VLP-16 parent="base_footprint" name="lidar" topic="/velodyne_points" hz="10" samples="500" gpu="true">
-        <origin xyz=".825 -0.19 0.27875" rpy="0 0 0" />
-    </xacro:VLP-16>
     <!-- FLIR Blackfly + wide-angle lens -->
     <gazebo reference="camera">

Commit message: updates launch file

File: rr_description/urdf/rigatoni.urdf.xacro (robot description, xacro)
@@ -4,4 +4,5 @@
     <xacro:property name="body_inertia" value="${props['body_inertia']}"/>
     <xacro:include filename="$(find velodyne_description)/urdf/VLP-16.urdf.xacro"/>
+    <!-- <xacro:include filename="$(find rr_description)/" -->
     <!-- ************************** Links *************************** -->
     <xacro:macro name="null_inertia">
@@ -13,5 +14,5 @@
     <xacro:macro name="mesh_geometry">
         <geometry>
-            <mesh filename="package://rr_description/meshes/rigatoni.stl" scale="0.01 0.01 0.01"/>
+            <mesh filename="$(find rr_description)/meshes/rigatoni.stl" scale="0.01 0.01 0.01"/>
         </geometry>
     </xacro:macro>
@@ -347,6 +348,9 @@
     <!-- ****************** Actuators ********************** -->
     <gazebo>
-        <plugin name="gazebo_ros_control" filename="libgazebo_ros_control.so">
-            <robotNamespace>/</robotNamespace>
+        <plugin name="gazebo_ros2_control" filename="libgazebo_ros2_control.so">
+            <robot_namespace>rigatoni</robot_namespace>
+            <robot_param>robot_description</robot_param>
+            <robot_param_node>robot_state_publisher</robot_param_node>
+            <parameters>$(find rr_description)/conf/controller.yaml</parameters>
         </plugin>
     </gazebo>

Commit message: working simulator fixing controls

File: rr_description/urdf/rigatoni.urdf.xacro (robot description, xacro)
@@ -1,5 +1,5 @@
 <robot name="rigatoni" xmlns:xacro="http://www.ros.org/wiki/xacro">
     <xacro:property name="use_gpu" value="false"/>
-    <xacro:property name="props" value="${load_yaml('../conf/evgp_car_params.yaml')}"/>
+    <xacro:property name="props" value="${load_yaml('../src/conf/evgp_car_params.yaml')}"/>
     <xacro:property name="body_inertia" value="${props['body_inertia']}"/>
     <xacro:include filename="$(find velodyne_description)/urdf/VLP-16.urdf.xacro"/>
@@ -143,13 +143,4 @@
     </link>
     <xacro:set_link_color link="imu_top_link" color="Gold"/>
-    <link name="imu_bottom_link">
-        <xacro:null_inertia/>
-        <visual>
-            <geometry>
-                <box size="0.05 0.05 0.05"/>
-            </geometry>
-        </visual>
-    </link>
-    <xacro:set_link_color link="imu_bottom_link" color="Gold"/>
     <xacro:macro name="april_link" params="name tag_number">
         <link name="${name}">
@@ -224,5 +215,4 @@
     <xacro:set_base_footprint_to_link link_name="gps_link" xyz="0.55 0.39 1.22" rpy="0 0 0"/>
     <xacro:set_base_footprint_to_link link_name="camera" xyz="0.61 0.39 1.03" rpy="0 0.4 0"/>
-    <xacro:set_base_footprint_to_link link_name="imu_bottom_link" xyz="0 0 0.21" rpy="0 0 0"/>
     <xacro:set_base_footprint_to_link link_name="imu_top_link" xyz="0.60 0.39 0.95" rpy="0 0 0"/>
     <xacro:set_base_footprint_to_link link_name="april_2" xyz=".48  -0.55 0.26" rpy="0 0 ${pi/2}"/>
@@ -233,5 +223,5 @@
     <!-- ******************* Sensors *********************** -->
     <!-- Velodyne Puck VLP-16 -->
-    <xacro:VLP-16 parent="base_footprint" name="lidar" topic="/velodyne_points" hz="10" samples="500" gpu="true">
+    <xacro:VLP-16 parent="base_footprint" name="velodyne" topic="/velodyne_points" organize_cloud="false" hz="10" samples="440" gpu="true">
         <origin xyz="1.175 0 0.175" rpy="0 0 0" />
     </xacro:VLP-16>
@@ -312,26 +302,5 @@
         </sensor>
     </gazebo>
-    <!-- GPS -->
-    <gazebo>
-        <plugin name="gps_controller" filename="libhector_gazebo_ros_gps.so">
-            <robotNamespace>/</robotNamespace>
-            <updateRate>10</updateRate>
-            <bodyName>gps_link</bodyName>
-            <frameId>gps_link</frameId>
-            <topicName>gps/fix</topicName>
-            <velocityTopicName>gps/vel</velocityTopicName>
-            <referenceLatitude>33.8</referenceLatitude>
-            <referenceLongitude>-84.4</referenceLongitude>
-            <referenceHeading>0</referenceHeading>
-            <referenceAltitude>0</referenceAltitude>
-            <drift>0.2 0.2 0.2</drift>
-            <driftFrequency>0.01 0.01 0.01</driftFrequency>
-            <gaussianNoise>0.05 0.05 0.05</gaussianNoise>
-            <velocityDrift>0.05 0.05 0.05</velocityDrift>
-            <velocityDriftFrequency>0.1 0.1 0.1</velocityDriftFrequency>
-            <velocityGaussianNoise>0.05 0.05 0.05</velocityGaussianNoise>
-        </plugin>
-    </gazebo>
-    <!-- ground-truth localization plugin -->
+        <!-- ground-truth localization plugin -->
     <gazebo>
         <plugin name="ground_truth_tracker" filename="libgazebo_ros_p3d.so">
