Commit message: remove urdfs

File: rr_description/urdf/opponents/evgp_body.urdf.xacro (robot description, xacro)
@@ -1,5 +1,3 @@
 <robot name="evgp" xmlns:xacro="http://www.ros.org/wiki/xacro">
-    <xacro:property name="props" value="${load_yaml('../../conf/evgp_car_params.yaml')}"/>
-    <xacro:property name="body_inertia" value="${props['body_inertia']}"/>
     <xacro:macro name="null_inertia">
         <inertial>
@@ -42,12 +40,4 @@
             </collision>
         </gazebo>
-        <link name="body_inertial_center">
-            <inertial>
-                <mass value="${props['body_mass']}"/>
-                <inertia ixx="${body_inertia[0]}" ixy="${body_inertia[1]}" ixz="${body_inertia[2]}"
-                         iyy="${body_inertia[3]}" iyz="${body_inertia[4]}" izz="${body_inertia[5]}"/>
-            </inertial>
-        </link>
-        <gazebo reference="body_inertial_center"/>
         <!-- ************************** Joints *************************** -->
         <joint name="base_footprint_to_mesh_origin" type="fixed">
@@ -56,9 +46,4 @@
             <origin xyz="1.45 0.515 -0.051" rpy="${pi/2} 0 ${-pi/2}"/>
         </joint>
-        <joint name="base_footprint_to_body_inertial_center" type="fixed">
-            <parent link="base_footprint"/>
-            <child link="body_inertial_center"/>
-            <origin xyz="${' '.join(str(x) for x in props['body_com'])}"/>
-        </joint>
     </xacro:macro>
 </robot>

Commit message: changes

File: rr_description/urdf/opponents/evgp_body.urdf.xacro (robot description, xacro)
@@ -8,5 +8,5 @@
     <xacro:macro name="mesh_geometry">
         <geometry>
-            <mesh filename="package://rr_description/meshes/EVGP_robot.STL" scale="0.001 0.001 0.001"/>
+            <mesh filename="package://rr_description/meshes/rigatoni.stl" scale="0.01 0.01 0.01"/>
         </geometry>
     </xacro:macro>
@@ -40,9 +40,12 @@
             </collision>
         </gazebo>
+        <gazebo reference="body_visual_origin">
+            <turnGravityOff>true</turnGravityOff>
+        </gazebo>
         <!-- ************************** Joints *************************** -->
         <joint name="base_footprint_to_mesh_origin" type="fixed">
             <parent link="base_footprint"/>
             <child link="body_visual_origin"/>
-            <origin xyz="1.45 0.515 -0.051" rpy="${pi/2} 0 ${-pi/2}"/>
+            <origin xyz="0.53 0 0.1" rpy="${pi/2} 0 ${pi/2}"/>
         </joint>
     </xacro:macro>

Commit message: changes

File: rr_description/urdf/opponents/evgp_body.urdf.xacro (robot description, xacro)
@@ -16,5 +16,5 @@
         </gazebo>
     </xacro:macro>
-    <xacro:macro name="evgp_body" params="collision_bitmask color">
+    <xacro:macro name="evgp_body" params="collision_bitmask color april0 april1 april2 april3 april4">
         <!-- ************************** Links *************************** -->
         <link name="base_footprint">
@@ -43,10 +43,40 @@
             <turnGravityOff>true</turnGravityOff>
         </gazebo>
+        <xacro:macro name="april_link" params="name tag_number">
+            <link name="${name}">
+                <xacro:null_inertia/>
+                <visual>
+                    <geometry>
+                        <box size="0.001 0.127 0.127 "/>
+                    </geometry>
+                </visual>
+            </link>
+            <gazebo reference="${name}">
+                <material>${tag_number}</material>
+            </gazebo>
+        </xacro:macro>
+        <xacro:april_link name="april_0" tag_number="${april0}"/>
+        <xacro:april_link name="april_1" tag_number="${april1}"/>
+        <xacro:april_link name="april_2" tag_number="${april2}"/>
+        <xacro:april_link name="april_3" tag_number="${april3}"/>
+        <xacro:april_link name="april_4" tag_number="${april4}"/>
         <!-- ************************** Joints *************************** -->
         <joint name="base_footprint_to_mesh_origin" type="fixed">
             <parent link="base_footprint"/>
             <child link="body_visual_origin"/>
-            <origin xyz="0.53 0 0.1" rpy="${pi/2} 0 ${pi/2}"/>
+            <origin xyz="0.53 0 -0.05" rpy="${pi/2} 0 ${pi/2}"/>
         </joint>
+        <xacro:macro name="set_base_footprint_to_link" params="link_name xyz rpy">
+            <joint name="base_footprint_to_${link_name}" type="fixed">
+                <parent link="base_footprint"/>
+                <child link="${link_name}"/>
+                <origin xyz="${xyz}" rpy="${rpy}"/>
+            </joint>
+        </xacro:macro>
+        <xacro:set_base_footprint_to_link link_name="april_0" xyz="-.38  0    0.26" rpy="0 0 0"/>
+        <xacro:set_base_footprint_to_link link_name="april_1" xyz="-.19  0.43 0.26" rpy="0 0 -${pi/4}"/>
+        <xacro:set_base_footprint_to_link link_name="april_2" xyz="-.19 -0.43 0.26" rpy="0 0 ${pi/4}"/>
+        <xacro:set_base_footprint_to_link link_name="april_3" xyz=".48  -0.55 0.26" rpy="0 0 ${pi/2}"/>
+        <xacro:set_base_footprint_to_link link_name="april_4" xyz=".48   0.55 0.26" rpy="0 0 ${pi/2}"/>
     </xacro:macro>
 </robot>

File: rr_description/urdf/opponents/evgp_opponent_0.urdf.xacro (robot description, xacro)
@@ -1,5 +1,12 @@
 <robot name="evgp_opponent" xmlns:xacro="http://www.ros.org/wiki/xacro">
     <xacro:include filename="evgp_body.urdf.xacro"/>
-    <xacro:evgp_body collision_bitmask="0x4" color="Blue"/>
+    <xacro:evgp_body
+    collision_bitmask="0x4"
+    color="Blue"
+    april0="tag36_11_00000"
+    april1="tag36_11_00000"
+    april2="tag36_11_00000"
+    april3="tag36_11_00000"
+    april4="tag36_11_00000"/>
     <gazebo reference="base_footprint">
         <kinematic>true</kinematic>

File: rr_description/urdf/opponents/evgp_opponent_1.urdf.xacro (robot description, xacro)
@@ -1,5 +1,10 @@
 <robot name="evgp_opponent" xmlns:xacro="http://www.ros.org/wiki/xacro">
     <xacro:include filename="evgp_body.urdf.xacro"/>
-    <xacro:evgp_body collision_bitmask="0x8" color="Green"/>
+    <xacro:evgp_body collision_bitmask="0x8" color="Green"
+    april0="tag36_11_00000"
+    april1="tag36_11_00000"
+    april2="tag36_11_00000"
+    april3="tag36_11_00000"
+    april4="tag36_11_00000"/>
     <gazebo reference="base_footprint">
         <kinematic>true</kinematic>

File: rr_description/urdf/opponents/evgp_opponent_2.urdf.xacro (robot description, xacro)
@@ -1,5 +1,10 @@
 <robot name="evgp_opponent" xmlns:xacro="http://www.ros.org/wiki/xacro">
     <xacro:include filename="evgp_body.urdf.xacro"/>
-    <xacro:evgp_body collision_bitmask="0x10" color="Yellow"/>
+    <xacro:evgp_body collision_bitmask="0x10" color="Yellow"
+    april0="tag36_11_00000"
+    april1="tag36_11_00000"
+    april2="tag36_11_00000"
+    april3="tag36_11_00000"
+    april4="tag36_11_00000"/>
     <gazebo reference="base_footprint">
         <kinematic>true</kinematic>

File: rr_description/urdf/opponents/evgp_opponent_3.urdf.xacro (robot description, xacro)
@@ -1,5 +1,10 @@
 <robot name="evgp_opponent" xmlns:xacro="http://www.ros.org/wiki/xacro">
     <xacro:include filename="evgp_body.urdf.xacro"/>
-    <xacro:evgp_body collision_bitmask="0x20" color="Red"/>
+    <xacro:evgp_body collision_bitmask="0x20" color="Red"
+    april0="tag36_11_00000"
+    april1="tag36_11_00000"
+    april2="tag36_11_00000"
+    april3="tag36_11_00000"
+    april4="tag36_11_00000"/>
     <gazebo reference="base_footprint">
         <kinematic>true</kinematic>

File: rr_description/urdf/opponents/evgp_opponent_4.urdf.xacro (robot description, xacro)
@@ -1,5 +1,10 @@
 <robot name="evgp_opponent" xmlns:xacro="http://www.ros.org/wiki/xacro">
     <xacro:include filename="evgp_body.urdf.xacro"/>
-    <xacro:evgp_body collision_bitmask="0x40" color="Purple"/>
+    <xacro:evgp_body collision_bitmask="0x40" color="Purple"
+    april0="tag36_11_00000"
+    april1="tag36_11_00000"
+    april2="tag36_11_00000"
+    april3="tag36_11_00000"
+    april4="tag36_11_00000"/>
     <gazebo reference="base_footprint">
         <kinematic>true</kinematic>

File: rr_description/urdf/rigatoni.urdf.xacro (robot description, xacro)
@@ -57,5 +57,5 @@
             <parent link="base_footprint"/>
             <child link="body_visual_origin"/>
-            <origin xyz="0.53 0 0" rpy="${pi/2} 0 ${pi/2}"/>
+            <origin xyz="0.53 0 -0.05" rpy="${pi/2} 0 ${pi/2}"/>
         </joint>
         <joint name="base_footprint_to_body_inertial_center" type="fixed">
@@ -151,15 +151,22 @@
     </link>
     <xacro:set_link_color link="imu_bottom_link" color="Gold"/>
-    <link name='april'>
-        <xacro:null_inertia/>
-        <visual>
-            <geometry>
-                <box size="0.001 0.3 0.3 "/>
-            </geometry>
-        </visual>
-    </link>
-    <gazebo reference="april">
-        <material>Apriltag</material>
-    </gazebo>
+    <xacro:macro name="april_link" params="name tag_number">
+        <link name="${name}">
+            <xacro:null_inertia/>
+            <visual>
+                <geometry>
+                    <box size="0.001 0.127 0.127 "/>
+                </geometry>
+            </visual>
+        </link>
+        <gazebo reference="${name}">
+            <material>${tag_number}</material>
+        </gazebo>
+    </xacro:macro>
+    <xacro:april_link name="april_0" tag_number="tag36_11_00000"/>
+    <xacro:april_link name="april_1" tag_number="tag36_11_00001"/>
+    <xacro:april_link name="april_2" tag_number="tag36_11_00002"/>
+    <xacro:april_link name="april_3" tag_number="tag36_11_00003"/>
+    <xacro:april_link name="april_4" tag_number="tag36_11_00004"/>
     <!-- ************************** Joints *************************** -->
     <xacro:property name="joint_flop_both" value="0.03"/>
@@ -196,14 +203,4 @@
     <xacro:steering_joints steering_link="steering_link_left" wheel_link="wheel_FL" y="${props['track'] / 2}"/>
     <xacro:steering_joints steering_link="steering_link_right" wheel_link="wheel_FR" y="${-props['track'] / 2}"/>
-    <joint name="base_footprint_to_gps" type="fixed">
-        <parent link="base_footprint"/>
-        <child link="gps_link"/>
-        <origin xyz="0.63 0.4 1.27" rpy="0 0 0"/>
-    </joint>
-    <joint name="base_footprint_to_camera" type="fixed">
-        <parent link="base_footprint"/>
-        <child link="camera"/>
-        <origin xyz="0.68 0.4 0.8" rpy="0 0.2 0"/>
-    </joint>
     <xacro:macro name="camera_optical_frame" params="camera_link">
         <link name="${camera_link}_optical">
@@ -217,23 +214,24 @@
     </xacro:macro>
     <xacro:camera_optical_frame camera_link="camera"/>
-    <joint name="base_footprint_to_imu" type="fixed">
-        <parent link="base_footprint"/>
-        <child link="imu_top_link"/>
-        <origin xyz="0.67 0.4 0.67" rpy="0 0 0"/>
-    </joint>
-    <joint name="base_footprint_to_imu2" type="fixed">
-        <parent link="base_footprint"/>
-        <child link="imu_bottom_link"/>
-        <origin xyz="0 0 0.21" rpy="0 0 0"/>
-    </joint>
-    <joint name="base_footprint_to_april" type="fixed">
-        <parent link="base_footprint"/>
-        <child link="april"/>
-        <origin xyz="-.3 0 0.51" rpy="0 0 0"/>
-    </joint>
+    <xacro:macro name="set_base_footprint_to_link" params="link_name xyz rpy">
+        <joint name="base_footprint_to_${link_name}" type="fixed">
+            <parent link="base_footprint"/>
+            <child link="${link_name}"/>
+            <origin xyz="${xyz}" rpy="${rpy}"/>
+        </joint>
+    </xacro:macro>
+    <xacro:set_base_footprint_to_link link_name="gps_link" xyz="0.55 0.39 1.22" rpy="0 0 0"/>
+    <xacro:set_base_footprint_to_link link_name="camera" xyz="0.61 0.39 1.03" rpy="0 0.4 0"/>
+    <xacro:set_base_footprint_to_link link_name="imu_bottom_link" xyz="0 0 0.21" rpy="0 0 0"/>
+    <xacro:set_base_footprint_to_link link_name="imu_top_link" xyz="0.60 0.39 0.95" rpy="0 0 0"/>
+    <xacro:set_base_footprint_to_link link_name="april_0" xyz="-.38 0 0.26"  rpy="0 0 0"/>
+    <xacro:set_base_footprint_to_link link_name="april_1" xyz="-.19  0.43 0.26" rpy="0 0 -${pi/4}"/>
+    <xacro:set_base_footprint_to_link link_name="april_2" xyz="-.19 -0.43 0.26" rpy="0 0 ${pi/4}"/>
+    <xacro:set_base_footprint_to_link link_name="april_3" xyz=".48 -0.55 0.26" rpy="0 0 ${pi/2}"/>
+    <xacro:set_base_footprint_to_link link_name="april_4" xyz=".48  0.55 0.26" rpy="0 0 ${pi/2}"/>
     <!-- ******************* Sensors *********************** -->
     <!-- Velodyne Puck VLP-16 -->
     <xacro:VLP-16 parent="base_footprint" name="lidar" topic="/velodyne_points" hz="10" samples="500" gpu="true">
-        <origin xyz="1.25 0 0.3" rpy="0 0 0" />
+        <origin xyz="1.175 0 0.175" rpy="0 0 0" />
     </xacro:VLP-16>
     <!-- FLIR Blackfly + wide-angle lens -->

Commit message: change

File: rr_description/urdf/opponents/evgp_body.urdf.xacro (robot description, xacro)
@@ -16,5 +16,5 @@
         </gazebo>
     </xacro:macro>
-    <xacro:macro name="evgp_body" params="collision_bitmask color april0 april1 april2 april3 april4">
+    <xacro:macro name="evgp_body" params="collision_bitmask color april2 april3 april4 april5 april6">
         <!-- ************************** Links *************************** -->
         <link name="base_footprint">
@@ -56,9 +56,9 @@
             </gazebo>
         </xacro:macro>
-        <xacro:april_link name="april_0" tag_number="${april0}"/>
-        <xacro:april_link name="april_1" tag_number="${april1}"/>
         <xacro:april_link name="april_2" tag_number="${april2}"/>
         <xacro:april_link name="april_3" tag_number="${april3}"/>
         <xacro:april_link name="april_4" tag_number="${april4}"/>
+        <xacro:april_link name="april_5" tag_number="${april5}"/>
+        <xacro:april_link name="april_6" tag_number="${april6}"/>
         <!-- ************************** Joints *************************** -->
         <joint name="base_footprint_to_mesh_origin" type="fixed">
@@ -74,9 +74,9 @@
             </joint>
         </xacro:macro>
-        <xacro:set_base_footprint_to_link link_name="april_0" xyz=".48  -0.55 0.26" rpy="0 0 ${pi/2}"/>
-        <xacro:set_base_footprint_to_link link_name="april_1" xyz="-.19 -0.43 0.26" rpy="0 0 ${pi/4}"/>
-        <xacro:set_base_footprint_to_link link_name="april_2" xyz="-.38  0    0.26" rpy="0 0 0"/>
-        <xacro:set_base_footprint_to_link link_name="april_3" xyz="-.19  0.43 0.26" rpy="0 0 -${pi/4}"/>
-        <xacro:set_base_footprint_to_link link_name="april_4" xyz=".48   0.55 0.26" rpy="0 0 ${pi/2}"/>
+        <xacro:set_base_footprint_to_link link_name="april_2" xyz=".48  -0.55 0.26" rpy="0 0 ${pi/2}"/>
+        <xacro:set_base_footprint_to_link link_name="april_3" xyz="-.19 -0.43 0.26" rpy="0 0 ${pi/4}"/>
+        <xacro:set_base_footprint_to_link link_name="april_4" xyz="-.38  0    0.26" rpy="0 0 0"/>
+        <xacro:set_base_footprint_to_link link_name="april_5" xyz="-.19  0.43 0.26" rpy="0 0 -${pi/4}"/>
+        <xacro:set_base_footprint_to_link link_name="april_6" xyz=".48   0.55 0.26" rpy="0 0 ${pi/2}"/>
         <gazebo reference="base_footprint">
             <kinematic>true</kinematic>

File: rr_description/urdf/opponents/evgp_opponent_0.urdf.xacro (robot description, xacro)
@@ -2,8 +2,8 @@
     <xacro:include filename="evgp_body.urdf.xacro"/>
     <xacro:evgp_body collision_bitmask="0x4" color="Blue"
-    april0="tag36_11_00002"
-    april1="tag36_11_00003"
-    april2="tag36_11_00004"
-    april3="tag36_11_00005"
-    april4="tag36_11_00006"/>
+    april2="tag36_11_00002"
+    april3="tag36_11_00003"
+    april4="tag36_11_00004"
+    april5="tag36_11_00005"
+    april6="tag36_11_00006"/>
 </robot>

File: rr_description/urdf/opponents/evgp_opponent_1.urdf.xacro (robot description, xacro)
@@ -2,8 +2,8 @@
     <xacro:include filename="evgp_body.urdf.xacro"/>
     <xacro:evgp_body collision_bitmask="0x8" color="Green"
-    april0="tag36_11_00012"
-    april1="tag36_11_00013"
-    april2="tag36_11_00014"
-    april3="tag36_11_00015"
-    april4="tag36_11_00016"/>
+    april2="tag36_11_00012"
+    april3="tag36_11_00013"
+    april4="tag36_11_00014"
+    april5="tag36_11_00015"
+    april6="tag36_11_00016"/>
 </robot>

File: rr_description/urdf/opponents/evgp_opponent_2.urdf.xacro (robot description, xacro)
@@ -2,8 +2,8 @@
     <xacro:include filename="evgp_body.urdf.xacro"/>
     <xacro:evgp_body collision_bitmask="0x10" color="Yellow"
-    april0="tag36_11_00022"
-    april1="tag36_11_00023"
-    april2="tag36_11_00024"
-    april3="tag36_11_00025"
-    april4="tag36_11_00026"/>
+    april2="tag36_11_00022"
+    april3="tag36_11_00023"
+    april4="tag36_11_00024"
+    april5="tag36_11_00025"
+    april6="tag36_11_00026"/>
 </robot>

File: rr_description/urdf/opponents/evgp_opponent_3.urdf.xacro (robot description, xacro)
@@ -2,8 +2,8 @@
     <xacro:include filename="evgp_body.urdf.xacro"/>
     <xacro:evgp_body collision_bitmask="0x20" color="Red"
-    april0="tag36_11_00032"
-    april1="tag36_11_00033"
-    april2="tag36_11_00034"
-    april3="tag36_11_00035"
-    april4="tag36_11_00036"/>
+    april2="tag36_11_00032"
+    april3="tag36_11_00033"
+    april4="tag36_11_00034"
+    april5="tag36_11_00035"
+    april6="tag36_11_00036"/>
 </robot>

File: rr_description/urdf/opponents/evgp_opponent_4.urdf.xacro (robot description, xacro)
@@ -2,8 +2,8 @@
     <xacro:include filename="evgp_body.urdf.xacro"/>
     <xacro:evgp_body collision_bitmask="0x40" color="Purple"
-    april0="tag36_11_00042"
-    april1="tag36_11_00043"
-    april2="tag36_11_00044"
-    april3="tag36_11_00045"
-    april4="tag36_11_00046"/>
+    april2="tag36_11_00042"
+    april3="tag36_11_00043"
+    april4="tag36_11_00044"
+    april5="tag36_11_00045"
+    april6="tag36_11_00046"/>
 </robot>

File: rr_description/urdf/rigatoni.urdf.xacro (robot description, xacro)
@@ -164,9 +164,9 @@
         </gazebo>
     </xacro:macro>
-    <xacro:april_link name="april_0" tag_number="tag36_11_00052"/>
-    <xacro:april_link name="april_1" tag_number="tag36_11_00053"/>
-    <xacro:april_link name="april_2" tag_number="tag36_11_00054"/>
-    <xacro:april_link name="april_3" tag_number="tag36_11_00055"/>
-    <xacro:april_link name="april_4" tag_number="tag36_11_00056"/>
+    <xacro:april_link name="april_2" tag_number="tag36_11_00052"/>
+    <xacro:april_link name="april_3" tag_number="tag36_11_00053"/>
+    <xacro:april_link name="april_4" tag_number="tag36_11_00054"/>
+    <xacro:april_link name="april_5" tag_number="tag36_11_00055"/>
+    <xacro:april_link name="april_6" tag_number="tag36_11_00056"/>
     <!-- ************************** Joints *************************** -->
     <xacro:property name="joint_flop_both" value="0.03"/>
@@ -225,9 +225,9 @@
     <xacro:set_base_footprint_to_link link_name="imu_bottom_link" xyz="0 0 0.21" rpy="0 0 0"/>
     <xacro:set_base_footprint_to_link link_name="imu_top_link" xyz="0.60 0.39 0.95" rpy="0 0 0"/>
-    <xacro:set_base_footprint_to_link link_name="april_0" xyz=".48  -0.55 0.26" rpy="0 0 ${pi/2}"/>
-    <xacro:set_base_footprint_to_link link_name="april_1" xyz="-.19 -0.43 0.26" rpy="0 0 ${pi/4}"/>
-    <xacro:set_base_footprint_to_link link_name="april_2" xyz="-.38  0    0.26" rpy="0 0 0"/>
-    <xacro:set_base_footprint_to_link link_name="april_3" xyz="-.19  0.43 0.26" rpy="0 0 -${pi/4}"/>
-    <xacro:set_base_footprint_to_link link_name="april_4" xyz=".48   0.55 0.26" rpy="0 0 ${pi/2}"/>
+    <xacro:set_base_footprint_to_link link_name="april_2" xyz=".48  -0.55 0.26" rpy="0 0 ${pi/2}"/>
+    <xacro:set_base_footprint_to_link link_name="april_3" xyz="-.19 -0.43 0.26" rpy="0 0 ${pi/4}"/>
+    <xacro:set_base_footprint_to_link link_name="april_4" xyz="-.38  0    0.26" rpy="0 0 0"/>
+    <xacro:set_base_footprint_to_link link_name="april_5" xyz="-.19  0.43 0.26" rpy="0 0 -${pi/4}"/>
+    <xacro:set_base_footprint_to_link link_name="april_6" xyz=".48   0.55 0.26" rpy="0 0 ${pi/2}"/>
     <!-- ******************* Sensors *********************** -->
     <!-- Velodyne Puck VLP-16 -->

Commit message: Enlarge tags

File: rr_description/urdf/opponents/evgp_body.urdf.xacro (robot description, xacro)
@@ -48,5 +48,5 @@
                 <visual>
                     <geometry>
-                        <box size="0.001 0.127 0.127 "/>
+                        <box size="0.001 0.15 0.15 "/>
                     </geometry>
                 </visual>

File: rr_description/urdf/rigatoni.urdf.xacro (robot description, xacro)
@@ -156,5 +156,5 @@
             <visual>
                 <geometry>
-                    <box size="0.001 0.127 0.127 "/>
+                    <box size="0.001 0.15 0.15 "/>
                 </geometry>
             </visual>
