Commit message: Update Rigatoni URDF  (#359)
* add lidar

* add close map

* Add model launch args

* Added new opponent_detection node and created new clusters.msg

* Added opponent detection launch file

* Revert "Add model launch args"

This reverts commit 1bc72f8419210b8e9e6922205c8438bd5df5be55.

* Revert "Revert "Add model launch args""

This reverts commit 29cda88199b929be88c043b3ce71577b1167bc02.

* Revert "Added opponent detection launch file"

This reverts commit 662664759f54ab249f1246931a67c566c3a7b980.

* Revert "Added new opponent_detection node and created new clusters.msg"

This reverts commit d574754a2ef08f669526dca5c9d07701fbc9ba9a.

* Add 3D Lidar Thresholding (#366)

* Added pcl_ros passthrough nodelet for 3D lidar z thresholding via lidar_z_threshold.launch and included it in mapping_sim.launch.

* Update Filter Max Z Value To Match Image

Changed filter_limit_max from 1 to 0.1 to match the image included in PR #366.

* Remove Newline From lidar_z_threshold.launch

Removed ending newline from lidar_z_threshold.launch.

* Change From /scan For Mapping to 3D Lidar /lidar_thresholded

* Change From /scan For Mapping to 3D Lidar /lidar_thresholded

* changes

* typo

* update rviz

* update rviz

* changes

* Removed submodule

* remove script

* update

* working'

* change

* Enlargen tags

* change param

Co-authored-by: Jeffrey Shao <shao.j109@gmail.com>
Co-authored-by: William Beard <52893758+wbeard01@users.noreply.github.com>
Co-authored-by: Charlie Jenkins <cjenkins72@gatech.edu>

File: rr_description/urdf/opponents/evgp_body.urdf.xacro (robot description, xacro)
@@ -8,5 +8,5 @@
     <xacro:macro name="mesh_geometry">
         <geometry>
-            <mesh filename="package://rr_description/meshes/EVGP_robot.STL" scale="0.001 0.001 0.001"/>
+            <mesh filename="package://rr_description/meshes/rigatoni.stl" scale="0.01 0.01 0.01"/>
         </geometry>
     </xacro:macro>
@@ -16,5 +16,5 @@
         </gazebo>
     </xacro:macro>
-    <xacro:macro name="evgp_body" params="collision_bitmask color">
+    <xacro:macro name="evgp_body" params="collision_bitmask color april2 april3 april4 april5 april6">
         <!-- ************************** Links *************************** -->
         <link name="base_footprint">
@@ -40,10 +40,46 @@
             </collision>
         </gazebo>
+        <gazebo reference="body_visual_origin">
+            <turnGravityOff>true</turnGravityOff>
+        </gazebo>
+        <xacro:macro name="april_link" params="name tag_number">
+            <link name="${name}">
+                <xacro:null_inertia/>
+                <visual>
+                    <geometry>
+                        <box size="0.001 0.127 0.127 "/>
+                    </geometry>
+                </visual>
+            </link>
+            <gazebo reference="${name}">
+                <material>${tag_number}</material>
+            </gazebo>
+        </xacro:macro>
+        <xacro:april_link name="april_2" tag_number="${april2}"/>
+        <xacro:april_link name="april_3" tag_number="${april3}"/>
+        <xacro:april_link name="april_4" tag_number="${april4}"/>
+        <xacro:april_link name="april_5" tag_number="${april5}"/>
+        <xacro:april_link name="april_6" tag_number="${april6}"/>
         <!-- ************************** Joints *************************** -->
         <joint name="base_footprint_to_mesh_origin" type="fixed">
             <parent link="base_footprint"/>
             <child link="body_visual_origin"/>
-            <origin xyz="1.45 0.515 -0.051" rpy="${pi/2} 0 ${-pi/2}"/>
+            <origin xyz="0.53 0 -0.05" rpy="${pi/2} 0 ${pi/2}"/>
         </joint>
+        <xacro:macro name="set_base_footprint_to_link" params="link_name xyz rpy">
+            <joint name="base_footprint_to_${link_name}" type="fixed">
+                <parent link="base_footprint"/>
+                <child link="${link_name}"/>
+                <origin xyz="${xyz}" rpy="${rpy}"/>
+            </joint>
+        </xacro:macro>
+        <xacro:set_base_footprint_to_link link_name="april_2" xyz=".48  -0.55 0.26" rpy="0 0 ${pi/2}"/>
+        <xacro:set_base_footprint_to_link link_name="april_3" xyz="-.19 -0.43 0.26" rpy="0 0 ${pi/4}"/>
+        <xacro:set_base_footprint_to_link link_name="april_4" xyz="-.38  0    0.26" rpy="0 0 0"/>
+        <xacro:set_base_footprint_to_link link_name="april_5" xyz="-.19  0.43 0.26" rpy="0 0 -${pi/4}"/>
+        <xacro:set_base_footprint_to_link link_name="april_6" xyz=".48   0.55 0.26" rpy="0 0 ${pi/2}"/>
+        <gazebo reference="base_footprint">
+            <kinematic>true</kinematic>
+        </gazebo>
     </xacro:macro>
 </robot>

File: rr_description/urdf/opponents/evgp_opponent_0.urdf.xacro (robot description, xacro)
@@ -1,7 +1,9 @@
 <robot name="evgp_opponent" xmlns:xacro="http://www.ros.org/wiki/xacro">
     <xacro:include filename="evgp_body.urdf.xacro"/>
-    <xacro:evgp_body collision_bitmask="0x4" color="Blue"/>
-    <gazebo reference="base_footprint">
-        <kinematic>true</kinematic>
-    </gazebo>
+    <xacro:evgp_body collision_bitmask="0x4" color="Blue"
+    april2="tag36_11_00002"
+    april3="tag36_11_00003"
+    april4="tag36_11_00004"
+    april5="tag36_11_00005"
+    april6="tag36_11_00006"/>
 </robot>

File: rr_description/urdf/opponents/evgp_opponent_1.urdf.xacro (robot description, xacro)
@@ -1,7 +1,9 @@
 <robot name="evgp_opponent" xmlns:xacro="http://www.ros.org/wiki/xacro">
     <xacro:include filename="evgp_body.urdf.xacro"/>
-    <xacro:evgp_body collision_bitmask="0x8" color="Green"/>
-    <gazebo reference="base_footprint">
-        <kinematic>true</kinematic>
-    </gazebo>
+    <xacro:evgp_body collision_bitmask="0x8" color="Green"
+    april2="tag36_11_00012"
+    april3="tag36_11_00013"
+    april4="tag36_11_00014"
+    april5="tag36_11_00015"
+    april6="tag36_11_00016"/>
 </robot>

File: rr_description/urdf/opponents/evgp_opponent_2.urdf.xacro (robot description, xacro)
@@ -1,7 +1,9 @@
 <robot name="evgp_opponent" xmlns:xacro="http://www.ros.org/wiki/xacro">
     <xacro:include filename="evgp_body.urdf.xacro"/>
-    <xacro:evgp_body collision_bitmask="0x10" color="Yellow"/>
-    <gazebo reference="base_footprint">
-        <kinematic>true</kinematic>
-    </gazebo>
+    <xacro:evgp_body collision_bitmask="0x10" color="Yellow"
+    april2="tag36_11_00022"
+    april3="tag36_11_00023"
+    april4="tag36_11_00024"
+    april5="tag36_11_00025"
+    april6="tag36_11_00026"/>
 </robot>

File: rr_description/urdf/opponents/evgp_opponent_3.urdf.xacro (robot description, xacro)
@@ -1,7 +1,9 @@
 <robot name="evgp_opponent" xmlns:xacro="http://www.ros.org/wiki/xacro">
     <xacro:include filename="evgp_body.urdf.xacro"/>
-    <xacro:evgp_body collision_bitmask="0x20" color="Red"/>
-    <gazebo reference="base_footprint">
-        <kinematic>true</kinematic>
-    </gazebo>
+    <xacro:evgp_body collision_bitmask="0x20" color="Red"
+    april2="tag36_11_00032"
+    april3="tag36_11_00033"
+    april4="tag36_11_00034"
+    april5="tag36_11_00035"
+    april6="tag36_11_00036"/>
 </robot>

File: rr_description/urdf/opponents/evgp_opponent_4.urdf.xacro (robot description, xacro)
@@ -1,7 +1,9 @@
 <robot name="evgp_opponent" xmlns:xacro="http://www.ros.org/wiki/xacro">
     <xacro:include filename="evgp_body.urdf.xacro"/>
-    <xacro:evgp_body collision_bitmask="0x40" color="Purple"/>
-    <gazebo reference="base_footprint">
-        <kinematic>true</kinematic>
-    </gazebo>
+    <xacro:evgp_body collision_bitmask="0x40" color="Purple"
+    april2="tag36_11_00042"
+    april3="tag36_11_00043"
+    april4="tag36_11_00044"
+    april5="tag36_11_00045"
+    april6="tag36_11_00046"/>
 </robot>
